File: PCB/motor-x.sch (KiCad schematic (older format))
At the start: 28 parts

Commit message: Fixed annotations and assignment errors.
Parts:
- removed C? (x5): 100nF, Capacitor_SMD:C_0603_1608Metric, symbol Device:C
- removed C?: 22nF - 50V, Capacitor_SMD:C_0603_1608Metric, symbol Device:C
- removed C?: 4.7uF, Resistor_SMD:R_0603_1608Metric, symbol Device:C
- removed C? (x2): 1nF, Resistor_SMD:R_0603_1608Metric, symbol Device:C
- removed R?: 10k, Resistor_SMD:R_0603_1608Metric, symbol Device:R
- removed R?: 0.12, Resistor_SMD:R_1206_3216Metric, symbol Device:R
- removed R? (x2): 100R, Resistor_SMD:R_0603_1608Metric, symbol Device:R
- removed TP?: X_OA1, TestPoint:TestPoint_Pad_D1.0mm, symbol Connector_Specialized:Test_Point
- removed TP?: X_OB2, TestPoint:TestPoint_Pad_D1.0mm, symbol Connector_Specialized:Test_Point
- removed U?: TMC2130-TA, custom-footprints:TQFP-48-1EP_7x7mm_P0.5mm_EP4.8x4.8mm-Heatsink, symbol remram-custom:TMC2130-TA
- added C34, C36, C37, C42, C44: 100nF, Capacitor_SMD:C_0603_1608Metric, symbol Device:C
- added C39: 22nF, Capacitor_SMD:C_0603_1608Metric, symbol Device:C
- added C43: 4.7uF, Capacitor_SMD:C_0603_1608Metric, symbol Device:C
- added C46, C47: 1nF, Capacitor_SMD:C_0603_1608Metric, symbol Device:C
- added R24: 0.12, Resistor_SMD:R_1206_3216Metric, symbol Device:R
- added R26: 10k, Resistor_SMD:R_0603_1608Metric, symbol Device:R
- added R28, R29: 100, Resistor_SMD:R_0603_1608Metric, symbol Device:R
- added TP12: X_OA1, TestPoint:TestPoint_Pad_D1.0mm, symbol Connector_Specialized:Test_Point
- added TP13: X_OB2, TestPoint:TestPoint_Pad_D1.0mm, symbol Connector_Specialized:Test_Point
- added U6: TMC2130-TA, custom-footprints:TQFP-48-1EP_7x7mm_P0.5mm_EP4.8x4.8mm-Heatsink, symbol remram-custom:TMC2130-TA
- C45, C48: renamed from C?; footprint Resistor_SMD:R_0603_1608Metric -> Capacitor_SMD:C_0603_1608Metric
- R27, R30: renamed from R?; value 100R -> 100
- gave numbers to parts that had none: 8

Commit message: Saving work in progress.
Every component now has a 3D mode.
Parts:
- J3: footprint Connector_PinHeader_2.54mm:PinHeader_1x04_P2.54mm_Vertical -> custom-footprints:70543-0003
Changed lines of the file:
@@
 $Descr A4 11693 8268
 encoding utf-8
-Sheet 6 9
+Sheet 5 9
 Title "Motor X-Axis"
 Date ""
@@
 X_EN
 $Comp
-L power:GNDA #PWR0151
+L power:GNDA #PWR058
 U 1 1 5AF8CE9A
 P 3550 3550
-F 0 "#PWR0151" H 3550 3300 50  0001 C CNN
+F 0 "#PWR058" H 3550 3300 50  0001 C CNN
 F 1 "GNDA" H 3555 3377 50  0000 C CNN
 F 2 "" H 3550 3550 50  0001 C CNN
@@
 MISO
 $Comp
-L power:GNDA #PWR0152
+L power:GNDA #PWR053
 U 1 1 5B0399AA
 P 1750 2150
-F 0 "#PWR0152" H 1750 1900 50  0001 C CNN
+F 0 "#PWR053" H 1750 1900 50  0001 C CNN
 F 1 "GNDA" V 1755 2023 50  0000 R CNN
 F 2 "" H 1750 2150 50  0001 C CNN
@@
 VDD_IN
 $Comp
-L power:GNDA #PWR0153
+L power:GNDA #PWR055
 U 1 1 5AF8CE9F
 P 2450 3550
-F 0 "#PWR0153" H 2450 3300 50  0001 C CNN
+F 0 "#PWR055" H 2450 3300 50  0001 C CNN
 F 1 "GNDA" H 2455 3377 50  0000 C CNN
 F 2 "" H 2450 3550 50  0001 C CNN
@@
 	3650 950  3900 950
 $Comp
-L power:GNDA #PWR0154
+L power:GNDA #PWR059
 U 1 1 5B03CBB9
 P 3650 1250
-F 0 "#PWR0154" H 3650 1000 50  0001 C CNN
+F 0 "#PWR059" H 3650 1000 50  0001 C CNN
 F 1 "GNDA" H 3655 1077 50  0000 C CNN
 F 2 "" H 3650 1250 50  0001 C CNN
@@
 $EndComp
 $Comp
-L power:GNDA #PWR0155
+L power:GNDA #PWR061
 U 1 1 5AF8CEA9
 P 4500 1950
-F 0 "#PWR0155" H 4500 1700 50  0001 C CNN
+F 0 "#PWR061" H 4500 1700 50  0001 C CNN
 F 1 "GNDA" H 4505 1777 50  0000 C CNN
 F 2 "" H 4500 1950 50  0001 C CNN
@@
 $EndComp
 $Comp
-L power:GNDA #PWR0156
+L power:GNDA #PWR052
 U 1 1 5B03E652
 P 1250 3250
-F 0 "#PWR0156" H 1250 3000 50  0001 C CNN
+F 0 "#PWR052" H 1250 3000 50  0001 C CNN
 F 1 "GNDA" H 1255 3077 50  0000 C CNN
 F 2 "" H 1250 3250 50  0001 C CNN
@@
 Connection ~ 4500 2250
 $Comp
-L power:GNDA #PWR0157
+L power:GNDA #PWR060
 U 1 1 5B043BF7
 P 4150 2450
-F 0 "#PWR0157" H 4150 2200 50  0001 C CNN
+F 0 "#PWR060" H 4150 2200 50  0001 C CNN
 F 1 "GNDA" V 4155 2322 50  0000 R CNN
 F 2 "" H 4150 2450 50  0001 C CNN
@@
 $EndComp
 $Comp
-L power:GNDA #PWR0158
+L power:GNDA #PWR063
 U 1 1 5AF8CEAF
 P 5600 2350
-F 0 "#PWR0158" H 5600 2100 50  0001 C CNN
+F 0 "#PWR063" H 5600 2100 50  0001 C CNN
 F 1 "GNDA" H 5605 2177 50  0000 C CNN
 F 2 "" H 5600 2350 50  0001 C CNN
@@
 $EndComp
 $Comp
-L power:GNDA #PWR0159
+L power:GNDA #PWR057
 U 1 1 5AF8CEB4
 P 2850 4250
-F 0 "#PWR0159" H 2850 4000 50  0001 C CNN
+F 0 "#PWR057" H 2850 4000 50  0001 C CNN
 F 1 "GNDA" H 2855 4077 50  0000 C CNN
 F 2 "" H 2850 4250 50  0001 C CNN
@@
 F 0 "J3" H 9779 1142 50  0000 L CNN
 F 1 "70543-0003" H 9779 1051 50  0000 L CNN
-F 2 "Connector_PinHeader_2.54mm:PinHeader_1x04_P2.54mm_Vertical" H 9700 1150 50  0001 C CNN
+F 2 "custom-footprints:70543-0003" H 9700 1150 50  0001 C CNN
 F 3 "https://www.mouser.de/ProductDetail/Molex/70543-0003?qs=sGAEpiMZZMs%252bGHln7q6pm%252bS0pk2Wo0XxCD3CKlCQrmU%3d" H 9700 1150 50  0001 C CNN
 	1    9700 1150
@@
 $EndComp
 $Comp
-L power:GNDA #PWR0160
+L power:GNDA #PWR056
 U 1 1 5AF8CEBE
 P 2850 1050
-F 0 "#PWR0160" H 2850 800 50  0001 C CNN
+F 0 "#PWR056" H 2850 800 50  0001 C CNN
 F 1 "GNDA" H 2855 877 50  0000 C CNN
 F 2 "" H 2850 1050 50  0001 C CNN
@@
 $EndComp
 $Comp
-L power:GNDA #PWR0161
+L power:GNDA #PWR067
 U 1 1 5B0AC243
 P 8050 1750
-F 0 "#PWR0161" H 8050 1500 50  0001 C CNN
+F 0 "#PWR067" H 8050 1500 50  0001 C CNN
 F 1 "GNDA" H 8055 1577 50  0000 C CNN
 F 2 "" H 8050 1750 50  0001 C CNN
@@
 $EndComp
 $Comp
-L power:GNDA #PWR0162
+L power:GNDA #PWR066
 U 1 1 5B0AC39D
 P 7700 1750
-F 0 "#PWR0162" H 7700 1500 50  0001 C CNN
+F 0 "#PWR066" H 7700 1500 50  0001 C CNN
 F 1 "GNDA" H 7705 1577 50  0000 C CNN
 F 2 "" H 7700 1750 50  0001 C CNN
@@
 $EndComp
 $Comp
-L power:GNDA #PWR0163
+L power:GNDA #PWR065
 U 1 1 5AF8CECA
 P 7350 1750
-F 0 "#PWR0163" H 7350 1500 50  0001 C CNN
+F 0 "#PWR065" H 7350 1500 50  0001 C CNN
 F 1 "GNDA" H 7355 1577 50  0000 C CNN
 F 2 "" H 7350 1750 50  0001 C CNN
@@
 $EndComp
 $Comp
-L power:GNDA #PWR0164
+L power:GNDA #PWR064
 U 1 1 5B0AD57A
 P 7000 1750
-F 0 "#PWR0164" H 7000 1500 50  0001 C CNN
+F 0 "#PWR064" H 7000 1500 50  0001 C CNN
 F 1 "GNDA" H 7005 1577 50  0000 C CNN
 F 2 "" H 7000 1750 50  0001 C CNN
@@
 $EndComp
 $Comp
-L power:GNDA #PWR0165
+L power:GNDA #PWR062
 U 1 1 5B0D4996
 P 4600 4300
-F 0 "#PWR0165" H 4600 4050 50  0001 C CNN
+F 0 "#PWR062" H 4600 4050 50  0001 C CNN
 F 1 "GNDA" V 4605 4173 50  0000 R CNN
 F 2 "" H 4600 4300 50  0001 C CNN
@@
 $EndComp
 $Comp
-L power:GNDA #PWR0166
+L power:GNDA #PWR054
 U 1 1 5AF8CE97
 P 2350 1550
-F 0 "#PWR0166" H 2350 1300 50  0001 C CNN
+F 0 "#PWR054" H 2350 1300 50  0001 C CNN
 F 1 "GNDA" H 2355 1377 50  0000 C CNN
 F 2 "" H 2350 1550 50  0001 C CNN

Commit message: Removed logic level converter. Changed LDO.
Parts:
- renumbered C38 to C13, C35 to C14, C37 to C15, C45 to C16, C46 to C17, C47 to C18, C48 to C19, C39 to C20, C40 to C21, C43 to C22, C34 to C23, C36 to C24, C41 to C25, C42 to C26, C44 to C27, R27 to R12, R28 to R13, R25 to R14, R29 to R15, R30 to R16, R26 to R17, R24 to R18, TP12 to TP11, TP14 to TP12, TP15 to TP14, U6 to U3
Connections:
- net labels added: SS_X
- net labels removed: SSX
