File: PCB/motor-y.sch (KiCad schematic (older format))
At the start: 28 parts

Commit message: Fixed annotations and assignment errors.
Parts:
- removed C? (x4): 100nF, Capacitor_SMD:C_0603_1608Metric, symbol Device:C
- removed C?: 470nF, Capacitor_SMD:C_0603_1608Metric, symbol Device:C
- removed C? (x3): 1nF, Resistor_SMD:R_0603_1608Metric, symbol Device:C
- removed C?: 100uF, Capacitor_THT:CP_Radial_D6.3mm_P2.50mm, symbol Device:CP
- removed J?: 70543-0003, Connector_PinHeader_2.54mm:PinHeader_1x04_P2.54mm_Vertical, symbol Connector_Generic:Conn_01x04
- removed R? (x2): 0.12, Resistor_SMD:R_1206_3216Metric, symbol Device:R
- removed R? (x2): 100R, Resistor_SMD:R_0603_1608Metric, symbol Device:R
- removed TP?: X_OA2, TestPoint:TestPoint_Pad_D1.0mm, symbol Connector_Specialized:Test_Point
- removed TP?: X_OA1, TestPoint:TestPoint_Pad_D1.0mm, symbol Connector_Specialized:Test_Point
- removed TP?: X_OB1, TestPoint:TestPoint_Pad_D1.0mm, symbol Connector_Specialized:Test_Point
- added C50, C53, C57, C59: 100nF, Capacitor_SMD:C_0603_1608Metric, symbol Device:C
- added C55: 470nF, Capacitor_SMD:C_0603_1608Metric, symbol Device:C
- added C56: 100uF, Capacitor_THT:CP_Radial_D6.3mm_P2.50mm, symbol Device:CP
- added C60, C62, C63: 1nF, Capacitor_SMD:C_0603_1608Metric, symbol Device:C
- added J4: 70543-0003, Connector_PinHeader_2.54mm:PinHeader_1x04_P2.54mm_Vertical, symbol Connector_Generic:Conn_01x04
- added R31, R32: 0.12, Resistor_SMD:R_1206_3216Metric, symbol Device:R
- added R34, R37: 100, Resistor_SMD:R_0603_1608Metric, symbol Device:R
- added TP16: X_OA1, TestPoint:TestPoint_Pad_D1.0mm, symbol Connector_Specialized:Test_Point
- added TP18: X_OA2, TestPoint:TestPoint_Pad_D1.0mm, symbol Connector_Specialized:Test_Point
- added TP19: X_OB1, TestPoint:TestPoint_Pad_D1.0mm, symbol Connector_Specialized:Test_Point
- C54: renamed from C?; value 22nF - 50V -> 22nF
- C58, C61: renamed from C?; footprint Resistor_SMD:R_0603_1608Metric -> Capacitor_SMD:C_0603_1608Metric
- R35, R36: renamed from R?; value 100R -> 100
- gave numbers to parts that had none: 6
Connections:
- net labels added: SSY, Y_DIAG, Y_DIR, Y_EN, Y_STEP
- net labels removed: SSX, X_DIAG, X_DIR, X_EN, X_STEP

Commit message: Saving work in progress.
Every component now has a 3D mode.
Parts:
- J4: footprint Connector_PinHeader_2.54mm:PinHeader_1x04_P2.54mm_Vertical -> custom-footprints:70543-0003
Changed lines of the file:
@@
 Y_EN
 $Comp
-L power:GNDA #PWR0167
+L power:GNDA #PWR074
 U 1 1 5B038691
 P 3550 3550
-F 0 "#PWR0167" H 3550 3300 50  0001 C CNN
+F 0 "#PWR074" H 3550 3300 50  0001 C CNN
 F 1 "GNDA" H 3555 3377 50  0000 C CNN
 F 2 "" H 3550 3550 50  0001 C CNN
@@
 MISO
 $Comp
-L power:GNDA #PWR0168
+L power:GNDA #PWR069
 U 1 1 5AF8CE9C
 P 1750 2150
-F 0 "#PWR0168" H 1750 1900 50  0001 C CNN
+F 0 "#PWR069" H 1750 1900 50  0001 C CNN
 F 1 "GNDA" V 1755 2023 50  0000 R CNN
 F 2 "" H 1750 2150 50  0001 C CNN
@@
 VDD_IN
 $Comp
-L power:GNDA #PWR0169
+L power:GNDA #PWR071
 U 1 1 5B03A4B5
 P 2450 3550
-F 0 "#PWR0169" H 2450 3300 50  0001 C CNN
+F 0 "#PWR071" H 2450 3300 50  0001 C CNN
 F 1 "GNDA" H 2455 3377 50  0000 C CNN
 F 2 "" H 2450 3550 50  0001 C CNN
@@
 	3650 950  3900 950
 $Comp
-L power:GNDA #PWR0170
+L power:GNDA #PWR075
 U 1 1 5AF8CEA6
 P 3650 1250
-F 0 "#PWR0170" H 3650 1000 50  0001 C CNN
+F 0 "#PWR075" H 3650 1000 50  0001 C CNN
 F 1 "GNDA" H 3655 1077 50  0000 C CNN
 F 2 "" H 3650 1250 50  0001 C CNN
@@
 $EndComp
 $Comp
-L power:GNDA #PWR0171
+L power:GNDA #PWR077
 U 1 1 5B03D801
 P 4500 1950
-F 0 "#PWR0171" H 4500 1700 50  0001 C CNN
+F 0 "#PWR077" H 4500 1700 50  0001 C CNN
 F 1 "GNDA" H 4505 1777 50  0000 C CNN
 F 2 "" H 4500 1950 50  0001 C CNN
@@
 $EndComp
 $Comp
-L power:GNDA #PWR0172
+L power:GNDA #PWR068
 U 1 1 5AF8CEAB
 P 1250 3250
-F 0 "#PWR0172" H 1250 3000 50  0001 C CNN
+F 0 "#PWR068" H 1250 3000 50  0001 C CNN
 F 1 "GNDA" H 1255 3077 50  0000 C CNN
 F 2 "" H 1250 3250 50  0001 C CNN
@@
 Connection ~ 4500 2250
 $Comp
-L power:GNDA #PWR0173
+L power:GNDA #PWR076
 U 1 1 5AF8CEAC
 P 4150 2450
-F 0 "#PWR0173" H 4150 2200 50  0001 C CNN
+F 0 "#PWR076" H 4150 2200 50  0001 C CNN
 F 1 "GNDA" V 4155 2322 50  0000 R CNN
 F 2 "" H 4150 2450 50  0001 C CNN
@@
 $EndComp
 $Comp
-L power:GNDA #PWR0174
+L power:GNDA #PWR079
 U 1 1 5B044BA0
 P 5600 2350
-F 0 "#PWR0174" H 5600 2100 50  0001 C CNN
+F 0 "#PWR079" H 5600 2100 50  0001 C CNN
 F 1 "GNDA" H 5605 2177 50  0000 C CNN
 F 2 "" H 5600 2350 50  0001 C CNN
@@
 $EndComp
 $Comp
-L power:GNDA #PWR0175
+L power:GNDA #PWR073
 U 1 1 5B04739D
 P 2850 4250
-F 0 "#PWR0175" H 2850 4000 50  0001 C CNN
+F 0 "#PWR073" H 2850 4000 50  0001 C CNN
 F 1 "GNDA" H 2855 4077 50  0000 C CNN
 F 2 "" H 2850 4250 50  0001 C CNN
@@
 F 0 "J4" H 9779 1142 50  0000 L CNN
 F 1 "70543-0003" H 9779 1051 50  0000 L CNN
-F 2 "Connector_PinHeader_2.54mm:PinHeader_1x04_P2.54mm_Vertical" H 9700 1150 50  0001 C CNN
+F 2 "custom-footprints:70543-0003" H 9700 1150 50  0001 C CNN
 F 3 "https://www.mouser.de/ProductDetail/Molex/70543-0003?qs=sGAEpiMZZMs%252bGHln7q6pm%252bS0pk2Wo0XxCD3CKlCQrmU%3d" H 9700 1150 50  0001 C CNN
 	1    9700 1150
@@
 $EndComp
 $Comp
-L power:GNDA #PWR0176
+L power:GNDA #PWR072
 U 1 1 5B0A4470
 P 2850 1050
-F 0 "#PWR0176" H 2850 800 50  0001 C CNN
+F 0 "#PWR072" H 2850 800 50  0001 C CNN
 F 1 "GNDA" H 2855 877 50  0000 C CNN
 F 2 "" H 2850 1050 50  0001 C CNN
@@
 $EndComp
 $Comp
-L power:GNDA #PWR0177
+L power:GNDA #PWR083
 U 1 1 5AF8CEC5
 P 8050 1750
-F 0 "#PWR0177" H 8050 1500 50  0001 C CNN
+F 0 "#PWR083" H 8050 1500 50  0001 C CNN
 F 1 "GNDA" H 8055 1577 50  0000 C CNN
 F 2 "" H 8050 1750 50  0001 C CNN
@@
 $EndComp
 $Comp
-L power:GNDA #PWR0178
+L power:GNDA #PWR082
 U 1 1 5AF8CEC7
 P 7700 1750
-F 0 "#PWR0178" H 7700 1500 50  0001 C CNN
+F 0 "#PWR082" H 7700 1500 50  0001 C CNN
 F 1 "GNDA" H 7705 1577 50  0000 C CNN
 F 2 "" H 7700 1750 50  0001 C CNN
@@
 $EndComp
 $Comp
-L power:GNDA #PWR0179
+L power:GNDA #PWR081
 U 1 1 5B0ACC86
 P 7350 1750
-F 0 "#PWR0179" H 7350 1500 50  0001 C CNN
+F 0 "#PWR081" H 7350 1500 50  0001 C CNN
 F 1 "GNDA" H 7355 1577 50  0000 C CNN
 F 2 "" H 7350 1750 50  0001 C CNN
@@
 $EndComp
 $Comp
-L power:GNDA #PWR0180
+L power:GNDA #PWR080
 U 1 1 5AF8CECC
 P 7000 1750
-F 0 "#PWR0180" H 7000 1500 50  0001 C CNN
+F 0 "#PWR080" H 7000 1500 50  0001 C CNN
 F 1 "GNDA" H 7005 1577 50  0000 C CNN
 F 2 "" H 7000 1750 50  0001 C CNN
@@
 $EndComp
 $Comp
-L power:GNDA #PWR0181
+L power:GNDA #PWR078
 U 1 1 5AF8CED3
 P 4600 4300
-F 0 "#PWR0181" H 4600 4050 50  0001 C CNN
+F 0 "#PWR078" H 4600 4050 50  0001 C CNN
 F 1 "GNDA" V 4605 4173 50  0000 R CNN
 F 2 "" H 4600 4300 50  0001 C CNN
@@
 $EndComp
 $Comp
-L power:GNDA #PWR0182
+L power:GNDA #PWR070
 U 1 1 5AF9A5D7
 P 2350 1550
-F 0 "#PWR0182" H 2350 1300 50  0001 C CNN
+F 0 "#PWR070" H 2350 1300 50  0001 C CNN
 F 1 "GNDA" H 2355 1377 50  0000 C CNN
 F 2 "" H 2350 1550 50  0001 C CNN

Commit message: Removed logic level converter. Changed LDO.
Parts:
- renumbered C53 to C28, C50 to C29, C52 to C30, C60 to C31, C61 to C32, C62 to C33, C63 to C34, C54 to C35, C55 to C36, C58 to C37, C49 to C38, C51 to C39, C56 to C40, C57 to C41, C59 to C42, R34 to R19, R35 to R20, R32 to R21, R36 to R22, R37 to R23, R33 to R24, R31 to R25, TP16 to TP15, TP18 to TP16, TP19 to TP18, U7 to U4
Connections:
- net labels added: SS_Y
- net labels removed: SSY
