File: PCB/connectors.sch (KiCad schematic (older format))
At the start: 38 parts, among them J10 67068-8000, J11 61201021621, J12 61201021621, J13 70543-0002, J14 70543-0002, J15 61201021621, J16 70543-0001, J17 70543-0002, J18 70543-0002, J19 62201021121, J20 70543-0001, J21 70543-0001, J22 70543-0001, J7 70543-0002, J8 70543-0002, J9 70543-0001

Commit message: Finished TMC2130 placement.
Motor sheets is now instanced. That way I simply could use
a KiCad plugin to duplicate the layout in Pcbnew.
Parts:
- renumbered C93 to C48, C94 to C49, C95 to C50, J13 to J10, J14 to J11, J15 to J12, J16 to J13, J17 to J14, J18 to J15, J19 to J16, J20 to J17, J21 to J18, J22 to J19, J7 to J4, J8 to J5, J9 to J6, J10 to J7, J11 to J8, J12 to J9, R48 to R27, R49 to R28, R50 to R29, R51 to R30, R52 to R31, R53 to R32, TP28 to TP16, TP29 to TP17, TP30 to TP18, TP31 to TP19, TP32 to TP20, TP33 to TP21, TP34 to TP22

Commit message: Finished placement. Currently routing last paths.
Parts:
- renumbered C48 to C42, C49 to C43, C50 to C44, R27 to R23, R28 to R24, R29 to R25, R30 to R26, R31 to R27, R32 to R28
Changed lines of the file:
@@
 $Descr A4 11693 8268
 encoding utf-8
-Sheet 9 9
+Sheet 6 9
 Title "Connectors"
 Date ""
@@
 $EndComp
 $Comp
-L Device:R R28
+L Device:R R24
 U 1 1 5B1719A1
 P 2600 4600
-F 0 "R28" V 2393 4600 50  0000 C CNN
+F 0 "R24" V 2393 4600 50  0000 C CNN
 F 1 "4.7k" V 2484 4600 50  0000 C CNN
 F 2 "Resistor_SMD:R_0603_1608Metric" V 2530 4600 50  0001 C CNN
@@
 $EndComp
 $Comp
-L Device:R R27
+L Device:R R23
 U 1 1 5B1719A8
 P 3050 4350
-F 0 "R27" H 3120 4396 50  0000 L CNN
+F 0 "R23" H 3120 4396 50  0000 L CNN
 F 1 "4.7k" H 3120 4305 50  0000 L CNN
 F 2 "Resistor_SMD:R_0603_1608Metric" V 2980 4350 50  0001 C CNN
@@
 	3050 4600 2750 4600
 $Comp
-L power:GND #PWR078
+L power:GND #PWR075
 U 1 1 5B1719B0
 P 2000 5000
-F 0 "#PWR078" H 2000 4750 50  0001 C CNN
+F 0 "#PWR075" H 2000 4750 50  0001 C CNN
 F 1 "GND" H 2005 4827 50  0000 C CNN
 F 2 "" H 2000 5000 50  0001 C CNN
@@
 Connection ~ 3050 4600
 $Comp
-L power:GND #PWR076
+L power:GND #PWR073
 U 1 1 5B1719CA
 P 3950 4700
-F 0 "#PWR076" H 3950 4450 50  0001 C CNN
+F 0 "#PWR073" H 3950 4450 50  0001 C CNN
 F 1 "GND" H 3955 4527 50  0000 C CNN
 F 2 "" H 3950 4700 50  0001 C CNN
@@
 	3400 4600 3050 4600
 $Comp
-L Device:C C48
+L Device:C C42
 U 1 1 5B1719D4
 P 1250 4750
-F 0 "C48" H 1365 4796 50  0000 L CNN
+F 0 "C42" H 1365 4796 50  0000 L CNN
 F 1 "100nF" H 1365 4705 50  0000 L CNN
 F 2 "Capacitor_SMD:C_0603_1608Metric" H 1288 4600 50  0001 C CNN
@@
 Connection ~ 1250 4600
 $Comp
-L power:GND #PWR077
+L power:GND #PWR074
 U 1 1 5B1719DF
 P 1250 4900
-F 0 "#PWR077" H 1250 4650 50  0001 C CNN
+F 0 "#PWR074" H 1250 4650 50  0001 C CNN
 F 1 "GND" H 1255 4727 50  0000 C CNN
 F 2 "" H 1250 4900 50  0001 C CNN
@@
 $EndComp
 $Comp
-L Device:R R30
+L Device:R R26
 U 1 1 5B171A02
 P 2600 5800
-F 0 "R30" V 2393 5800 50  0000 C CNN
+F 0 "R26" V 2393 5800 50  0000 C CNN
 F 1 "4.7k" V 2484 5800 50  0000 C CNN
 F 2 "Resistor_SMD:R_0603_1608Metric" V 2530 5800 50  0001 C CNN
@@
 $EndComp
 $Comp
-L Device:R R29
+L Device:R R25
 U 1 1 5B171A09
 P 3050 5550
-F 0 "R29" H 3120 5596 50  0000 L CNN
+F 0 "R25" H 3120 5596 50  0000 L CNN
 F 1 "4.7k" H 3120 5505 50  0000 L CNN
 F 2 "Resistor_SMD:R_0603_1608Metric" V 2980 5550 50  0001 C CNN
@@
 	3050 5800 2750 5800
 $Comp
-L power:GND #PWR081
+L power:GND #PWR078
 U 1 1 5B171A11
 P 2000 6150
-F 0 "#PWR081" H 2000 5900 50  0001 C CNN
+F 0 "#PWR078" H 2000 5900 50  0001 C CNN
 F 1 "GND" H 2005 5977 50  0000 C CNN
 F 2 "" H 2000 6150 50  0001 C CNN
@@
 Connection ~ 3050 5800
 $Comp
-L power:GND #PWR079
+L power:GND #PWR076
 U 1 1 5B171A2B
 P 3950 5900
-F 0 "#PWR079" H 3950 5650 50  0001 C CNN
+F 0 "#PWR076" H 3950 5650 50  0001 C CNN
 F 1 "GND" H 3955 5727 50  0000 C CNN
 F 2 "" H 3950 5900 50  0001 C CNN
@@
 	3400 5800 3050 5800
 $Comp
-L Device:C C49
+L Device:C C43
 U 1 1 5B171A35
 P 1250 5950
-F 0 "C49" H 1365 5996 50  0000 L CNN
+F 0 "C43" H 1365 5996 50  0000 L CNN
 F 1 "100nF" H 1365 5905 50  0000 L CNN
 F 2 "Capacitor_SMD:C_0603_1608Metric" H 1288 5800 50  0001 C CNN
@@
 Connection ~ 1250 5800
 $Comp
-L power:GND #PWR080
+L power:GND #PWR077
 U 1 1 5B171A40
 P 1250 6100
-F 0 "#PWR080" H 1250 5850 50  0001 C CNN
+F 0 "#PWR077" H 1250 5850 50  0001 C CNN
 F 1 "GND" H 1255 5927 50  0000 C CNN
 F 2 "" H 1250 6100 50  0001 C CNN
@@
 $EndComp
 $Comp
-L Device:R R32
+L Device:R R28
 U 1 1 5B171A63
 P 2600 7000
-F 0 "R32" V 2393 7000 50  0000 C CNN
+F 0 "R28" V 2393 7000 50  0000 C CNN
 F 1 "4.7k" V 2484 7000 50  0000 C CNN
 F 2 "Resistor_SMD:R_0603_1608Metric" V 2530 7000 50  0001 C CNN
@@
 $EndComp
 $Comp
-L Device:R R31
+L Device:R R27
 U 1 1 5B171A6A
 P 3050 6750
-F 0 "R31" H 3120 6796 50  0000 L CNN
+F 0 "R27" H 3120 6796 50  0000 L CNN
 F 1 "4.7k" H 3120 6705 50  0000 L CNN
 F 2 "Resistor_SMD:R_0603_1608Metric" V 2980 6750 50  0001 C CNN
@@
 	3050 7000 2750 7000
 $Comp
-L power:GND #PWR084
+L power:GND #PWR081
 U 1 1 5B171A72
 P 2000 7350
-F 0 "#PWR084" H 2000 7100 50  0001 C CNN
+F 0 "#PWR081" H 2000 7100 50  0001 C CNN
 F 1 "GND" H 2005 7177 50  0000 C CNN
 F 2 "" H 2000 7350 50  0001 C CNN
@@
 Connection ~ 3050 7000
 $Comp
-L power:GND #PWR082
+L power:GND #PWR079
 U 1 1 5B171A8C
 P 3950 7100
-F 0 "#PWR082" H 3950 6850 50  0001 C CNN
+F 0 "#PWR079" H 3950 6850 50  0001 C CNN
 F 1 "GND" H 3955 6927 50  0000 C CNN
 F 2 "" H 3950 7100 50  0001 C CNN
@@
 	3400 7000 3050 7000
 $Comp
-L Device:C C50
+L Device:C C44
 U 1 1 5B171A96
 P 1250 7150
-F 0 "C50" H 1365 7196 50  0000 L CNN
+F 0 "C44" H 1365 7196 50  0000 L CNN
 F 1 "100nF" H 1365 7105 50  0000 L CNN
 F 2 "Capacitor_SMD:C_0603_1608Metric" H 1288 7000 50  0001 C CNN
@@
 Connection ~ 1250 7000
 $Comp
-L power:GND #PWR083
+L power:GND #PWR080
 U 1 1 5B171AA1
 P 1250 7300
-F 0 "#PWR083" H 1250 7050 50  0001 C CNN
+F 0 "#PWR080" H 1250 7050 50  0001 C CNN
 F 1 "GND" H 1255 7127 50  0000 C CNN
 F 2 "" H 1250 7300 50  0001 C CNN
@@
 Endstops
 $Comp
-L power:GND #PWR066
+L power:GND #PWR063
 U 1 1 5B171AAF
 P 5550 950
-F 0 "#PWR066" H 5550 700 50  0001 C CNN
+F 0 "#PWR063" H 5550 700 50  0001 C CNN
 F 1 "GND" V 5555 822 50  0000 R CNN
 F 2 "" H 5550 950 50  0001 C CNN
@@
 $EndComp
 $Comp
-L power:GND #PWR067
+L power:GND #PWR064
 U 1 1 5B171ABF
 P 6750 950
-F 0 "#PWR067" H 6750 700 50  0001 C CNN
+F 0 "#PWR064" H 6750 700 50  0001 C CNN
 F 1 "GND" V 6755 822 50  0000 R CNN
 F 2 "" H 6750 950 50  0001 C CNN
@@
 $EndComp
 $Comp
-L power:GND #PWR068
+L power:GND #PWR065
 U 1 1 5B171ACF
 P 5550 1350
-F 0 "#PWR068" H 5550 1100 50  0001 C CNN
+F 0 "#PWR065" H 5550 1100 50  0001 C CNN
 F 1 "GND" V 5555 1222 50  0000 R CNN
 F 2 "" H 5550 1350 50  0001 C CNN
@@
 $EndComp
 $Comp
-L power:GND #PWR069
+L power:GND #PWR066
 U 1 1 5B171ADD
 P 6750 1350
-F 0 "#PWR069" H 6750 1100 50  0001 C CNN
+F 0 "#PWR066" H 6750 1100 50  0001 C CNN
 F 1 "GND" V 6755 1222 50  0000 R CNN
 F 2 "" H 6750 1350 50  0001 C CNN
@@
 $EndComp
 $Comp
-L power:GND #PWR073
+L power:GND #PWR070
 U 1 1 5B171AED
 P 5550 1750
-F 0 "#PWR073" H 5550 1500 50  0001 C CNN
+F 0 "#PWR070" H 5550 1500 50  0001 C CNN
 F 1 "GND" V 5555 1622 50  0000 R CNN
 F 2 "" H 5550 1750 50  0001 C CNN
@@
 $EndComp
 $Comp
-L power:GND #PWR074
+L power:GND #PWR071
 U 1 1 5B171AFB
 P 6750 1750
-F 0 "#PWR074" H 6750 1500 50  0001 C CNN
+F 0 "#PWR071" H 6750 1500 50  0001 C CNN
 F 1 "GND" V 6755 1622 50  0000 R CNN
 F 2 "" H 6750 1750 50  0001 C CNN
@@
 SWD
 $Comp
-L power:GND #PWR075
+L power:GND #PWR072
 U 1 1 5B17C4C4
 P 850 2900
-F 0 "#PWR075" H 850 2650 50  0001 C CNN
+F 0 "#PWR072" H 850 2650 50  0001 C CNN
 F 1 "GND" H 855 2727 50  0000 C CNN
 F 2 "" H 850 2900 50  0001 C CNN
@@
 VBUS
 $Comp
-L power:GNDS #PWR072
+L power:GNDS #PWR069
 U 1 1 5AF8309F
 P 1150 1700
-F 0 "#PWR072" H 1150 1450 50  0001 C CNN
+F 0 "#PWR069" H 1150 1450 50  0001 C CNN
 F 1 "GNDS" H 1155 1527 50  0000 C CNN
 F 2 "" H 1150 1700 50  0001 C CNN
@@
 VDD5V
 $Comp
-L power:GND #PWR070
+L power:GND #PWR067
 U 1 1 5AFA04BE
 P 2500 1500
-F 0 "#PWR070" H 2500 1250 50  0001 C CNN
+F 0 "#PWR067" H 2500 1250 50  0001 C CNN
 F 1 "GND" V 2505 1372 50  0000 R CNN
 F 2 "" H 2500 1500 50  0001 C CNN
@@
 VDD3V3
 $Comp
-L power:GND #PWR071
+L power:GND #PWR068
 U 1 1 5B067CCF
 P 8300 1600
-F 0 "#PWR071" H 8300 1350 50  0001 C CNN
+F 0 "#PWR068" H 8300 1350 50  0001 C CNN
 F 1 "GND" V 8305 1472 50  0000 R CNN
 F 2 "" H 8300 1600 50  0001 C CNN

Commit message: Added the secnd Z connection.
Parts:
- added J16: 70543-0003, custom-footprints:70543-0003, symbol Connector_Generic:Conn_01x04
- renumbered J16 to J17, J17 to J18, J18 to J19, J19 to J20
Connections:
- net labels added: Z_OA1, Z_OA2, Z_OB1, Z_OB2
- wire segments 67 -> 71
Other:
- note added: "Z-Axis second connector"
Changed lines of the file:
@@
 	3050 4600 3050 4500
 $Comp
-L Connector_Generic:Conn_01x02 J17
+L Connector_Generic:Conn_01x02 J18
 U 1 1 5B1719C1
 P 4150 4600
-F 0 "J17" H 4229 4592 50  0000 L CNN
+F 0 "J18" H 4229 4592 50  0000 L CNN
 F 1 "70543-0001" H 4229 4501 50  0000 L CNN
 F 2 "custom-footprints:70543-0001" H 4150 4600 50  0001 C CNN
@@
 	3050 5800 3050 5700
 $Comp
-L Connector_Generic:Conn_01x02 J18
+L Connector_Generic:Conn_01x02 J19
 U 1 1 5B171A22
 P 4150 5800
-F 0 "J18" H 4229 5792 50  0000 L CNN
+F 0 "J19" H 4229 5792 50  0000 L CNN
 F 1 "70543-0001" H 4229 5701 50  0000 L CNN
 F 2 "custom-footprints:70543-0001" H 4150 5800 50  0001 C CNN
@@
 	3050 7000 3050 6900
 $Comp
-L Connector_Generic:Conn_01x02 J19
+L Connector_Generic:Conn_01x02 J20
 U 1 1 5B171A83
 P 4150 7000
-F 0 "J19" H 4229 6992 50  0000 L CNN
+F 0 "J20" H 4229 6992 50  0000 L CNN
 F 1 "70543-0001" H 4229 6901 50  0000 L CNN
 F 2 "custom-footprints:70543-0001" H 4150 7000 50  0001 C CNN
@@
 	7650 2100 5150 2100
 $Comp
-L Connector_Generic:Conn_02x05_Odd_Even J16
+L Connector_Generic:Conn_02x05_Odd_Even J17
 U 1 1 5B17C4BC
-P 1200 2700
-F 0 "J16" H 1250 3150 50  0000 C CNN
-F 1 "62201021121" H 1250 3050 50  0000 C CNN
-F 2 "Connector_PinHeader_1.27mm:PinHeader_2x05_P1.27mm_Vertical" H 1200 2700 50  0001 C CNN
-F 3 "https://www.mouser.de/datasheet/2/445/6220xx21121-542317.pdf" H 1200 2700 50  0001 C CNN
-	1    1200 2700
-	1    0    0    -1
-$EndComp
-Text Notes 1250 2150 0    50   ~ 0
+P 1200 2750
+F 0 "J17" H 1250 3200 50  0000 C CNN
+F 1 "62201021121" H 1250 3100 50  0000 C CNN
+F 2 "Connector_PinHeader_1.27mm:PinHeader_2x05_P1.27mm_Vertical" H 1200 2750 50  0001 C CNN
+F 3 "https://www.mouser.de/datasheet/2/445/6220xx21121-542317.pdf" H 1200 2750 50  0001 C CNN
+	1    1200 2750
+	1    0    0    -1
+$EndComp
+Text Notes 1250 2200 0    50   ~ 0
 SWD
 $Comp
 L power:GND #PWR072
 U 1 1 5B17C4C4
-P 850 2900
-F 0 "#PWR072" H 850 2650 50  0001 C CNN
-F 1 "GND" H 855 2727 50  0000 C CNN
-F 2 "" H 850 2900 50  0001 C CNN
-F 3 "" H 850 2900 50  0001 C CNN
-	1    850  2900
-	1    0    0    -1
-$EndComp
-Wire Wire Line
-	1000 2900 850  2900
-Wire Wire Line
-	850  2900 850  2700
-Wire Wire Line
-	850  2700 1000 2700
-Connection ~ 850  2900
-Wire Wire Line
-	850  2700 850  2600
-Wire Wire Line
-	850  2600 1000 2600
-Connection ~ 850  2700
-Text GLabel 1000 2500 0    50   Input ~ 0
-VDD3V3
-Wire Wire Line
-	1500 2500 1750 2500
-Wire Wire Line
-	1750 2600 1500 2600
-Wire Wire Line
-	1500 2900 1750 2900
-Wire Notes Line
-	2100 2200 2100 3150
-Wire Notes Line
-	600  3150 600  2200
-Text HLabel 1750 2900 2    50   Input ~ 0
+P 850 2950
+F 0 "#PWR072" H 850 2700 50  0001 C CNN
+F 1 "GND" H 855 2777 50  0000 C CNN
+F 2 "" H 850 2950 50  0001 C CNN
+F 3 "" H 850 2950 50  0001 C CNN
+	1    850  2950
+	1    0    0    -1
+$EndComp
+Wire Wire Line
+	1000 2950 850  2950
+Wire Wire Line
+	850  2950 850  2750
+Wire Wire Line
+	850  2750 1000 2750
+Connection ~ 850  2950
+Wire Wire Line
+	850  2750 850  2650
+Wire Wire Line
+	850  2650 1000 2650
+Connection ~ 850  2750
+Text GLabel 1000 2550 0    50   Input ~ 0
+VDD3V3
+Wire Wire Line
+	1500 2550 1750 2550
+Wire Wire Line
+	1750 2650 1500 2650
+Wire Wire Line
+	1500 2950 1750 2950
+Wire Notes Line
+	2100 2250 2100 3200
+Wire Notes Line
+	600  3200 600  2250
+Text HLabel 1750 2950 2    50   Input ~ 0
 nRESET
-Text HLabel 1750 2600 2    50   Input ~ 0
+Text HLabel 1750 2650 2    50   Input ~ 0
 SWDIO
-Text HLabel 1750 2500 2    50   Input ~ 0
+Text HLabel 1750 2550 2    50   Input ~ 0
 SWCLK
 Text Notes 650  2050 0    50   ~ 0
 ESD protected by USB isolator
 Wire Notes Line
-	600  3150 2100 3150
-Wire Notes Line
-	600  2200 2100 2200
+	600  3200 2100 3200
+Wire Notes Line
+	600  2250 2100 2250
 Text HLabel 1450 1100 2    50   Input ~ 0
 VBUS
@@
 NoConn ~ 4650 1500
 NoConn ~ 4150 1500
-NoConn ~ 1000 2800
-NoConn ~ 1500 2800
-NoConn ~ 1500 2700
+NoConn ~ 1000 2850
+NoConn ~ 1500 2850
+NoConn ~ 1500 2750
 Wire Wire Line
 	2000 5850 2000 5800
@@
 Text GLabel 8800 1600 2    50   Input ~ 0
 VDD5V
+Wire Notes Line
+	2250 2250 2250 3200
+Wire Notes Line
+	4150 3200 4150 2250
+Text Notes 2650 2200 0    50   ~ 0
+Z-Axis second connector
+$Comp
+L Connector_Generic:Conn_01x04 J16
+U 1 1 5AFD917C
+P 3500 2650
+F 0 "J16" H 3579 2642 50  0000 L CNN
+F 1 "70543-0003" H 3579 2551 50  0000 L CNN
+F 2 "custom-footprints:70543-0003" H 3500 2650 50  0001 C CNN
+F 3 "https://www.mouser.de/ProductDetail/Molex/70543-0003?qs=sGAEpiMZZMs%252bGHln7q6pm%252bS0pk2Wo0XxCD3CKlCQrmU%3d" H 3500 2650 50  0001 C CNN
+	1    3500 2650
+	1    0    0    -1
+$EndComp
+Text HLabel 2600 2550 0    50   Input ~ 0
+Z_OA1
+Text HLabel 2600 2650 0    50   Input ~ 0
+Z_OA2
+Text HLabel 2600 2850 0    50   Input ~ 0
+Z_OB2
+Text HLabel 2600 2750 0    50   Input ~ 0
+Z_OB1
+Wire Notes Line
+	2250 2250 4150 2250
+Wire Notes Line
+	2250 3200 4150 3200
+Wire Wire Line
+	2600 2550 3300 2550
+Wire Wire Line
+	2600 2650 3300 2650
+Wire Wire Line
+	2600 2750 3300 2750
+Wire Wire Line
+	2600 2850 3300 2850
 $EndSCHEMATC

Commit message: Reworked some traces for better layout.
This will also come in handy, when we add more external
connections (10 to 20pin external).
Parts:
- C42, C43, C44: symbol Device:C -> remram-rescue:C-Device
- D10, D11, D12, D13, D14, D9: symbol Device:D_Schottky -> remram-rescue:D_Schottky-Device
- J10, J11, J14, J15, J4, J5: symbol Connector_Generic:Conn_01x03 -> remram-rescue:Conn_01x03-Connector_Generic
- J12, J17, J8, J9: symbol Connector_Generic:Conn_02x05_Odd_Even -> remram-rescue:Conn_02x05_Odd_Even-Connector_Generic
- J13, J18, J19, J20, J6: symbol Connector_Generic:Conn_01x02 -> remram-rescue:Conn_01x02-Connector_Generic
- J16: symbol Connector_Generic:Conn_01x04 -> remram-rescue:Conn_01x04-Connector_Generic
- J7: symbol Connector_Specialized:USB_B -> remram-rescue:USB_B-Connector_Specialized
- R23, R24, R25, R26, R27, R28: symbol Device:R -> remram-rescue:R-Device
- TP16, TP17, TP18, TP19, TP20, TP21, TP22: symbol Connector_Specialized:Test_Point -> remram-rescue:Test_Point-Connector_Specialized
Changed lines of the file:
@@
 $EndDescr
 $Comp
-L Connector_Specialized:USB_B J7
+L remram-rescue:USB_B-Connector_Specialized J7
 U 1 1 5B16E55B
 P 1150 1300
@@
 EXT-SPI-L2C
 $Comp
-L Connector_Generic:Conn_02x05_Odd_Even J8
+L remram-rescue:Conn_02x05_Odd_Even-Connector_Generic J8
 U 1 1 5B16F6B4
 P 2700 1300
@@
 $EndComp
 $Comp
-L Connector_Generic:Conn_02x05_Odd_Even J9
+L remram-rescue:Conn_02x05_Odd_Even-Connector_Generic J9
 U 1 1 5B16F736
 P 4350 1300
@@
 $EndComp
 $Comp
-L Connector_Generic:Conn_02x05_Odd_Even J12
+L remram-rescue:Conn_02x05_Odd_Even-Connector_Generic J12
 U 1 1 5B16F775
 P 8500 1400
@@
 THERM_1
 $Comp
-L Connector_Specialized:Test_Point TP20
+L remram-rescue:Test_Point-Connector_Specialized TP20
 U 1 1 5B171985
 P 3400 4450
@@
 $EndComp
 $Comp
-L Device:D_Schottky D9
+L remram-rescue:D_Schottky-Device D9
 U 1 1 5B17198C
 P 2000 4350
@@
 $EndComp
 $Comp
-L Device:R R24
+L remram-rescue:R-Device R24
 U 1 1 5B1719A1
 P 2600 4600
@@
 $EndComp
 $Comp
-L Device:R R23
+L remram-rescue:R-Device R23
 U 1 1 5B1719A8
 P 3050 4350
@@
 	3050 4600 3050 4500
 $Comp
-L Connector_Generic:Conn_01x02 J18
+L remram-rescue:Conn_01x02-Connector_Generic J18
 U 1 1 5B1719C1
 P 4150 4600
@@
 	3400 4600 3050 4600
 $Comp
-L Device:C C42
+L remram-rescue:C-Device C42
 U 1 1 5B1719D4
 P 1250 4750
@@
 THERM_2
 $Comp
-L Connector_Specialized:Test_Point TP21
+L remram-rescue:Test_Point-Connector_Specialized TP21
 U 1 1 5B1719E6
 P 3400 5650
@@
 $EndComp
 $Comp
-L Device:R R26
+L remram-rescue:R-Device R26
 U 1 1 5B171A02
 P 2600 5800
@@
 $EndComp
 $Comp
-L Device:R R25
+L remram-rescue:R-Device R25
 U 1 1 5B171A09
 P 3050 5550
@@
 	3050 5800 3050 5700
 $Comp
-L Connector_Generic:Conn_01x02 J19
+L remram-rescue:Conn_01x02-Connector_Generic J19
 U 1 1 5B171A22
 P 4150 5800
@@
 	3400 5800 3050 5800
 $Comp
-L Device:C C43
+L remram-rescue:C-Device C43
 U 1 1 5B171A35
 P 1250 5950
@@
 THERM_3
 $Comp
-L Connector_Specialized:Test_Point TP22
+L remram-rescue:Test_Point-Connector_Specialized TP22
 U 1 1 5B171A47
 P 3400 6850
@@
 $EndComp
 $Comp
-L Device:R R28
+L remram-rescue:R-Device R28
 U 1 1 5B171A63
 P 2600 7000
@@
 $EndComp
 $Comp
-L Device:R R27
+L remram-rescue:R-Device R27
 U 1 1 5B171A6A
 P 3050 6750
@@
 	3050 7000 3050 6900
 $Comp
-L Connector_Generic:Conn_01x02 J20
+L remram-rescue:Conn_01x02-Connector_Generic J20
 U 1 1 5B171A83
 P 4150 7000
@@
 	3400 7000 3050 7000
 $Comp
-L Device:C C44
+L remram-rescue:C-Device C44
 U 1 1 5B171A96
 P 1250 7150
@@
 	5150 750  7650 750
 $Comp
-L Connector_Generic:Conn_01x03 J4
+L remram-rescue:Conn_01x03-Connector_Generic J4
 U 1 1 5B171AB8
 P 5750 950
@@
 VDD3V3
 $Comp
-L Connector_Generic:Conn_01x03 J5
+L remram-rescue:Conn_01x03-Connector_Generic J5
 U 1 1 5B171AC6
 P 6950 950
@@
 VDD3V3
 $Comp
-L Connector_Generic:Conn_01x03 J10
+L remram-rescue:Conn_01x03-Connector_Generic J10
 U 1 1 5B171AD6
 P 5750 1350
@@
 VDD3V3
 $Comp
-L Connector_Generic:Conn_01x03 J11
+L remram-rescue:Conn_01x03-Connector_Generic J11
 U 1 1 5B171AE4
 P 6950 1350
@@
 VDD3V3
 $Comp
-L Connector_Generic:Conn_01x03 J14
+L remram-rescue:Conn_01x03-Connector_Generic J14
 U 1 1 5B171AF4
 P 5750 1750
@@
 VDD3V3
 $Comp
-L Connector_Generic:Conn_01x03 J15
+L remram-rescue:Conn_01x03-Connector_Generic J15
 U 1 1 5B171B02
 P 6950 1750
@@
 	7650 2100 5150 2100
 $Comp
-L Connector_Generic:Conn_02x05_Odd_Even J17
+L remram-rescue:Conn_02x05_Odd_Even-Connector_Generic J17
 U 1 1 5B17C4BC
 P 1200 2750
@@
 	1250 7000 2000 7000
 $Comp
-L Device:D_Schottky D10
+L remram-rescue:D_Schottky-Device D10
 U 1 1 5AFA7311
 P 2000 4850
@@
 $EndComp
 $Comp
-L Device:D_Schottky D11
+L remram-rescue:D_Schottky-Device D11
 U 1 1 5AFA961C
 P 2000 5550
@@
 $EndComp
 $Comp
-L Device:D_Schottky D12
+L remram-rescue:D_Schottky-Device D12
 U 1 1 5AFAB94C
 P 2000 6000
@@
 $EndComp
 $Comp
-L Device:D_Schottky D13
+L remram-rescue:D_Schottky-Device D13
 U 1 1 5AFADC4D
 P 2000 6750
@@
 $EndComp
 $Comp
-L Device:D_Schottky D14
+L remram-rescue:D_Schottky-Device D14
 U 1 1 5AFAFF57
 P 2000 7200
@@
 $EndComp
 $Comp
-L Connector_Generic:Conn_01x02 J6
+L remram-rescue:Conn_01x02-Connector_Generic J6
 U 1 1 5AFC19C7
 P 10300 1050
@@
 VDD_PWR
 $Comp
-L Connector_Generic:Conn_01x02 J13
+L remram-rescue:Conn_01x02-Connector_Generic J13
 U 1 1 5AFDD4E7
 P 10300 1700
@@
 	9400 750  10900 750
 $Comp
-L Connector_Specialized:Test_Point TP16
+L remram-rescue:Test_Point-Connector_Specialized TP16
 U 1 1 5AFF4AC9
 P 9750 950
@@
 $EndComp
 $Comp
-L Connector_Specialized:Test_Point TP18
+L remram-rescue:Test_Point-Connector_Specialized TP18
 U 1 1 5AFFF980
 P 9750 1550
@@
 	9850 1800 10050 1800
 $Comp
-L Connector_Specialized:Test_Point TP19
+L remram-rescue:Test_Point-Connector_Specialized TP19
 U 1 1 5B00F821
 P 10150 1550
@@
 	10050 1800 10100 1800
 $Comp
-L Connector_Specialized:Test_Point TP17
+L remram-rescue:Test_Point-Connector_Specialized TP17
 U 1 1 5B068C7B
 P 10150 950
@@
 Z-Axis second connector
 $Comp
-L Connector_Generic:Conn_01x04 J16
+L remram-rescue:Conn_01x04-Connector_Generic J16
 U 1 1 5AFD917C
 P 3500 2650

Commit message: Reworked some traces and labels.
Parts:
- renumbered J20 to J10, J9 to J11, J4 to J12, J10 to J13, J5 to J15, J11 to J16, J15 to J17, J12 to J18, J6 to J19, J13 to J20, J7 to J4, J17 to J5, J8 to J6, J16 to J7, J18 to J8, J19 to J9, R24 to R23, R26 to R24, R28 to R25, R23 to R26, R25 to R27, R27 to R28, TP20 to TP15, TP21 to TP16, TP22 to TP17, TP16 to TP18, TP18 to TP19, TP17 to TP20, TP19 to TP21

Commit message: First draft of RemRam.
I added a 20 pin expansion connector with the following pins:
 - SPI
 - I2C
 - USART
 - 4x PWM
 - 4x GPIO
Parts:
- removed J18: 61201021621, custom-footprints:Box_Header_2x05x2.54mm_Straight, symbol remram-rescue:Conn_02x05_Odd_Even-Connector_Generic
- added J12: Conn_02x10, Connector_PinHeader_2.54mm:PinHeader_2x10_P2.54mm_Vertical, symbol Connector_Generic:Conn_02x10_Odd_Even
- J8: renamed from J6; value 61201021621 -> Conn_02x05
- J9: renamed from J11; value 61201021621 -> Conn_02x05
- renumbered J13 to J10, J16 to J11, J20 to J13, J17 to J15, J7 to J16, J5 to J17, J8 to J18, J9 to J19, J10 to J20, J12 to J4, J15 to J5, J19 to J6, J4 to J7, R26 to R23, R23 to R24, R27 to R25, R24 to R26, R28 to R27, R25 to R28, TP18 to TP15, TP20 to TP16, TP19 to TP17, TP21 to TP18, TP15 to TP19, TP16 to TP20, TP17 to TP21
Connections:
- net labels added: EXT_D3, EXT_D4, PWM_EXT1, PWM_EXT2, PWM_EXT3, PWM_EXT4, USART_CK, USART_RX, USART_TX
Other:
- note added: "EXT1"
- note added: "EXT2"
- note added: "EXT3"
- note removed: "EXT-LCD"
- note removed: "EXT-SD"
- note removed: "EXT-SPI-L2C"

Commit message: v0.2 of PCB.
After some feedback, we changed following:
 - Switched FAN VDD from 24 to 5V.
 - FAN now have a ADC pin for speed sensing.
 - Expanded EXP-3 connector to 26 pin
   - Included 24V VDD.
   - Could be used to connect up to two
     extra stepper.
 - Removed GND connections on TMC2130 to
   middel GND plane.
Parts:
- removed J12: Conn_02x10, Connector_PinHeader_2.54mm:PinHeader_2x10_P2.54mm_Vertical, symbol Connector_Generic:Conn_02x10_Odd_Even
- removed J13, J6: 70543-0001, custom-footprints:70543-0001, symbol remram-rescue:Conn_01x02-Connector_Generic
- added J12: Conn_02x13_Odd_Even, Connector_PinHeader_2.54mm:PinHeader_2x13_P2.54mm_Vertical, symbol Connector_Generic:Conn_02x13_Odd_Even
- added J15, J6: 70543-0002, custom-footprints:70543-0002, symbol remram-rescue:Conn_01x03-Connector_Generic
- added TP19: FAN1-, TestPoint:TestPoint_Pad_D1.0mm, symbol remram-rescue:Test_Point-Connector_Specialized
- added TP20: FAN1S, TestPoint:TestPoint_Pad_D1.0mm, symbol remram-rescue:Test_Point-Connector_Specialized
- TP17: value FAN2+ -> FAN1S
- TP18: value FAN2- -> FAN1+
- renumbered J14 to J13, J15 to J14, TP19 to TP21, TP20 to TP22, TP21 to TP23
Connections:
- net labels added: FAN_SPEED1, FAN_SPEED2
- wire segments 71 -> 79
