File: PCB/connectors.sch (KiCad schematic (older format))
At the start: 41 parts, among them J10 70543-0002, J11 70543-0002, J12 Conn_02x13_Odd_Even, J13 70543-0002, J14 70543-0002, J15 70543-0002, J16 70543-0003, J17 62201021121, J18 70543-0001, J19 70543-0001, J20 70543-0001, J4 70543-0002, J5 70543-0002, J6 70543-0002, J7 67068-8000, J8 Conn_02x05, J9 Conn_02x05

Commit message: Version 0.3.
Parts:
- renumbered C42 to C43, C43 to C44, C44 to C45
Changed lines of the file:
@@
 	3050 4600 2750 4600
 $Comp
-L power:GND #PWR078
+L power:GND #PWR079
 U 1 1 5B1719B0
 P 2000 5000
-F 0 "#PWR078" H 2000 4750 50  0001 C CNN
+F 0 "#PWR079" H 2000 4750 50  0001 C CNN
 F 1 "GND" H 2005 4827 50  0000 C CNN
 F 2 "" H 2000 5000 50  0001 C CNN
@@
 Connection ~ 3050 4600
 $Comp
-L power:GND #PWR076
+L power:GND #PWR077
 U 1 1 5B1719CA
 P 3950 4700
-F 0 "#PWR076" H 3950 4450 50  0001 C CNN
+F 0 "#PWR077" H 3950 4450 50  0001 C CNN
 F 1 "GND" H 3955 4527 50  0000 C CNN
 F 2 "" H 3950 4700 50  0001 C CNN
@@
 	3400 4600 3050 4600
 $Comp
-L remram-rescue:C-Device C42
+L remram-rescue:C-Device C43
 U 1 1 5B1719D4
 P 1250 4750
-F 0 "C42" H 1365 4796 50  0000 L CNN
+F 0 "C43" H 1365 4796 50  0000 L CNN
 F 1 "100nF" H 1365 4705 50  0000 L CNN
 F 2 "Capacitor_SMD:C_0603_1608Metric" H 1288 4600 50  0001 C CNN
@@
 Connection ~ 1250 4600
 $Comp
-L power:GND #PWR077
+L power:GND #PWR078
 U 1 1 5B1719DF
 P 1250 4900
-F 0 "#PWR077" H 1250 4650 50  0001 C CNN
+F 0 "#PWR078" H 1250 4650 50  0001 C CNN
 F 1 "GND" H 1255 4727 50  0000 C CNN
 F 2 "" H 1250 4900 50  0001 C CNN
@@
 	3050 5800 2750 5800
 $Comp
-L power:GND #PWR081
+L power:GND #PWR082
 U 1 1 5B171A11
 P 2000 6150
-F 0 "#PWR081" H 2000 5900 50  0001 C CNN
+F 0 "#PWR082" H 2000 5900 50  0001 C CNN
 F 1 "GND" H 2005 5977 50  0000 C CNN
 F 2 "" H 2000 6150 50  0001 C CNN
@@
 Connection ~ 3050 5800
 $Comp
-L power:GND #PWR079
+L power:GND #PWR080
 U 1 1 5B171A2B
 P 3950 5900
-F 0 "#PWR079" H 3950 5650 50  0001 C CNN
+F 0 "#PWR080" H 3950 5650 50  0001 C CNN
 F 1 "GND" H 3955 5727 50  0000 C CNN
 F 2 "" H 3950 5900 50  0001 C CNN
@@
 	3400 5800 3050 5800
 $Comp
-L remram-rescue:C-Device C43
+L remram-rescue:C-Device C44
 U 1 1 5B171A35
 P 1250 5950
-F 0 "C43" H 1365 5996 50  0000 L CNN
+F 0 "C44" H 1365 5996 50  0000 L CNN
 F 1 "100nF" H 1365 5905 50  0000 L CNN
 F 2 "Capacitor_SMD:C_0603_1608Metric" H 1288 5800 50  0001 C CNN
@@
 Connection ~ 1250 5800
 $Comp
-L power:GND #PWR080
+L power:GND #PWR081
 U 1 1 5B171A40
 P 1250 6100
-F 0 "#PWR080" H 1250 5850 50  0001 C CNN
+F 0 "#PWR081" H 1250 5850 50  0001 C CNN
 F 1 "GND" H 1255 5927 50  0000 C CNN
 F 2 "" H 1250 6100 50  0001 C CNN
@@
 	3050 7000 2750 7000
 $Comp
-L power:GND #PWR084
+L power:GND #PWR085
 U 1 1 5B171A72
 P 2000 7350
-F 0 "#PWR084" H 2000 7100 50  0001 C CNN
+F 0 "#PWR085" H 2000 7100 50  0001 C CNN
 F 1 "GND" H 2005 7177 50  0000 C CNN
 F 2 "" H 2000 7350 50  0001 C CNN
@@
 Connection ~ 3050 7000
 $Comp
-L power:GND #PWR082
+L power:GND #PWR083
 U 1 1 5B171A8C
 P 3950 7100
-F 0 "#PWR082" H 3950 6850 50  0001 C CNN
+F 0 "#PWR083" H 3950 6850 50  0001 C CNN
 F 1 "GND" H 3955 6927 50  0000 C CNN
 F 2 "" H 3950 7100 50  0001 C CNN
@@
 	3400 7000 3050 7000
 $Comp
-L remram-rescue:C-Device C44
+L remram-rescue:C-Device C45
 U 1 1 5B171A96
 P 1250 7150
-F 0 "C44" H 1365 7196 50  0000 L CNN
+F 0 "C45" H 1365 7196 50  0000 L CNN
 F 1 "100nF" H 1365 7105 50  0000 L CNN
 F 2 "Capacitor_SMD:C_0603_1608Metric" H 1288 7000 50  0001 C CNN
@@
 Connection ~ 1250 7000
 $Comp
-L power:GND #PWR083
+L power:GND #PWR084
 U 1 1 5B171AA1
 P 1250 7300
-F 0 "#PWR083" H 1250 7050 50  0001 C CNN
+F 0 "#PWR084" H 1250 7050 50  0001 C CNN
 F 1 "GND" H 1255 7127 50  0000 C CNN
 F 2 "" H 1250 7300 50  0001 C CNN
@@
 Endstops
 $Comp
-L power:GND #PWR063
+L power:GND #PWR064
 U 1 1 5B171AAF
 P 5550 950
-F 0 "#PWR063" H 5550 700 50  0001 C CNN
+F 0 "#PWR064" H 5550 700 50  0001 C CNN
 F 1 "GND" V 5555 822 50  0000 R CNN
 F 2 "" H 5550 950 50  0001 C CNN
@@
 $EndComp
 $Comp
-L power:GND #PWR064
+L power:GND #PWR065
 U 1 1 5B171ABF
 P 6750 950
-F 0 "#PWR064" H 6750 700 50  0001 C CNN
+F 0 "#PWR065" H 6750 700 50  0001 C CNN
 F 1 "GND" V 6755 822 50  0000 R CNN
 F 2 "" H 6750 950 50  0001 C CNN
@@
 $EndComp
 $Comp
-L power:GND #PWR067
+L power:GND #PWR066
 U 1 1 5B171ACF
 P 5550 1350
-F 0 "#PWR067" H 5550 1100 50  0001 C CNN
+F 0 "#PWR066" H 5550 1100 50  0001 C CNN
 F 1 "GND" V 5555 1222 50  0000 R CNN
 F 2 "" H 5550 1350 50  0001 C CNN
@@
 $EndComp
 $Comp
-L power:GND #PWR068
+L power:GND #PWR067
 U 1 1 5B171ADD
 P 6750 1350
-F 0 "#PWR068" H 6750 1100 50  0001 C CNN
+F 0 "#PWR067" H 6750 1100 50  0001 C CNN
 F 1 "GND" V 6755 1222 50  0000 R CNN
 F 2 "" H 6750 1350 50  0001 C CNN
@@
 $EndComp
 $Comp
-L power:GND #PWR071
+L power:GND #PWR070
 U 1 1 5B171AED
 P 5550 1750
-F 0 "#PWR071" H 5550 1500 50  0001 C CNN
+F 0 "#PWR070" H 5550 1500 50  0001 C CNN
 F 1 "GND" V 5555 1622 50  0000 R CNN
 F 2 "" H 5550 1750 50  0001 C CNN
@@
 $EndComp
 $Comp
-L power:GND #PWR072
+L power:GND #PWR071
 U 1 1 5B171AFB
 P 6750 1750
-F 0 "#PWR072" H 6750 1500 50  0001 C CNN
+F 0 "#PWR071" H 6750 1500 50  0001 C CNN
 F 1 "GND" V 6755 1622 50  0000 R CNN
 F 2 "" H 6750 1750 50  0001 C CNN
@@
 SWD
 $Comp
-L power:GND #PWR075
+L power:GND #PWR076
 U 1 1 5B17C4C4
 P 850 2950
-F 0 "#PWR075" H 850 2700 50  0001 C CNN
+F 0 "#PWR076" H 850 2700 50  0001 C CNN
 F 1 "GND" H 855 2777 50  0000 C CNN
 F 2 "" H 850 2950 50  0001 C CNN
@@
 VBUS
 $Comp
-L power:GNDS #PWR070
+L power:GNDS #PWR069
 U 1 1 5AF8309F
 P 1150 1700
-F 0 "#PWR070" H 1150 1450 50  0001 C CNN
+F 0 "#PWR069" H 1150 1450 50  0001 C CNN
 F 1 "GNDS" H 1155 1527 50  0000 C CNN
 F 2 "" H 1150 1700 50  0001 C CNN
@@
 VDD5V
 $Comp
-L power:GND #PWR069
+L power:GND #PWR068
 U 1 1 5AFA04BE
 P 2500 1500
-F 0 "#PWR069" H 2500 1250 50  0001 C CNN
+F 0 "#PWR068" H 2500 1250 50  0001 C CNN
 F 1 "GND" V 2505 1372 50  0000 R CNN
 F 2 "" H 2500 1500 50  0001 C CNN
@@
 VDD3V3
 $Comp
-L power:GND #PWR073
+L power:GND #PWR074
 U 1 1 5B067CCF
 P 8300 2250
-F 0 "#PWR073" H 8300 2000 50  0001 C CNN
+F 0 "#PWR074" H 8300 2000 50  0001 C CNN
 F 1 "GND" V 8305 2122 50  0000 R CNN
 F 2 "" H 8300 2250 50  0001 C CNN
@@
 	9350 2350 7700 2350
 $Comp
-L power:GND #PWR074
+L power:GND #PWR075
 U 1 1 5B009A39
 P 8800 2250
-F 0 "#PWR074" H 8800 2000 50  0001 C CNN
+F 0 "#PWR075" H 8800 2000 50  0001 C CNN
 F 1 "GND" V 8805 2122 50  0000 R CNN
 F 2 "" H 8800 2250 50  0001 C CNN
@@
 VDD5V
 $Comp
-L power:GND #PWR0124
+L power:GND #PWR073
 U 1 1 5B089613
 P 8800 1950
-F 0 "#PWR0124" H 8800 1700 50  0001 C CNN
+F 0 "#PWR073" H 8800 1700 50  0001 C CNN
 F 1 "GND" V 8805 1822 50  0000 R CNN
 F 2 "" H 8800 1950 50  0001 C CNN
@@
 $EndComp
 $Comp
-L power:GND #PWR0125
+L power:GND #PWR072
 U 1 1 5B08B3F7
 P 8300 1950
-F 0 "#PWR0125" H 8300 1700 50  0001 C CNN
+F 0 "#PWR072" H 8300 1700 50  0001 C CNN
 F 1 "GND" V 8305 1822 50  0000 R CNN
 F 2 "" H 8300 1950 50  0001 C CNN
