File: PCB/connectors.sch (KiCad schematic (older format))
At the start: 41 parts, among them J10 70543-0002, J11 70543-0002, J12 Conn_02x13_Odd_Even, J13 70543-0002, J14 70543-0002, J15 70543-0002, J16 70543-0003, J17 62201021121, J18 70543-0001, J19 70543-0001, J20 70543-0001, J4 70543-0002, J5 70543-0002, J6 70543-0002, J7 67068-8000, J8 Conn_02x05, J9 Conn_02x05

Commit message: Changed ordering of parts. Version 0.4.
Parts:
- renumbered C43 to C34, C44 to C35, C45 to C36, D9 to D10, D10 to D11, D11 to D12, D12 to D13, D13 to D14, D14 to D15, J11 to J10, J12 to J11, J13 to J12, J14 to J13, J15 to J14, J16 to J15, J17 to J16, J18 to J17, J19 to J18, J20 to J19, J4 to J3, J5 to J4, J6 to J5, J7 to J6, J8 to J7, J9 to J8, J10 to J9, R23 to R21, R24 to R22, R25 to R23, R26 to R24, R27 to R25, R28 to R26, TP15 to TP11, TP16 to TP12, TP17 to TP13, TP18 to TP14, TP19 to TP15, TP20 to TP16, TP21 to TP17, TP22 to TP18, TP23 to TP19

Commit message: Removed USART1 CK pin and added another digial pin.
STM32duino doesn't seem to support USART. So I will only
implement the UART pins.
Connections:
- net labels added: EXT_D5
- net labels removed: USART_CK
Other:
- note added: "TODO:\n - STM32duino doesn't use CK pin of USART"
Changed lines of the file:
@@
 $Descr A4 11693 8268
 encoding utf-8
-Sheet 6 9
+Sheet 5 9
 Title "Connectors"
 Date ""
@@
 Text HLabel 8300 1250 0    50   Input ~ 0
 EXT_D2
-Text HLabel 8300 1450 0    50   Input ~ 0
+Text HLabel 8800 1450 2    50   Input ~ 0
 SCL
-Text HLabel 8800 1350 2    50   BiDi ~ 0
+Text HLabel 8300 1450 0    50   BiDi ~ 0
 SDA
 Wire Notes Line
@@
 Text HLabel 8800 1750 2    50   Input ~ 0
 USART_RX
-Text HLabel 8800 1650 2    50   Input ~ 0
-USART_CK
-Text HLabel 8800 1450 2    50   Input ~ 0
+Text HLabel 8300 1550 0    50   Input ~ 0
 PWM_EXT1
-Text HLabel 8300 1550 0    50   Input ~ 0
+Text HLabel 8800 1550 2    50   Input ~ 0
 PWM_EXT2
 Text HLabel 8800 1250 2    50   Input ~ 0
@@
 Text HLabel 8300 1350 0    50   Input ~ 0
 EXT_D4
-Text HLabel 8800 1550 2    50   Input ~ 0
+Text HLabel 8300 1650 0    50   Input ~ 0
 PWM_EXT3
-Text HLabel 8300 1650 0    50   Input ~ 0
+Text HLabel 8800 1650 2    50   Input ~ 0
 PWM_EXT4
 $Comp
@@
 	0    1    1    0
 $EndComp
+Text Notes 7650 2600 0    50   ~ 0
+TODO:\n - STM32duino doesn't use CK pin of USART
+Text HLabel 8800 1350 2    50   Input ~ 0
+EXT_D5
 $EndSCHEMATC

Commit message: Added a battery for SRAM backup.
Parts:
- renumbered C34 to C33, C35 to C34, C36 to C35
Changed lines of the file:
@@
 	3050 4600 2750 4600
 $Comp
-L power:GND #PWR067
+L power:GND #PWR068
 U 1 1 5B1719B0
 P 2000 5000
-F 0 "#PWR067" H 2000 4750 50  0001 C CNN
+F 0 "#PWR068" H 2000 4750 50  0001 C CNN
 F 1 "GND" H 2005 4827 50  0000 C CNN
 F 2 "" H 2000 5000 50  0001 C CNN
@@
 Connection ~ 3050 4600
 $Comp
-L power:GND #PWR065
+L power:GND #PWR066
 U 1 1 5B1719CA
 P 3950 4700
-F 0 "#PWR065" H 3950 4450 50  0001 C CNN
+F 0 "#PWR066" H 3950 4450 50  0001 C CNN
 F 1 "GND" H 3955 4527 50  0000 C CNN
 F 2 "" H 3950 4700 50  0001 C CNN
@@
 	3400 4600 3050 4600
 $Comp
-L remram-rescue:C-Device C34
+L remram-rescue:C-Device C33
 U 1 1 5B1719D4
 P 1250 4750
-F 0 "C34" H 1365 4796 50  0000 L CNN
+F 0 "C33" H 1365 4796 50  0000 L CNN
 F 1 "100nF" H 1365 4705 50  0000 L CNN
 F 2 "Capacitor_SMD:C_0603_1608Metric" H 1288 4600 50  0001 C CNN
@@
 Connection ~ 1250 4600
 $Comp
-L power:GND #PWR066
+L power:GND #PWR067
 U 1 1 5B1719DF
 P 1250 4900
-F 0 "#PWR066" H 1250 4650 50  0001 C CNN
+F 0 "#PWR067" H 1250 4650 50  0001 C CNN
 F 1 "GND" H 1255 4727 50  0000 C CNN
 F 2 "" H 1250 4900 50  0001 C CNN
@@
 	3050 5800 2750 5800
 $Comp
-L power:GND #PWR070
+L power:GND #PWR071
 U 1 1 5B171A11
 P 2000 6150
-F 0 "#PWR070" H 2000 5900 50  0001 C CNN
+F 0 "#PWR071" H 2000 5900 50  0001 C CNN
 F 1 "GND" H 2005 5977 50  0000 C CNN
 F 2 "" H 2000 6150 50  0001 C CNN
@@
 Connection ~ 3050 5800
 $Comp
-L power:GND #PWR068
+L power:GND #PWR069
 U 1 1 5B171A2B
 P 3950 5900
-F 0 "#PWR068" H 3950 5650 50  0001 C CNN
+F 0 "#PWR069" H 3950 5650 50  0001 C CNN
 F 1 "GND" H 3955 5727 50  0000 C CNN
 F 2 "" H 3950 5900 50  0001 C CNN
@@
 	3400 5800 3050 5800
 $Comp
-L remram-rescue:C-Device C35
+L remram-rescue:C-Device C34
 U 1 1 5B171A35
 P 1250 5950
-F 0 "C35" H 1365 5996 50  0000 L CNN
+F 0 "C34" H 1365 5996 50  0000 L CNN
 F 1 "100nF" H 1365 5905 50  0000 L CNN
 F 2 "Capacitor_SMD:C_0603_1608Metric" H 1288 5800 50  0001 C CNN
@@
 Connection ~ 1250 5800
 $Comp
-L power:GND #PWR069
+L power:GND #PWR070
 U 1 1 5B171A40
 P 1250 6100
-F 0 "#PWR069" H 1250 5850 50  0001 C CNN
+F 0 "#PWR070" H 1250 5850 50  0001 C CNN
 F 1 "GND" H 1255 5927 50  0000 C CNN
 F 2 "" H 1250 6100 50  0001 C CNN
@@
 	3050 7000 2750 7000
 $Comp
-L power:GND #PWR073
+L power:GND #PWR074
 U 1 1 5B171A72
 P 2000 7350
-F 0 "#PWR073" H 2000 7100 50  0001 C CNN
+F 0 "#PWR074" H 2000 7100 50  0001 C CNN
 F 1 "GND" H 2005 7177 50  0000 C CNN
 F 2 "" H 2000 7350 50  0001 C CNN
@@
 Connection ~ 3050 7000
 $Comp
-L power:GND #PWR071
+L power:GND #PWR072
 U 1 1 5B171A8C
 P 3950 7100
-F 0 "#PWR071" H 3950 6850 50  0001 C CNN
+F 0 "#PWR072" H 3950 6850 50  0001 C CNN
 F 1 "GND" H 3955 6927 50  0000 C CNN
 F 2 "" H 3950 7100 50  0001 C CNN
@@
 	3400 7000 3050 7000
 $Comp
-L remram-rescue:C-Device C36
+L remram-rescue:C-Device C35
 U 1 1 5B171A96
 P 1250 7150
-F 0 "C36" H 1365 7196 50  0000 L CNN
+F 0 "C35" H 1365 7196 50  0000 L CNN
 F 1 "100nF" H 1365 7105 50  0000 L CNN
 F 2 "Capacitor_SMD:C_0603_1608Metric" H 1288 7000 50  0001 C CNN
@@
 Connection ~ 1250 7000
 $Comp
-L power:GND #PWR072
+L power:GND #PWR073
 U 1 1 5B171AA1
 P 1250 7300
-F 0 "#PWR072" H 1250 7050 50  0001 C CNN
+F 0 "#PWR073" H 1250 7050 50  0001 C CNN
 F 1 "GND" H 1255 7127 50  0000 C CNN
 F 2 "" H 1250 7300 50  0001 C CNN
@@
 Endstops
 $Comp
-L power:GND #PWR052
+L power:GND #PWR053
 U 1 1 5B171AAF
 P 5550 950
-F 0 "#PWR052" H 5550 700 50  0001 C CNN
+F 0 "#PWR053" H 5550 700 50  0001 C CNN
 F 1 "GND" V 5555 822 50  0000 R CNN
 F 2 "" H 5550 950 50  0001 C CNN
@@
 $EndComp
 $Comp
-L power:GND #PWR053
+L power:GND #PWR054
 U 1 1 5B171ABF
 P 6750 950
-F 0 "#PWR053" H 6750 700 50  0001 C CNN
+F 0 "#PWR054" H 6750 700 50  0001 C CNN
 F 1 "GND" V 6755 822 50  0000 R CNN
 F 2 "" H 6750 950 50  0001 C CNN
@@
 $EndComp
 $Comp
-L power:GND #PWR054
+L power:GND #PWR055
 U 1 1 5B171ACF
 P 5550 1350
-F 0 "#PWR054" H 5550 1100 50  0001 C CNN
+F 0 "#PWR055" H 5550 1100 50  0001 C CNN
 F 1 "GND" V 5555 1222 50  0000 R CNN
 F 2 "" H 5550 1350 50  0001 C CNN
@@
 $EndComp
 $Comp
-L power:GND #PWR055
+L power:GND #PWR056
 U 1 1 5B171ADD
 P 6750 1350
-F 0 "#PWR055" H 6750 1100 50  0001 C CNN
+F 0 "#PWR056" H 6750 1100 50  0001 C CNN
 F 1 "GND" V 6755 1222 50  0000 R CNN
 F 2 "" H 6750 1350 50  0001 C CNN
@@
 $EndComp
 $Comp
-L power:GND #PWR058
+L power:GND #PWR059
 U 1 1 5B171AED
 P 5550 1750
-F 0 "#PWR058" H 5550 1500 50  0001 C CNN
+F 0 "#PWR059" H 5550 1500 50  0001 C CNN
 F 1 "GND" V 5555 1622 50  0000 R CNN
 F 2 "" H 5550 1750 50  0001 C CNN
@@
 $EndComp
 $Comp
-L power:GND #PWR059
+L power:GND #PWR060
 U 1 1 5B171AFB
 P 6750 1750
-F 0 "#PWR059" H 6750 1500 50  0001 C CNN
+F 0 "#PWR060" H 6750 1500 50  0001 C CNN
 F 1 "GND" V 6755 1622 50  0000 R CNN
 F 2 "" H 6750 1750 50  0001 C CNN
@@
 SWD
 $Comp
-L power:GND #PWR064
+L power:GND #PWR065
 U 1 1 5B17C4C4
 P 850 2950
-F 0 "#PWR064" H 850 2700 50  0001 C CNN
+F 0 "#PWR065" H 850 2700 50  0001 C CNN
 F 1 "GND" H 855 2777 50  0000 C CNN
 F 2 "" H 850 2950 50  0001 C CNN
@@
 VBUS
 $Comp
-L power:GNDS #PWR057
+L power:GNDS #PWR058
 U 1 1 5AF8309F
 P 1150 1700
-F 0 "#PWR057" H 1150 1450 50  0001 C CNN
+F 0 "#PWR058" H 1150 1450 50  0001 C CNN
 F 1 "GNDS" H 1155 1527 50  0000 C CNN
 F 2 "" H 1150 1700 50  0001 C CNN
@@
 VDD5V
 $Comp
-L power:GND #PWR056
+L power:GND #PWR057
 U 1 1 5AFA04BE
 P 2500 1500
-F 0 "#PWR056" H 2500 1250 50  0001 C CNN
+F 0 "#PWR057" H 2500 1250 50  0001 C CNN
 F 1 "GND" V 2505 1372 50  0000 R CNN
 F 2 "" H 2500 1500 50  0001 C CNN
@@
 VDD3V3
 $Comp
-L power:GND #PWR062
+L power:GND #PWR063
 U 1 1 5B067CCF
 P 8300 2250
-F 0 "#PWR062" H 8300 2000 50  0001 C CNN
+F 0 "#PWR063" H 8300 2000 50  0001 C CNN
 F 1 "GND" V 8305 2122 50  0000 R CNN
 F 2 "" H 8300 2250 50  0001 C CNN
@@
 	9350 2350 7700 2350
 $Comp
-L power:GND #PWR063
+L power:GND #PWR064
 U 1 1 5B009A39
 P 8800 2250
-F 0 "#PWR063" H 8800 2000 50  0001 C CNN
+F 0 "#PWR064" H 8800 2000 50  0001 C CNN
 F 1 "GND" V 8805 2122 50  0000 R CNN
 F 2 "" H 8800 2250 50  0001 C CNN
@@
 VDD5V
 $Comp
-L power:GND #PWR061
+L power:GND #PWR062
 U 1 1 5B089613
 P 8800 1950
-F 0 "#PWR061" H 8800 1700 50  0001 C CNN
+F 0 "#PWR062" H 8800 1700 50  0001 C CNN
 F 1 "GND" V 8805 1822 50  0000 R CNN
 F 2 "" H 8800 1950 50  0001 C CNN
@@
 $EndComp
 $Comp
-L power:GND #PWR060
+L power:GND #PWR061
 U 1 1 5B08B3F7
 P 8300 1950
-F 0 "#PWR060" H 8300 1700 50  0001 C CNN
+F 0 "#PWR061" H 8300 1700 50  0001 C CNN
 F 1 "GND" V 8305 1822 50  0000 R CNN
 F 2 "" H 8300 1950 50  0001 C CNN

Commit message: Final version that goes to the lab.
Parts:
- J16: footprint Connector_PinHeader_1.27mm:PinHeader_2x05_P1.27mm_Vertical -> custom-footprints:PinHeader_2x05_P1.27mm_Vertical
Changed lines of the file:
@@
 F 0 "J16" H 1250 3200 50  0000 C CNN
 F 1 "62201021121" H 1250 3100 50  0000 C CNN
-F 2 "Connector_PinHeader_1.27mm:PinHeader_2x05_P1.27mm_Vertical" H 1200 2750 50  0001 C CNN
+F 2 "custom-footprints:PinHeader_2x05_P1.27mm_Vertical" H 1200 2750 50  0001 C CNN
 F 3 "https://www.mouser.de/datasheet/2/445/6220xx21121-542317.pdf" H 1200 2750 50  0001 C CNN
 	1    1200 2750

Commit message: Remove an old TODO
Other:
- note removed: "TODO:\n - STM32duino doesn't use CK pin of USART"
Changed lines of the file:
@@
 	0    1    1    0
 $EndComp
-Text Notes 7650 2600 0    50   ~ 0
-TODO:\n - STM32duino doesn't use CK pin of USART
 Text HLabel 8800 1350 2    50   Input ~ 0
 EXT_D5

Commit message: Change DC-DC layout
The ripple on the 5V and 3V3 rail was too high (360mV).

In an attempt to reduce the RF and HF noise, I changed the layout
to a more compact one. I also added a third 22uF output capacitor
behind the inductor to lower ESR. I also added a 100nf input
capacitor to combat HF noise, as recommended in the datasheet.

The BOM needs to be updated in such a way, that we specificly
choose low ESR resistors.
Parts:
- renumbered C33 to C34, C34 to C35, C35 to C36
Changed lines of the file:
@@
 	3050 4600 2750 4600
 $Comp
-L power:GND #PWR068
+L power:GND #PWR069
 U 1 1 5B1719B0
 P 2000 5000
-F 0 "#PWR068" H 2000 4750 50  0001 C CNN
+F 0 "#PWR069" H 2000 4750 50  0001 C CNN
 F 1 "GND" H 2005 4827 50  0000 C CNN
 F 2 "" H 2000 5000 50  0001 C CNN
@@
 Connection ~ 3050 4600
 $Comp
-L power:GND #PWR066
+L power:GND #PWR067
 U 1 1 5B1719CA
 P 3950 4700
-F 0 "#PWR066" H 3950 4450 50  0001 C CNN
+F 0 "#PWR067" H 3950 4450 50  0001 C CNN
 F 1 "GND" H 3955 4527 50  0000 C CNN
 F 2 "" H 3950 4700 50  0001 C CNN
@@
 	3400 4600 3050 4600
 $Comp
-L remram-rescue:C-Device C33
+L remram-rescue:C-Device C34
 U 1 1 5B1719D4
 P 1250 4750
-F 0 "C33" H 1365 4796 50  0000 L CNN
+F 0 "C34" H 1365 4796 50  0000 L CNN
 F 1 "100nF" H 1365 4705 50  0000 L CNN
 F 2 "Capacitor_SMD:C_0603_1608Metric" H 1288 4600 50  0001 C CNN
@@
 Connection ~ 1250 4600
 $Comp
-L power:GND #PWR067
+L power:GND #PWR068
 U 1 1 5B1719DF
 P 1250 4900
-F 0 "#PWR067" H 1250 4650 50  0001 C CNN
+F 0 "#PWR068" H 1250 4650 50  0001 C CNN
 F 1 "GND" H 1255 4727 50  0000 C CNN
 F 2 "" H 1250 4900 50  0001 C CNN
@@
 	3050 5800 2750 5800
 $Comp
-L power:GND #PWR071
+L power:GND #PWR072
 U 1 1 5B171A11
 P 2000 6150
-F 0 "#PWR071" H 2000 5900 50  0001 C CNN
+F 0 "#PWR072" H 2000 5900 50  0001 C CNN
 F 1 "GND" H 2005 5977 50  0000 C CNN
 F 2 "" H 2000 6150 50  0001 C CNN
@@
 Connection ~ 3050 5800
 $Comp
-L power:GND #PWR069
+L power:GND #PWR070
 U 1 1 5B171A2B
 P 3950 5900
-F 0 "#PWR069" H 3950 5650 50  0001 C CNN
+F 0 "#PWR070" H 3950 5650 50  0001 C CNN
 F 1 "GND" H 3955 5727 50  0000 C CNN
 F 2 "" H 3950 5900 50  0001 C CNN
@@
 	3400 5800 3050 5800
 $Comp
-L remram-rescue:C-Device C34
+L remram-rescue:C-Device C35
 U 1 1 5B171A35
 P 1250 5950
-F 0 "C34" H 1365 5996 50  0000 L CNN
+F 0 "C35" H 1365 5996 50  0000 L CNN
 F 1 "100nF" H 1365 5905 50  0000 L CNN
 F 2 "Capacitor_SMD:C_0603_1608Metric" H 1288 5800 50  0001 C CNN
@@
 Connection ~ 1250 5800
 $Comp
-L power:GND #PWR070
+L power:GND #PWR071
 U 1 1 5B171A40
 P 1250 6100
-F 0 "#PWR070" H 1250 5850 50  0001 C CNN
+F 0 "#PWR071" H 1250 5850 50  0001 C CNN
 F 1 "GND" H 1255 5927 50  0000 C CNN
 F 2 "" H 1250 6100 50  0001 C CNN
@@
 	3050 7000 2750 7000
 $Comp
-L power:GND #PWR074
+L power:GND #PWR075
 U 1 1 5B171A72
 P 2000 7350
-F 0 "#PWR074" H 2000 7100 50  0001 C CNN
+F 0 "#PWR075" H 2000 7100 50  0001 C CNN
 F 1 "GND" H 2005 7177 50  0000 C CNN
 F 2 "" H 2000 7350 50  0001 C CNN
@@
 Connection ~ 3050 7000
 $Comp
-L power:GND #PWR072
+L power:GND #PWR073
 U 1 1 5B171A8C
 P 3950 7100
-F 0 "#PWR072" H 3950 6850 50  0001 C CNN
+F 0 "#PWR073" H 3950 6850 50  0001 C CNN
 F 1 "GND" H 3955 6927 50  0000 C CNN
 F 2 "" H 3950 7100 50  0001 C CNN
@@
 	3400 7000 3050 7000
 $Comp
-L remram-rescue:C-Device C35
+L remram-rescue:C-Device C36
 U 1 1 5B171A96
 P 1250 7150
-F 0 "C35" H 1365 7196 50  0000 L CNN
+F 0 "C36" H 1365 7196 50  0000 L CNN
 F 1 "100nF" H 1365 7105 50  0000 L CNN
 F 2 "Capacitor_SMD:C_0603_1608Metric" H 1288 7000 50  0001 C CNN
@@
 Connection ~ 1250 7000
 $Comp
-L power:GND #PWR073
+L power:GND #PWR074
 U 1 1 5B171AA1
 P 1250 7300
-F 0 "#PWR073" H 1250 7050 50  0001 C CNN
+F 0 "#PWR074" H 1250 7050 50  0001 C CNN
 F 1 "GND" H 1255 7127 50  0000 C CNN
 F 2 "" H 1250 7300 50  0001 C CNN
@@
 Endstops
 $Comp
-L power:GND #PWR053
+L power:GND #PWR054
 U 1 1 5B171AAF
 P 5550 950
-F 0 "#PWR053" H 5550 700 50  0001 C CNN
+F 0 "#PWR054" H 5550 700 50  0001 C CNN
 F 1 "GND" V 5555 822 50  0000 R CNN
 F 2 "" H 5550 950 50  0001 C CNN
@@
 $EndComp
 $Comp
-L power:GND #PWR054
+L power:GND #PWR055
 U 1 1 5B171ABF
 P 6750 950
-F 0 "#PWR054" H 6750 700 50  0001 C CNN
+F 0 "#PWR055" H 6750 700 50  0001 C CNN
 F 1 "GND" V 6755 822 50  0000 R CNN
 F 2 "" H 6750 950 50  0001 C CNN
@@
 $EndComp
 $Comp
-L power:GND #PWR055
+L power:GND #PWR056
 U 1 1 5B171ACF
 P 5550 1350
-F 0 "#PWR055" H 5550 1100 50  0001 C CNN
+F 0 "#PWR056" H 5550 1100 50  0001 C CNN
 F 1 "GND" V 5555 1222 50  0000 R CNN
 F 2 "" H 5550 1350 50  0001 C CNN
@@
 $EndComp
 $Comp
-L power:GND #PWR056
+L power:GND #PWR057
 U 1 1 5B171ADD
 P 6750 1350
-F 0 "#PWR056" H 6750 1100 50  0001 C CNN
+F 0 "#PWR057" H 6750 1100 50  0001 C CNN
 F 1 "GND" V 6755 1222 50  0000 R CNN
 F 2 "" H 6750 1350 50  0001 C CNN
@@
 $EndComp
 $Comp
-L power:GND #PWR059
+L power:GND #PWR060
 U 1 1 5B171AED
 P 5550 1750
-F 0 "#PWR059" H 5550 1500 50  0001 C CNN
+F 0 "#PWR060" H 5550 1500 50  0001 C CNN
 F 1 "GND" V 5555 1622 50  0000 R CNN
 F 2 "" H 5550 1750 50  0001 C CNN
@@
 $EndComp
 $Comp
-L power:GND #PWR060
+L power:GND #PWR061
 U 1 1 5B171AFB
 P 6750 1750
-F 0 "#PWR060" H 6750 1500 50  0001 C CNN
+F 0 "#PWR061" H 6750 1500 50  0001 C CNN
 F 1 "GND" V 6755 1622 50  0000 R CNN
 F 2 "" H 6750 1750 50  0001 C CNN
@@
 SWD
 $Comp
-L power:GND #PWR065
+L power:GND #PWR066
 U 1 1 5B17C4C4
 P 850 2950
-F 0 "#PWR065" H 850 2700 50  0001 C CNN
+F 0 "#PWR066" H 850 2700 50  0001 C CNN
 F 1 "GND" H 855 2777 50  0000 C CNN
 F 2 "" H 850 2950 50  0001 C CNN
@@
 VBUS
 $Comp
-L power:GNDS #PWR058
+L power:GNDS #PWR059
 U 1 1 5AF8309F
 P 1150 1700
-F 0 "#PWR058" H 1150 1450 50  0001 C CNN
+F 0 "#PWR059" H 1150 1450 50  0001 C CNN
 F 1 "GNDS" H 1155 1527 50  0000 C CNN
 F 2 "" H 1150 1700 50  0001 C CNN
@@
 VDD5V
 $Comp
-L power:GND #PWR057
+L power:GND #PWR058
 U 1 1 5AFA04BE
 P 2500 1500
-F 0 "#PWR057" H 2500 1250 50  0001 C CNN
+F 0 "#PWR058" H 2500 1250 50  0001 C CNN
 F 1 "GND" V 2505 1372 50  0000 R CNN
 F 2 "" H 2500 1500 50  0001 C CNN
@@
 VDD3V3
 $Comp
-L power:GND #PWR063
+L power:GND #PWR064
 U 1 1 5B067CCF
 P 8300 2250
-F 0 "#PWR063" H 8300 2000 50  0001 C CNN
+F 0 "#PWR064" H 8300 2000 50  0001 C CNN
 F 1 "GND" V 8305 2122 50  0000 R CNN
 F 2 "" H 8300 2250 50  0001 C CNN
@@
 	9350 2350 7700 2350
 $Comp
-L power:GND #PWR064
+L power:GND #PWR065
 U 1 1 5B009A39
 P 8800 2250
-F 0 "#PWR064" H 8800 2000 50  0001 C CNN
+F 0 "#PWR065" H 8800 2000 50  0001 C CNN
 F 1 "GND" V 8805 2122 50  0000 R CNN
 F 2 "" H 8800 2250 50  0001 C CNN
@@
 VDD5V
 $Comp
-L power:GND #PWR062
+L power:GND #PWR063
 U 1 1 5B089613
 P 8800 1950
-F 0 "#PWR062" H 8800 1700 50  0001 C CNN
+F 0 "#PWR063" H 8800 1700 50  0001 C CNN
 F 1 "GND" V 8805 1822 50  0000 R CNN
 F 2 "" H 8800 1950 50  0001 C CNN
@@
 $EndComp
 $Comp
-L power:GND #PWR061
+L power:GND #PWR062
 U 1 1 5B08B3F7
 P 8300 1950
-F 0 "#PWR061" H 8300 1700 50  0001 C CNN
+F 0 "#PWR062" H 8300 1700 50  0001 C CNN
 F 1 "GND" V 8305 1822 50  0000 R CNN
 F 2 "" H 8300 1950 50  0001 C CNN

Commit message: Fix the SWD connector
I screwed up and switched the SWDIO and SWCLK pins.
Changed lines of the file:
@@
 Text HLabel 1750 2950 2    50   Input ~ 0
 nRESET
+Text HLabel 1750 2550 2    50   Input ~ 0
+SWDIO
 Text HLabel 1750 2650 2    50   Input ~ 0
-SWDIO
-Text HLabel 1750 2550 2    50   Input ~ 0
 SWCLK
 Text Notes 650  2050 0    50   ~ 0

Commit message: Add diodes and PU to endstops and fans (SCH only)
For extra protection and PU, we added some diodes and a
pull up resistor to the endstops and the fan tachometer.
Parts:
- removed C36: 100nF, Capacitor_SMD:C_0603_1608Metric, symbol remram-rescue:C-Device
- removed D14: BAT54GWJ, Diode_SMD:D_SOD-123, symbol remram-rescue:D_Schottky-Device
- removed R25, R26: 4.7k, Resistor_SMD:R_0603_1608Metric, symbol remram-rescue:R-Device
- added C34, C37, C38, C39, C40, C41, C42, C43, C44: 100nF, Capacitor_SMD:C_0603_1608Metric, symbol remram-rescue:C-Device
- added D10, D11, D16, D17, D19, D20, D21, D22, D23, D24, D25, D26, D27, D28, D29, D30, D31: BAT54GWJ, Diode_SMD:D_SOD-123, symbol remram-rescue:D_Schottky-Device
- added R21, R22, R27, R28, R29, R32, R33, R34: 1k, Resistor_SMD:R_0603_1608Metric, symbol remram-rescue:R-Device
- added R30, R31, R35, R36: 4.7k, Resistor_SMD:R_0603_1608Metric, symbol remram-rescue:R-Device
- R23, R24: value 4.7k -> 1k
- renumbered C34 to C36, D10 to D14, D11 to D18, J11 to J10, J17 to J11, J3 to J12, J9 to J13, J12 to J14, J18 to J15, J4 to J16, J10 to J17, J13 to J18, J15 to J3, J6 to J4, J7 to J5, J8 to J6, J5 to J7, J14 to J8, J16 to J9, R21 to R25, R22 to R26
Connections:
- wire segments 79 -> 143
Other:
- note added: "Fans"
- note removed: "FANS"
- moved on the sheet: J10, J11, J15, J19, J3
