File: PCB/MCU.sch (KiCad schematic (older format))
At the start: 35 parts, among them SW1 PTS645VL39-2, SW2 OS102011MA1QN1, U4 ADUM4160, U5 STM32F765VIT6, Y1 TSX-3225 24.0000MF15X-AC3

Commit message: First draft of RemRam.
I added a 20 pin expansion connector with the following pins:
 - SPI
 - I2C
 - USART
 - 4x PWM
 - 4x GPIO
Parts:
- renumbered C28 to C23, C31 to C24, C23 to C25, C41 to C26, C30 to C27, C36 to C28, C25 to C29, C33 to C30, C37 to C31, C34 to C32, C38 to C33, C40 to C34, C24 to C35, C26 to C36, C27 to C37, C29 to C38, C32 to C39, C35 to C40, C39 to C41, R19 to R15, R20 to R16, R21 to R17, R22 to R18, R15 to R19, R17 to R20, R16 to R21, R18 to R22, SW2 to SW1, SW1 to SW2
Connections:
- net labels added: EXT_D3, EXT_D4, PWM_EXT1, PWM_EXT2, PWM_EXT3, PWM_EXT4, USART_CK, USART_RX, USART_TX
- no-connect marks 23 -> 14

Commit message: v0.2 of PCB.
After some feedback, we changed following:
 - Switched FAN VDD from 24 to 5V.
 - FAN now have a ADC pin for speed sensing.
 - Expanded EXP-3 connector to 26 pin
   - Included 24V VDD.
   - Could be used to connect up to two
     extra stepper.
 - Removed GND connections on TMC2130 to
   middel GND plane.
Connections:
- net labels added: FAN_SPEED1, FAN_SPEED2
- no-connect marks 14 -> 12
Changed lines of the file:
@@
 NoConn ~ 6900 2050
 NoConn ~ 7000 2050
-NoConn ~ 4900 4150
-NoConn ~ 5500 5250
 NoConn ~ 7100 2050
 NoConn ~ 7200 2050
@@
 NoConn ~ 5600 2050
 NoConn ~ 5500 2050
+Text HLabel 4900 4150 0    50   Input ~ 0
+FAN_SPEED1
+Text HLabel 5500 5250 3    50   Input ~ 0
+FAN_SPEED2
 $EndSCHEMATC

Commit message: Version 0.3.
Parts:
- Y1: symbol remram-rescue:Crystal-Device -> Device:Crystal_GND24
- renumbered C22 to C23, C23 to C24, C24 to C25, C25 to C26, C26 to C27, C27 to C28, C28 to C29, C29 to C30, C30 to C31, C31 to C32, C32 to C33, C33 to C34, C34 to C35, C35 to C36, C36 to C37, C37 to C38, C38 to C39, C39 to C40, C40 to C41, C41 to C42
Connections:
- wire segments 97 -> 101

Commit message: Added a yellow status LED.
Parts:
- added D15: LTST-C194KSKT, LED_SMD:LED_0603_1608Metric, symbol remram-rescue:LED-Device
- added R38: 1k, Resistor_SMD:R_0603_1608Metric, symbol remram-rescue:R-Device
Connections:
- net labels added: STATUS_LED
- wire segments 101 -> 103
- no-connect marks 12 -> 11
Changed lines of the file:
@@
 NoConn ~ 7000 2050
 NoConn ~ 7100 2050
-NoConn ~ 7200 2050
 NoConn ~ 6600 5250
 Text HLabel 1950 3250 0    50   Input ~ 0
@@
 PWM_EXT4
 NoConn ~ 5600 2050
-NoConn ~ 5500 2050
 Text HLabel 4900 4150 0    50   Input ~ 0
 FAN_SPEED1
@@
 Wire Wire Line
 	3700 3150 3700 2950
+Text Label 7200 2050 1    50   ~ 0
+STATUS_LED
+$Comp
+L remram-rescue:LED-Device D15
+U 1 1 5B007E50
+P 1700 6450
+F 0 "D15" H 1738 6332 50  0000 R CNN
+F 1 "LTST-C194KSKT" H 2000 6600 50  0000 R CNN
+F 2 "LED_SMD:LED_0603_1608Metric" H 1700 6450 50  0001 C CNN
+F 3 "~" H 1700 6450 50  0001 C CNN
+	1    1700 6450
+	-1   0    0    1
+$EndComp
+$Comp
+L remram-rescue:R-Device R38
+U 1 1 5B007E5D
+P 1400 6450
+F 0 "R38" V 1550 6450 50  0000 L CNN
+F 1 "1k" V 1470 6405 50  0000 L CNN
+F 2 "Resistor_SMD:R_0603_1608Metric" V 1330 6450 50  0001 C CNN
+F 3 "~" H 1400 6450 50  0001 C CNN
+	1    1400 6450
+	0    -1   -1   0
+$EndComp
+$Comp
+L power:GND #PWR0125
+U 1 1 5B010B0E
+P 2300 6450
+F 0 "#PWR0125" H 2300 6200 50  0001 C CNN
+F 1 "GND" H 2305 6277 50  0000 C CNN
+F 2 "" H 2300 6450 50  0001 C CNN
+F 3 "" H 2300 6450 50  0001 C CNN
+	1    2300 6450
+	1    0    0    -1
+$EndComp
+Wire Wire Line
+	1850 6450 2300 6450
+Text Label 750  6450 0    50   ~ 0
+STATUS_LED
+Wire Wire Line
+	750  6450 1250 6450
+NoConn ~ 5500 2050
 $EndSCHEMATC

Commit message: Changed the LED resistors to real values.
Parts:
- R38: value 1k -> 68
Changed lines of the file:
@@
 P 1400 6450
 F 0 "R38" V 1550 6450 50  0000 L CNN
-F 1 "1k" V 1470 6405 50  0000 L CNN
+F 1 "68" V 1470 6405 50  0000 L CNN
 F 2 "Resistor_SMD:R_0603_1608Metric" V 1330 6450 50  0001 C CNN
 F 3 "~" H 1400 6450 50  0001 C CNN

Commit message: Changed ordering of parts. Version 0.4.
Parts:
- renumbered C23 to C14, C24 to C15, C25 to C16, C26 to C17, C27 to C18, C28 to C19, C29 to C20, C30 to C21, C31 to C22, C32 to C23, C33 to C24, C34 to C25, C35 to C26, C36 to C27, C37 to C28, C38 to C29, C39 to C30, C40 to C31, C41 to C32, C42 to C33, D15 to D9, R15 to R12, R16 to R13, R17 to R14, R18 to R15, R19 to R16, R20 to R17, R21 to R18, R22 to R19, R38 to R20, U4 to U3, U5 to U4

Commit message: Removed USART1 CK pin and added another digial pin.
STM32duino doesn't seem to support USART. So I will only
implement the UART pins.
Connections:
- net labels added: EXT_D5
- net labels removed: USART_CK
Changed lines of the file:
@@
 $Descr A4 11693 8268
 encoding utf-8
-Sheet 5 9
+Sheet 4 9
 Title "MCU"
 Date ""
@@
 NoConn ~ 6500 2050
 NoConn ~ 5800 2050
-NoConn ~ 5700 2050
 Text HLabel 4900 2450 0    50   Input ~ 0
 EXT_D4
@@
 Text HLabel 8100 3150 2    50   Input ~ 0
 USART_TX
-Text HLabel 8100 3250 2    50   Input ~ 0
-USART_CK
 Text HLabel 8100 3450 2    50   Input ~ 0
 PWM_EXT3
@@
 Wire Wire Line
 	750  6450 1250 6450
-NoConn ~ 5500 2050
+Text HLabel 5500 2050 1    50   Input ~ 0
+EXT_D5
+NoConn ~ 5700 2050
+NoConn ~ 8100 3250
 $EndSCHEMATC

Commit message: Changed LED to sane values. Updated diodes. v0.5.
Parts:
- R20: value 68 -> 1k
Changed lines of the file:
@@
 P 1400 6450
 F 0 "R20" V 1550 6450 50  0000 L CNN
-F 1 "68" V 1470 6405 50  0000 L CNN
+F 1 "1k" V 1470 6405 50  0000 L CNN
 F 2 "Resistor_SMD:R_0603_1608Metric" V 1330 6450 50  0001 C CNN
 F 3 "~" H 1400 6450 50  0001 C CNN
