File: PCB/MCU.sch (KiCad schematic (older format))
At the start: 37 parts, among them SW1 OS102011MA1QN1, SW2 PTS645VL39-2, U3 ADUM4160, U4 STM32F765VIT6, Y1 TSX-3225 24.0000MF15X-AC3

Commit message: Added a battery for SRAM backup.
Parts:
- removed C33: 100nF, Capacitor_SMD:C_0603_1608Metric, symbol remram-rescue:C-Device
- added BT1: VBH2032-1, custom-footprints:VBH2032-1, symbol remram-custom:VBH2032-1
Connections:
- wire segments 103 -> 104
Changed lines of the file:
@@
 	0    1    1    0
 $EndComp
-Text GLabel 4900 2950 0    50   Input ~ 0
-VDD3V3
 Text GLabel 2600 4450 0    50   Input ~ 0
 VDD3V3
@@
 	-1   0    0    1
 $EndComp
-Connection ~ 3450 7450
-Wire Wire Line
-	3900 7450 3450 7450
-Connection ~ 3450 7150
-Wire Wire Line
-	3450 7150 3900 7150
-$Comp
-L remram-rescue:C-Device C33
-U 1 1 5AD09E9B
-P 3900 7300
-F 0 "C33" H 4015 7346 50  0000 L CNN
-F 1 "100nF" H 4015 7255 50  0000 L CNN
-F 2 "Capacitor_SMD:C_0603_1608Metric" H 3938 7150 50  0001 C CNN
-F 3 "~" H 3900 7300 50  0001 C CNN
-	1    3900 7300
-	1    0    0    -1
-$EndComp
-$Comp
-L power:GND #PWR048
+$Comp
+L power:GND #PWR049
 U 1 1 5AF57331
 P 5300 5350
-F 0 "#PWR048" H 5300 5100 50  0001 C CNN
+F 0 "#PWR049" H 5300 5100 50  0001 C CNN
 F 1 "GND" H 5305 5177 50  0000 C CNN
 F 2 "" H 5300 5350 50  0001 C CNN
@@
 $EndComp
 $Comp
-L power:GND #PWR047
+L power:GND #PWR048
 U 1 1 5AF579EA
 P 3850 4750
-F 0 "#PWR047" H 3850 4500 50  0001 C CNN
+F 0 "#PWR048" H 3850 4500 50  0001 C CNN
 F 1 "GND" H 3855 4577 50  0000 C CNN
 F 2 "" H 3850 4750 50  0001 C CNN
@@
 $EndComp
 $Comp
-L power:GND #PWR046
+L power:GND #PWR047
 U 1 1 5AF580A3
 P 3450 4750
-F 0 "#PWR046" H 3450 4500 50  0001 C CNN
+F 0 "#PWR047" H 3450 4500 50  0001 C CNN
 F 1 "GND" H 3455 4577 50  0000 C CNN
 F 2 "" H 3450 4750 50  0001 C CNN
@@
 $EndComp
 $Comp
-L power:GND #PWR043
+L power:GND #PWR044
 U 1 1 5AF58792
 P 3450 4050
-F 0 "#PWR043" H 3450 3800 50  0001 C CNN
+F 0 "#PWR044" H 3450 3800 50  0001 C CNN
 F 1 "GND" H 3455 3877 50  0000 C CNN
 F 2 "" H 3450 4050 50  0001 C CNN
@@
 $EndComp
 $Comp
-L power:GND #PWR044
+L power:GND #PWR045
 U 1 1 5AF59C69
 P 3850 4050
-F 0 "#PWR044" H 3850 3800 50  0001 C CNN
+F 0 "#PWR045" H 3850 3800 50  0001 C CNN
 F 1 "GND" H 3855 3877 50  0000 C CNN
 F 2 "" H 3850 4050 50  0001 C CNN
@@
 $EndComp
 $Comp
-L power:GND #PWR041
+L power:GND #PWR042
 U 1 1 5AF5B126
 P 4900 3350
-F 0 "#PWR041" H 4900 3100 50  0001 C CNN
+F 0 "#PWR042" H 4900 3100 50  0001 C CNN
 F 1 "GND" V 4905 3222 50  0000 R CNN
 F 2 "" H 4900 3350 50  0001 C CNN
@@
 $EndComp
 $Comp
-L power:GND #PWR045
+L power:GND #PWR046
 U 1 1 5AF5BF00
 P 4900 4250
-F 0 "#PWR045" H 4900 4000 50  0001 C CNN
+F 0 "#PWR046" H 4900 4000 50  0001 C CNN
 F 1 "GND" V 4905 4122 50  0000 R CNN
 F 2 "" H 4900 4250 50  0001 C CNN
@@
 $EndComp
 $Comp
-L power:GND #PWR038
+L power:GND #PWR039
 U 1 1 5AF5E7FC
 P 8750 2250
-F 0 "#PWR038" H 8750 2000 50  0001 C CNN
+F 0 "#PWR039" H 8750 2000 50  0001 C CNN
 F 1 "GND" H 8750 2100 50  0000 C CNN
 F 2 "" H 8750 2250 50  0001 C CNN
@@
 $EndComp
 $Comp
-L power:GND #PWR049
+L power:GND #PWR050
 U 1 1 5AF5F2E4
 P 7950 5800
-F 0 "#PWR049" H 7950 5550 50  0001 C CNN
+F 0 "#PWR050" H 7950 5550 50  0001 C CNN
 F 1 "GND" H 7955 5627 50  0000 C CNN
 F 2 "" H 7950 5800 50  0001 C CNN
@@
 $EndComp
 $Comp
-L power:GND #PWR040
+L power:GND #PWR041
 U 1 1 5AF5AB44
 P 3700 2950
-F 0 "#PWR040" H 3700 2700 50  0001 C CNN
+F 0 "#PWR041" H 3700 2700 50  0001 C CNN
 F 1 "GND" V 3705 2822 50  0000 R CNN
 F 2 "" H 3700 2950 50  0001 C CNN
@@
 $EndComp
 $Comp
-L power:GND #PWR039
+L power:GND #PWR040
 U 1 1 5AF5ABF2
 P 2700 2950
-F 0 "#PWR039" H 2700 2700 50  0001 C CNN
+F 0 "#PWR040" H 2700 2700 50  0001 C CNN
 F 1 "GND" V 2705 2822 50  0000 R CNN
 F 2 "" H 2700 2950 50  0001 C CNN
@@
 $EndComp
 $Comp
-L power:GND #PWR042
+L power:GND #PWR043
 U 1 1 5AF616AA
 P 1150 3750
-F 0 "#PWR042" H 1150 3500 50  0001 C CNN
+F 0 "#PWR043" H 1150 3500 50  0001 C CNN
 F 1 "GND" H 1155 3577 50  0000 C CNN
 F 2 "" H 1150 3750 50  0001 C CNN
@@
 Connection ~ 2050 2250
 $Comp
-L power:GND #PWR037
+L power:GND #PWR038
 U 1 1 5AF61872
 P 2050 2250
-F 0 "#PWR037" H 2050 2000 50  0001 C CNN
+F 0 "#PWR038" H 2050 2000 50  0001 C CNN
 F 1 "GND" H 2055 2077 50  0000 C CNN
 F 2 "" H 2050 2250 50  0001 C CNN
@@
 $EndComp
 $Comp
-L power:GNDS #PWR036
+L power:GNDS #PWR037
 U 1 1 5AF61805
 P 1650 2250
-F 0 "#PWR036" H 1650 2000 50  0001 C CNN
+F 0 "#PWR037" H 1650 2000 50  0001 C CNN
 F 1 "GNDS" H 1655 2077 50  0000 C CNN
 F 2 "" H 1650 2250 50  0001 C CNN
@@
 	6000 750  6000 900
 $Comp
-L power:GND #PWR051
+L power:GND #PWR052
 U 1 1 5AFDE2A1
 P 950 7450
-F 0 "#PWR051" H 950 7200 50  0001 C CNN
+F 0 "#PWR052" H 950 7200 50  0001 C CNN
 F 1 "GND" H 955 7277 50  0000 C CNN
 F 2 "" H 950 7450 50  0001 C CNN
@@
 $EndComp
 $Comp
-L power:GND #PWR050
+L power:GND #PWR051
 U 1 1 5B010B0E
 P 2300 6450
-F 0 "#PWR050" H 2300 6200 50  0001 C CNN
+F 0 "#PWR051" H 2300 6200 50  0001 C CNN
 F 1 "GND" H 2305 6277 50  0000 C CNN
 F 2 "" H 2300 6450 50  0001 C CNN
@@
 NoConn ~ 5700 2050
 NoConn ~ 8100 3250
+$Comp
+L power:GND #PWR036
+U 1 1 5B0EA618
+P 4150 2150
+F 0 "#PWR036" H 4150 1900 50  0001 C CNN
+F 1 "GND" H 4155 1977 50  0000 C CNN
+F 2 "" H 4150 2150 50  0001 C CNN
+F 3 "" H 4150 2150 50  0001 C CNN
+	1    4150 2150
+	-1   0    0    1
+$EndComp
+$Comp
+L remram-custom:VBH2032-1 BT1
+U 1 1 5B0EA684
+P 4150 2250
+F 0 "BT1" H 4268 2346 50  0000 L CNN
+F 1 "VBH2032-1" H 4268 2255 50  0000 L CNN
+F 2 "custom-footprints:VBH2032-1" V 4150 2310 50  0001 C CNN
+F 3 "https://www.mouser.de/datasheet/2/346/VBH2032-1_new-258024.pdf" V 4150 2310 50  0001 C CNN
+	1    4150 2250
+	-1   0    0    1
+$EndComp
+Wire Wire Line
+	4150 2450 4200 2450
+Wire Wire Line
+	4150 2450 4150 2950
+Wire Wire Line
+	4150 2950 4900 2950
+Connection ~ 4150 2450
 $EndSCHEMATC

Commit message: Change DC-DC layout
The ripple on the 5V and 3V3 rail was too high (360mV).

In an attempt to reduce the RF and HF noise, I changed the layout
to a more compact one. I also added a third 22uF output capacitor
behind the inductor to lower ESR. I also added a 100nf input
capacitor to combat HF noise, as recommended in the datasheet.

The BOM needs to be updated in such a way, that we specificly
choose low ESR resistors.
Parts:
- renumbered C14 to C15, C15 to C16, C16 to C17, C17 to C18, C18 to C19, C19 to C20, C20 to C21, C21 to C22, C22 to C23, C23 to C24, C24 to C25, C25 to C26, C26 to C27, C27 to C28, C28 to C29, C29 to C30, C30 to C31, C31 to C32, C32 to C33

Commit message: Change 1k resistors to 4.7k. Update Symbols
Had to update the symbols to the right library again, since
Kicad Nightly changed their library order.

Also changed the 1k resistors to 4.7k to unify resistors and
also upped the PU to a weaker value.
Parts:
- added Q?: IRLML6401, symbol Device:Q_PMOS_GSD
- C15, C16, C17, C18, C19, C20, C21, C22, C23, C24, C25, C26, C27, C28, C29, C30, C31, C32, C33: symbol remram-rescue:C-Device -> Device:C
- D9: symbol remram-rescue:LED-Device -> Device:LED
- FB1, FB2: symbol remram-rescue:Ferrite_Bead_Small-Device -> Device:Ferrite_Bead_Small
- R12, R13, R14, R15, R16, R17, R18, R19: symbol remram-rescue:R-Device -> Device:R
- R20: value 1k -> 4.7k; symbol remram-rescue:R-Device -> Device:R
- U3: symbol remram-rescue:ADUM4160-Interface_USB -> Interface_USB:ADUM4160
Changed lines of the file:
@@
 $EndDescr
 $Comp
-L remram-rescue:R-Device R12
+L Device:R R12
 U 1 1 5AD0B119
 P 5550 750
@@
 $EndComp
 $Comp
-L remram-rescue:R-Device R13
+L Device:R R13
 U 1 1 5AD0B198
 P 6300 750
@@
 VDD3V3
 $Comp
-L remram-rescue:C-Device C25
+L Device:C C25
 U 1 1 5AD085F7
 P 3450 4600
@@
 $EndComp
 $Comp
-L remram-rescue:C-Device C26
+L Device:C C26
 U 1 1 5AD086E9
 P 3850 4600
@@
 VDD3V3
 $Comp
-L remram-rescue:C-Device C23
+L Device:C C23
 U 1 1 5AD08A76
 P 3450 4200
@@
 $EndComp
 $Comp
-L remram-rescue:C-Device C24
+L Device:C C24
 U 1 1 5AD08A7D
 P 3850 4200
@@
 VDD3V3
 $Comp
-L remram-rescue:C-Device C28
+L Device:C C28
 U 1 1 5AD093F4
 P 1200 7300
@@
 $EndComp
 $Comp
-L remram-rescue:C-Device C29
+L Device:C C29
 U 1 1 5AD0945E
 P 1650 7300
@@
 $EndComp
 $Comp
-L remram-rescue:C-Device C30
+L Device:C C30
 U 1 1 5AD09C8C
 P 2100 7300
@@
 $EndComp
 $Comp
-L remram-rescue:C-Device C31
+L Device:C C31
 U 1 1 5AD09D94
 P 2550 7300
@@
 $EndComp
 $Comp
-L remram-rescue:C-Device C32
+L Device:C C32
 U 1 1 5AD09D9B
 P 3000 7300
@@
 $EndComp
 $Comp
-L remram-rescue:C-Device C33
+L Device:C C33
 U 1 1 5AD09E94
 P 3450 7300
@@
 VDD3V3
 $Comp
-L remram-rescue:C-Device C27
+L Device:C C27
 U 1 1 5AD0FCE6
 P 7650 5800
@@
 $EndComp
 $Comp
-L remram-rescue:C-Device C19
+L Device:C C19
 U 1 1 5AD117D1
 P 8750 2500
@@
 $EndComp
 $Comp
-L remram-rescue:C-Device C20
+L Device:C C20
 U 1 1 5AF5755A
 P 2850 2950
@@
 $EndComp
 $Comp
-L remram-rescue:C-Device C21
+L Device:C C21
 U 1 1 5AF58CDB
 P 3550 2950
@@
 	1150 3750 1400 3750
 $Comp
-L remram-rescue:C-Device C22
+L Device:C C22
 U 1 1 5AF62329
 P 1600 4100
@@
 	7500 5250 7500 5800
 $Comp
-L remram-rescue:Ferrite_Bead_Small-Device FB1
+L Device:Ferrite_Bead_Small FB1
 U 1 1 5AF6D789
 P 2900 4350
@@
 $EndComp
 $Comp
-L remram-rescue:Ferrite_Bead_Small-Device FB2
+L Device:Ferrite_Bead_Small FB2
 U 1 1 5AF6DF9B
 P 3000 4450
@@
 Connection ~ 3000 900
 $Comp
-L remram-rescue:C-Device C17
+L Device:C C17
 U 1 1 5AFAB97B
 P 3000 1050
@@
 Connection ~ 2450 750
 $Comp
-L remram-rescue:C-Device C16
+L Device:C C16
 U 1 1 5AF92848
 P 2450 900
@@
 Connection ~ 1100 750
 $Comp
-L remram-rescue:C-Device C15
+L Device:C C15
 U 1 1 5AF88ED8
 P 1100 900
@@
 	750  1150 750  1650
 $Comp
-L remram-rescue:C-Device C18
+L Device:C C18
 U 1 1 5AF7B28D
 P 1200 2250
@@
 $EndComp
 $Comp
-L remram-rescue:R-Device R19
+L Device:R R19
 U 1 1 5AF72C01
 P 2500 1550
@@
 $EndComp
 $Comp
-L remram-rescue:R-Device R17
+L Device:R R17
 U 1 1 5AF72BFA
 P 2500 1450
@@
 $EndComp
 $Comp
-L remram-rescue:R-Device R18
+L Device:R R18
 U 1 1 5AF724F0
 P 1200 1550
@@
 $EndComp
 $Comp
-L remram-rescue:R-Device R16
+L Device:R R16
 U 1 1 5AF72236
 P 1200 1450
@@
 VBUS
 $Comp
-L remram-rescue:ADUM4160-Interface_USB U3
+L Interface_USB:ADUM4160 U3
 U 1 1 5AF5F784
 P 1850 1550
@@
 	2350 1250 2650 1250
 $Comp
-L remram-rescue:R-Device R15
+L Device:R R15
 U 1 1 5AFBD0C4
 P 7350 1150
@@
 Connection ~ 7350 750
 $Comp
-L remram-rescue:R-Device R14
+L Device:R R14
 U 1 1 5AFBD0BD
 P 7000 1150
@@
 STATUS_LED
 $Comp
-L remram-rescue:LED-Device D9
+L Device:LED D9
 U 1 1 5B007E50
 P 1700 6450
@@
 $EndComp
 $Comp
-L remram-rescue:R-Device R20
+L Device:R R20
 U 1 1 5B007E5D
 P 1400 6450
 F 0 "R20" V 1550 6450 50  0000 L CNN
-F 1 "1k" V 1470 6405 50  0000 L CNN
+F 1 "4.7k" V 1470 6405 50  0000 L CNN
 F 2 "Resistor_SMD:R_0603_1608Metric" V 1330 6450 50  0001 C CNN
 F 3 "~" H 1400 6450 50  0001 C CNN
@@
 L power:GND #PWR037
 U 1 1 5B0EA618
-P 4150 2150
-F 0 "#PWR037" H 4150 1900 50  0001 C CNN
-F 1 "GND" H 4155 1977 50  0000 C CNN
-F 2 "" H 4150 2150 50  0001 C CNN
-F 3 "" H 4150 2150 50  0001 C CNN
-	1    4150 2150
+P 4150 1700
+F 0 "#PWR037" H 4150 1450 50  0001 C CNN
+F 1 "GND" H 4155 1527 50  0000 C CNN
+F 2 "" H 4150 1700 50  0001 C CNN
+F 3 "" H 4150 1700 50  0001 C CNN
+	1    4150 1700
 	-1   0    0    1
 $EndComp
@@
 L remram-custom:VBH2032-1 BT1
 U 1 1 5B0EA684
-P 4150 2250
-F 0 "BT1" H 4268 2346 50  0000 L CNN
-F 1 "VBH2032-1" H 4268 2255 50  0000 L CNN
-F 2 "custom-footprints:VBH2032-1" V 4150 2310 50  0001 C CNN
-F 3 "https://www.mouser.de/datasheet/2/346/VBH2032-1_new-258024.pdf" V 4150 2310 50  0001 C CNN
-	1    4150 2250
+P 4150 1800
+F 0 "BT1" H 4268 1896 50  0000 L CNN
+F 1 "VBH2032-1" H 4268 1805 50  0000 L CNN
+F 2 "custom-footprints:VBH2032-1" V 4150 1860 50  0001 C CNN
+F 3 "https://www.mouser.de/datasheet/2/346/VBH2032-1_new-258024.pdf" V 4150 1860 50  0001 C CNN
+	1    4150 1800
 	-1   0    0    1
 $EndComp
 Wire Wire Line
-	4150 2450 4200 2450
-Wire Wire Line
-	4150 2450 4150 2950
-Wire Wire Line
 	4150 2950 4900 2950
-Connection ~ 4150 2450
+$Comp
+L Device:Q_PMOS_GSD Q?
+U 1 1 5B3AC772
+P 4050 2200
+F 0 "Q?" H 4255 2246 50  0000 L CNN
+F 1 "IRLML6401" H 4255 2155 50  0000 L CNN
+F 2 "" H 4250 2300 50  0001 C CNN
+F 3 "~" H 4050 2200 50  0001 C CNN
+	1    4050 2200
+	1    0    0    -1
+$EndComp
+$Comp
+L power:GND #PWR?
+U 1 1 5B3AC87D
+P 3850 2200
+F 0 "#PWR?" H 3850 1950 50  0001 C CNN
+F 1 "GND" H 3855 2027 50  0000 C CNN
+F 2 "" H 3850 2200 50  0001 C CNN
+F 3 "" H 3850 2200 50  0001 C CNN
+	1    3850 2200
+	0    1    1    0
+$EndComp
+Wire Wire Line
+	4200 2000 4150 2000
+Connection ~ 4150 2000
+Wire Wire Line
+	4150 2400 4150 2950
 $EndSCHEMATC

Commit message: Added protection diodes to TMC2130
Diode on IO voltage protects chip to only accept command when
motor voltage is present.

Clamping diodes on motor outputs are for inductive loads.
Parts:
- gave numbers to parts that had none: 1
Changed lines of the file:
@@
 $EndComp
 $Comp
-L power:GND #PWR050
+L power:GND #PWR051
 U 1 1 5AF57331
 P 5300 5350
-F 0 "#PWR050" H 5300 5100 50  0001 C CNN
+F 0 "#PWR051" H 5300 5100 50  0001 C CNN
 F 1 "GND" H 5305 5177 50  0000 C CNN
 F 2 "" H 5300 5350 50  0001 C CNN
@@
 $EndComp
 $Comp
-L power:GND #PWR049
+L power:GND #PWR050
 U 1 1 5AF579EA
 P 3850 4750
-F 0 "#PWR049" H 3850 4500 50  0001 C CNN
+F 0 "#PWR050" H 3850 4500 50  0001 C CNN
 F 1 "GND" H 3855 4577 50  0000 C CNN
 F 2 "" H 3850 4750 50  0001 C CNN
@@
 $EndComp
 $Comp
-L power:GND #PWR048
+L power:GND #PWR049
 U 1 1 5AF580A3
 P 3450 4750
-F 0 "#PWR048" H 3450 4500 50  0001 C CNN
+F 0 "#PWR049" H 3450 4500 50  0001 C CNN
 F 1 "GND" H 3455 4577 50  0000 C CNN
 F 2 "" H 3450 4750 50  0001 C CNN
@@
 $EndComp
 $Comp
-L power:GND #PWR045
+L power:GND #PWR046
 U 1 1 5AF58792
 P 3450 4050
-F 0 "#PWR045" H 3450 3800 50  0001 C CNN
+F 0 "#PWR046" H 3450 3800 50  0001 C CNN
 F 1 "GND" H 3455 3877 50  0000 C CNN
 F 2 "" H 3450 4050 50  0001 C CNN
@@
 $EndComp
 $Comp
-L power:GND #PWR046
+L power:GND #PWR047
 U 1 1 5AF59C69
 P 3850 4050
-F 0 "#PWR046" H 3850 3800 50  0001 C CNN
+F 0 "#PWR047" H 3850 3800 50  0001 C CNN
 F 1 "GND" H 3855 3877 50  0000 C CNN
 F 2 "" H 3850 4050 50  0001 C CNN
@@
 $EndComp
 $Comp
-L power:GND #PWR043
+L power:GND #PWR044
 U 1 1 5AF5B126
 P 4900 3350
-F 0 "#PWR043" H 4900 3100 50  0001 C CNN
+F 0 "#PWR044" H 4900 3100 50  0001 C CNN
 F 1 "GND" V 4905 3222 50  0000 R CNN
 F 2 "" H 4900 3350 50  0001 C CNN
@@
 $EndComp
 $Comp
-L power:GND #PWR047
+L power:GND #PWR048
 U 1 1 5AF5BF00
 P 4900 4250
-F 0 "#PWR047" H 4900 4000 50  0001 C CNN
+F 0 "#PWR048" H 4900 4000 50  0001 C CNN
 F 1 "GND" V 4905 4122 50  0000 R CNN
 F 2 "" H 4900 4250 50  0001 C CNN
@@
 $EndComp
 $Comp
-L power:GND #PWR036
+L power:GND #PWR037
 U 1 1 5AF5CFF3
 P 5400 2050
-F 0 "#PWR036" H 5400 1800 50  0001 C CNN
+F 0 "#PWR037" H 5400 1800 50  0001 C CNN
 F 1 "GND" H 5405 1877 50  0000 C CNN
 F 2 "" H 5400 2050 50  0001 C CNN
@@
 $EndComp
 $Comp
-L power:GND #PWR040
+L power:GND #PWR041
 U 1 1 5AF5E7FC
 P 8750 2250
-F 0 "#PWR040" H 8750 2000 50  0001 C CNN
+F 0 "#PWR041" H 8750 2000 50  0001 C CNN
 F 1 "GND" H 8750 2100 50  0000 C CNN
 F 2 "" H 8750 2250 50  0001 C CNN
@@
 $EndComp
 $Comp
-L power:GND #PWR051
+L power:GND #PWR052
 U 1 1 5AF5F2E4
 P 7950 5800
-F 0 "#PWR051" H 7950 5550 50  0001 C CNN
+F 0 "#PWR052" H 7950 5550 50  0001 C CNN
 F 1 "GND" H 7955 5627 50  0000 C CNN
 F 2 "" H 7950 5800 50  0001 C CNN
@@
 $EndComp
 $Comp
-L power:GND #PWR042
+L power:GND #PWR043
 U 1 1 5AF5AB44
 P 3700 2950
-F 0 "#PWR042" H 3700 2700 50  0001 C CNN
+F 0 "#PWR043" H 3700 2700 50  0001 C CNN
 F 1 "GND" V 3705 2822 50  0000 R CNN
 F 2 "" H 3700 2950 50  0001 C CNN
@@
 $EndComp
 $Comp
-L power:GND #PWR041
+L power:GND #PWR042
 U 1 1 5AF5ABF2
 P 2700 2950
-F 0 "#PWR041" H 2700 2700 50  0001 C CNN
+F 0 "#PWR042" H 2700 2700 50  0001 C CNN
 F 1 "GND" V 2705 2822 50  0000 R CNN
 F 2 "" H 2700 2950 50  0001 C CNN
@@
 $EndComp
 $Comp
-L power:GND #PWR044
+L power:GND #PWR045
 U 1 1 5AF616AA
 P 1150 3750
-F 0 "#PWR044" H 1150 3500 50  0001 C CNN
+F 0 "#PWR045" H 1150 3500 50  0001 C CNN
 F 1 "GND" H 1155 3577 50  0000 C CNN
 F 2 "" H 1150 3750 50  0001 C CNN
@@
 Connection ~ 2050 2250
 $Comp
-L power:GND #PWR039
+L power:GND #PWR040
 U 1 1 5AF61872
 P 2050 2250
-F 0 "#PWR039" H 2050 2000 50  0001 C CNN
+F 0 "#PWR040" H 2050 2000 50  0001 C CNN
 F 1 "GND" H 2055 2077 50  0000 C CNN
 F 2 "" H 2050 2250 50  0001 C CNN
@@
 $EndComp
 $Comp
-L power:GNDS #PWR038
+L power:GNDS #PWR039
 U 1 1 5AF61805
 P 1650 2250
-F 0 "#PWR038" H 1650 2000 50  0001 C CNN
+F 0 "#PWR039" H 1650 2000 50  0001 C CNN
 F 1 "GNDS" H 1655 2077 50  0000 C CNN
 F 2 "" H 1650 2250 50  0001 C CNN
@@
 	6000 750  6000 900
 $Comp
-L power:GND #PWR053
+L power:GND #PWR054
 U 1 1 5AFDE2A1
 P 950 7450
-F 0 "#PWR053" H 950 7200 50  0001 C CNN
+F 0 "#PWR054" H 950 7200 50  0001 C CNN
 F 1 "GND" H 955 7277 50  0000 C CNN
 F 2 "" H 950 7450 50  0001 C CNN
@@
 $EndComp
 $Comp
-L power:GND #PWR052
+L power:GND #PWR053
 U 1 1 5B010B0E
 P 2300 6450
-F 0 "#PWR052" H 2300 6200 50  0001 C CNN
+F 0 "#PWR053" H 2300 6200 50  0001 C CNN
 F 1 "GND" H 2305 6277 50  0000 C CNN
 F 2 "" H 2300 6450 50  0001 C CNN
@@
 NoConn ~ 8100 3250
 $Comp
-L power:GND #PWR037
+L power:GND #PWR036
 U 1 1 5B0EA618
 P 4150 1700
-F 0 "#PWR037" H 4150 1450 50  0001 C CNN
+F 0 "#PWR036" H 4150 1450 50  0001 C CNN
 F 1 "GND" H 4155 1527 50  0000 C CNN
 F 2 "" H 4150 1700 50  0001 C CNN
@@
 	4150 2950 4900 2950
 $Comp
-L Device:Q_PMOS_GSD Q?
+L Device:Q_PMOS_GSD Q5
 U 1 1 5B3AC772
 P 4050 2200
-F 0 "Q?" H 4255 2246 50  0000 L CNN
+F 0 "Q5" H 4255 2246 50  0000 L CNN
 F 1 "IRLML6401" H 4255 2155 50  0000 L CNN
 F 2 "" H 4250 2300 50  0001 C CNN
@@
 $EndComp
 $Comp
-L power:GND #PWR?
+L power:GND #PWR038
 U 1 1 5B3AC87D
 P 3850 2200
-F 0 "#PWR?" H 3850 1950 50  0001 C CNN
+F 0 "#PWR038" H 3850 1950 50  0001 C CNN
 F 1 "GND" H 3855 2027 50  0000 C CNN
 F 2 "" H 3850 2200 50  0001 C CNN

Commit message: Add missing MOSFET footprint
Parts:
- Q5: footprint (none) -> Package_TO_SOT_SMD:SOT-23
Changed lines of the file:
@@
 F 0 "Q5" H 4255 2246 50  0000 L CNN
 F 1 "IRLML6401" H 4255 2155 50  0000 L CNN
-F 2 "" H 4250 2300 50  0001 C CNN
-F 3 "~" H 4050 2200 50  0001 C CNN
+F 2 "Package_TO_SOT_SMD:SOT-23" H 4250 2300 50  0001 C CNN
+F 3 "https://www.infineon.com/dgdl/irlml6401pbf.pdf?fileId=5546d462533600a401535668b96d2634" H 4050 2200 50  0001 C CNN
 	1    4050 2200
 	1    0    0    -1
