File: PCB/MCU.sch (KiCad schematic (older format))
At the start: 38 parts, among them Q5 IRLML6401, SW1 OS102011MA1QN1, SW2 PTS645VL39-2, U3 ADUM4160, U4 STM32F765VIT6, Y1 TSX-3225 24.0000MF15X-AC3

Commit message: Fix PU on FAN RPM, Endstops and Grounding
 * Fixes too weak PU on RPM for fans
 * Simplified endstop setup
 * Grounding fixes:
   * GND below SPI bus
   * 3V3 LDO directly attached
     to main PWR source

Fixes #20
Parts:
- R20: value 4.7k -> 1k
Changed lines of the file:
@@
 $EndComp
 $Comp
-L power:GND #PWR051
+L power:GND #PWR050
 U 1 1 5AF57331
 P 5300 5350
-F 0 "#PWR051" H 5300 5100 50  0001 C CNN
+F 0 "#PWR050" H 5300 5100 50  0001 C CNN
 F 1 "GND" H 5305 5177 50  0000 C CNN
 F 2 "" H 5300 5350 50  0001 C CNN
@@
 $EndComp
 $Comp
-L power:GND #PWR050
+L power:GND #PWR049
 U 1 1 5AF579EA
 P 3850 4750
-F 0 "#PWR050" H 3850 4500 50  0001 C CNN
+F 0 "#PWR049" H 3850 4500 50  0001 C CNN
 F 1 "GND" H 3855 4577 50  0000 C CNN
 F 2 "" H 3850 4750 50  0001 C CNN
@@
 $EndComp
 $Comp
-L power:GND #PWR049
+L power:GND #PWR048
 U 1 1 5AF580A3
 P 3450 4750
-F 0 "#PWR049" H 3450 4500 50  0001 C CNN
+F 0 "#PWR048" H 3450 4500 50  0001 C CNN
 F 1 "GND" H 3455 4577 50  0000 C CNN
 F 2 "" H 3450 4750 50  0001 C CNN
@@
 $EndComp
 $Comp
-L power:GND #PWR046
+L power:GND #PWR045
 U 1 1 5AF58792
 P 3450 4050
-F 0 "#PWR046" H 3450 3800 50  0001 C CNN
+F 0 "#PWR045" H 3450 3800 50  0001 C CNN
 F 1 "GND" H 3455 3877 50  0000 C CNN
 F 2 "" H 3450 4050 50  0001 C CNN
@@
 $EndComp
 $Comp
-L power:GND #PWR047
+L power:GND #PWR046
 U 1 1 5AF59C69
 P 3850 4050
-F 0 "#PWR047" H 3850 3800 50  0001 C CNN
+F 0 "#PWR046" H 3850 3800 50  0001 C CNN
 F 1 "GND" H 3855 3877 50  0000 C CNN
 F 2 "" H 3850 4050 50  0001 C CNN
@@
 $EndComp
 $Comp
-L power:GND #PWR044
+L power:GND #PWR043
 U 1 1 5AF5B126
 P 4900 3350
-F 0 "#PWR044" H 4900 3100 50  0001 C CNN
+F 0 "#PWR043" H 4900 3100 50  0001 C CNN
 F 1 "GND" V 4905 3222 50  0000 R CNN
 F 2 "" H 4900 3350 50  0001 C CNN
@@
 $EndComp
 $Comp
-L power:GND #PWR048
+L power:GND #PWR047
 U 1 1 5AF5BF00
 P 4900 4250
-F 0 "#PWR048" H 4900 4000 50  0001 C CNN
+F 0 "#PWR047" H 4900 4000 50  0001 C CNN
 F 1 "GND" V 4905 4122 50  0000 R CNN
 F 2 "" H 4900 4250 50  0001 C CNN
@@
 $EndComp
 $Comp
-L power:GND #PWR037
+L power:GND #PWR036
 U 1 1 5AF5CFF3
 P 5400 2050
-F 0 "#PWR037" H 5400 1800 50  0001 C CNN
+F 0 "#PWR036" H 5400 1800 50  0001 C CNN
 F 1 "GND" H 5405 1877 50  0000 C CNN
 F 2 "" H 5400 2050 50  0001 C CNN
@@
 $EndComp
 $Comp
-L power:GND #PWR041
+L power:GND #PWR040
 U 1 1 5AF5E7FC
 P 8750 2250
-F 0 "#PWR041" H 8750 2000 50  0001 C CNN
+F 0 "#PWR040" H 8750 2000 50  0001 C CNN
 F 1 "GND" H 8750 2100 50  0000 C CNN
 F 2 "" H 8750 2250 50  0001 C CNN
@@
 $EndComp
 $Comp
-L power:GND #PWR052
+L power:GND #PWR051
 U 1 1 5AF5F2E4
 P 7950 5800
-F 0 "#PWR052" H 7950 5550 50  0001 C CNN
+F 0 "#PWR051" H 7950 5550 50  0001 C CNN
 F 1 "GND" H 7955 5627 50  0000 C CNN
 F 2 "" H 7950 5800 50  0001 C CNN
@@
 $EndComp
 $Comp
-L power:GND #PWR043
+L power:GND #PWR042
 U 1 1 5AF5AB44
 P 3700 2950
-F 0 "#PWR043" H 3700 2700 50  0001 C CNN
+F 0 "#PWR042" H 3700 2700 50  0001 C CNN
 F 1 "GND" V 3705 2822 50  0000 R CNN
 F 2 "" H 3700 2950 50  0001 C CNN
@@
 $EndComp
 $Comp
-L power:GND #PWR042
+L power:GND #PWR041
 U 1 1 5AF5ABF2
 P 2700 2950
-F 0 "#PWR042" H 2700 2700 50  0001 C CNN
+F 0 "#PWR041" H 2700 2700 50  0001 C CNN
 F 1 "GND" V 2705 2822 50  0000 R CNN
 F 2 "" H 2700 2950 50  0001 C CNN
@@
 $EndComp
 $Comp
-L power:GND #PWR045
+L power:GND #PWR044
 U 1 1 5AF616AA
 P 1150 3750
-F 0 "#PWR045" H 1150 3500 50  0001 C CNN
+F 0 "#PWR044" H 1150 3500 50  0001 C CNN
 F 1 "GND" H 1155 3577 50  0000 C CNN
 F 2 "" H 1150 3750 50  0001 C CNN
@@
 	1150 4100 1450 4100
 $Comp
-L power:GND #PWR032
+L power:GND #PWR031
 U 1 1 5AF66D47
 P 5400 750
-F 0 "#PWR032" H 5400 500 50  0001 C CNN
+F 0 "#PWR031" H 5400 500 50  0001 C CNN
 F 1 "GND" H 5405 577 50  0000 C CNN
 F 2 "" H 5400 750 50  0001 C CNN
@@
 USB Isolation
 $Comp
-L power:GND #PWR035
+L power:GND #PWR034
 U 1 1 5AFE6191
 P 3000 1200
-F 0 "#PWR035" H 3000 950 50  0001 C CNN
+F 0 "#PWR034" H 3000 950 50  0001 C CNN
 F 1 "GND" V 3005 1072 50  0000 R CNN
 F 2 "" H 3000 1200 50  0001 C CNN
@@
 	1500 750  1500 950
 $Comp
-L power:GND #PWR034
+L power:GND #PWR033
 U 1 1 5AFC2033
 P 2450 1050
-F 0 "#PWR034" H 2450 800 50  0001 C CNN
+F 0 "#PWR033" H 2450 800 50  0001 C CNN
 F 1 "GND" V 2455 922 50  0000 R CNN
 F 2 "" H 2450 1050 50  0001 C CNN
@@
 $EndComp
 $Comp
-L power:GNDS #PWR033
+L power:GNDS #PWR032
 U 1 1 5AF88D47
 P 1100 1050
-F 0 "#PWR033" H 1100 800 50  0001 C CNN
+F 0 "#PWR032" H 1100 800 50  0001 C CNN
 F 1 "GNDS" V 1105 922 50  0000 R CNN
 F 2 "" H 1100 1050 50  0001 C CNN
@@
 Connection ~ 2050 2250
 $Comp
-L power:GND #PWR040
+L power:GND #PWR039
 U 1 1 5AF61872
 P 2050 2250
-F 0 "#PWR040" H 2050 2000 50  0001 C CNN
+F 0 "#PWR039" H 2050 2000 50  0001 C CNN
 F 1 "GND" H 2055 2077 50  0000 C CNN
 F 2 "" H 2050 2250 50  0001 C CNN
@@
 $EndComp
 $Comp
-L power:GNDS #PWR039
+L power:GNDS #PWR038
 U 1 1 5AF61805
 P 1650 2250
-F 0 "#PWR039" H 1650 2000 50  0001 C CNN
+F 0 "#PWR038" H 1650 2000 50  0001 C CNN
 F 1 "GNDS" H 1655 2077 50  0000 C CNN
 F 2 "" H 1650 2250 50  0001 C CNN
@@
 	6000 750  6000 900
 $Comp
-L power:GND #PWR054
+L power:GND #PWR053
 U 1 1 5AFDE2A1
 P 950 7450
-F 0 "#PWR054" H 950 7200 50  0001 C CNN
+F 0 "#PWR053" H 950 7200 50  0001 C CNN
 F 1 "GND" H 955 7277 50  0000 C CNN
 F 2 "" H 950 7450 50  0001 C CNN
@@
 P 1400 6450
 F 0 "R20" V 1550 6450 50  0000 L CNN
-F 1 "4.7k" V 1470 6405 50  0000 L CNN
+F 1 "1k" V 1470 6405 50  0000 L CNN
 F 2 "Resistor_SMD:R_0603_1608Metric" V 1330 6450 50  0001 C CNN
 F 3 "~" H 1400 6450 50  0001 C CNN
@@
 $EndComp
 $Comp
-L power:GND #PWR053
+L power:GND #PWR052
 U 1 1 5B010B0E
 P 2300 6450
-F 0 "#PWR053" H 2300 6200 50  0001 C CNN
+F 0 "#PWR052" H 2300 6200 50  0001 C CNN
 F 1 "GND" H 2305 6277 50  0000 C CNN
 F 2 "" H 2300 6450 50  0001 C CNN
@@
 NoConn ~ 8100 3250
 $Comp
-L power:GND #PWR036
+L power:GND #PWR035
 U 1 1 5B0EA618
 P 4150 1700
-F 0 "#PWR036" H 4150 1450 50  0001 C CNN
+F 0 "#PWR035" H 4150 1450 50  0001 C CNN
 F 1 "GND" H 4155 1527 50  0000 C CNN
 F 2 "" H 4150 1700 50  0001 C CNN
@@
 $EndComp
 $Comp
-L power:GND #PWR038
+L power:GND #PWR037
 U 1 1 5B3AC87D
 P 3850 2200
-F 0 "#PWR038" H 3850 1950 50  0001 C CNN
+F 0 "#PWR037" H 3850 1950 50  0001 C CNN
 F 1 "GND" H 3855 2027 50  0000 C CNN
 F 2 "" H 3850 2200 50  0001 C CNN

Commit message: Add a P MOSFET to protect the TPS54308
Since I fried two TPS54308 already, I think it would
be best to implement a reverse voltage protection
before the TPS that provides the 5V rail.

To reuse parts, I also switches the battery protection
P MOSFET to the same part.
Parts:
- Q6: renamed from Q5; value IRLML6401 -> PMV50EPEA
- renumbered D9 to D10, R12 to R13, R13 to R14, R14 to R15, R15 to R16, R16 to R17, R17 to R18, R18 to R19, R19 to R20, R20 to R21
Changed lines of the file:
@@
 $EndDescr
 $Comp
-L Device:R R12
+L Device:R R13
 U 1 1 5AD0B119
 P 5550 750
-F 0 "R12" V 5450 700 50  0000 L CNN
+F 0 "R13" V 5450 700 50  0000 L CNN
 F 1 "10k" V 5350 700 50  0000 L CNN
 F 2 "Resistor_SMD:R_0603_1608Metric" V 5480 750 50  0001 C CNN
@@
 $EndComp
 $Comp
-L Device:R R13
+L Device:R R14
 U 1 1 5AD0B198
 P 6300 750
-F 0 "R13" V 6400 650 50  0000 L CNN
+F 0 "R14" V 6400 650 50  0000 L CNN
 F 1 "10k" V 6500 650 50  0000 L CNN
 F 2 "Resistor_SMD:R_0603_1608Metric" V 6230 750 50  0001 C CNN
@@
 $EndComp
 $Comp
-L power:GND #PWR050
+L power:GND #PWR051
 U 1 1 5AF57331
 P 5300 5350
-F 0 "#PWR050" H 5300 5100 50  0001 C CNN
+F 0 "#PWR051" H 5300 5100 50  0001 C CNN
 F 1 "GND" H 5305 5177 50  0000 C CNN
 F 2 "" H 5300 5350 50  0001 C CNN
@@
 $EndComp
 $Comp
-L power:GND #PWR049
+L power:GND #PWR050
 U 1 1 5AF579EA
 P 3850 4750
-F 0 "#PWR049" H 3850 4500 50  0001 C CNN
+F 0 "#PWR050" H 3850 4500 50  0001 C CNN
 F 1 "GND" H 3855 4577 50  0000 C CNN
 F 2 "" H 3850 4750 50  0001 C CNN
@@
 $EndComp
 $Comp
-L power:GND #PWR048
+L power:GND #PWR049
 U 1 1 5AF580A3
 P 3450 4750
-F 0 "#PWR048" H 3450 4500 50  0001 C CNN
+F 0 "#PWR049" H 3450 4500 50  0001 C CNN
 F 1 "GND" H 3455 4577 50  0000 C CNN
 F 2 "" H 3450 4750 50  0001 C CNN
@@
 $EndComp
 $Comp
-L power:GND #PWR045
+L power:GND #PWR046
 U 1 1 5AF58792
 P 3450 4050
-F 0 "#PWR045" H 3450 3800 50  0001 C CNN
+F 0 "#PWR046" H 3450 3800 50  0001 C CNN
 F 1 "GND" H 3455 3877 50  0000 C CNN
 F 2 "" H 3450 4050 50  0001 C CNN
@@
 $EndComp
 $Comp
-L power:GND #PWR046
+L power:GND #PWR047
 U 1 1 5AF59C69
 P 3850 4050
-F 0 "#PWR046" H 3850 3800 50  0001 C CNN
+F 0 "#PWR047" H 3850 3800 50  0001 C CNN
 F 1 "GND" H 3855 3877 50  0000 C CNN
 F 2 "" H 3850 4050 50  0001 C CNN
@@
 $EndComp
 $Comp
-L power:GND #PWR043
+L power:GND #PWR044
 U 1 1 5AF5B126
 P 4900 3350
-F 0 "#PWR043" H 4900 3100 50  0001 C CNN
+F 0 "#PWR044" H 4900 3100 50  0001 C CNN
 F 1 "GND" V 4905 3222 50  0000 R CNN
 F 2 "" H 4900 3350 50  0001 C CNN
@@
 $EndComp
 $Comp
-L power:GND #PWR047
+L power:GND #PWR048
 U 1 1 5AF5BF00
 P 4900 4250
-F 0 "#PWR047" H 4900 4000 50  0001 C CNN
+F 0 "#PWR048" H 4900 4000 50  0001 C CNN
 F 1 "GND" V 4905 4122 50  0000 R CNN
 F 2 "" H 4900 4250 50  0001 C CNN
@@
 $EndComp
 $Comp
-L power:GND #PWR036
+L power:GND #PWR037
 U 1 1 5AF5CFF3
 P 5400 2050
-F 0 "#PWR036" H 5400 1800 50  0001 C CNN
+F 0 "#PWR037" H 5400 1800 50  0001 C CNN
 F 1 "GND" H 5405 1877 50  0000 C CNN
 F 2 "" H 5400 2050 50  0001 C CNN
@@
 $EndComp
 $Comp
-L power:GND #PWR040
+L power:GND #PWR041
 U 1 1 5AF5E7FC
 P 8750 2250
-F 0 "#PWR040" H 8750 2000 50  0001 C CNN
+F 0 "#PWR041" H 8750 2000 50  0001 C CNN
 F 1 "GND" H 8750 2100 50  0000 C CNN
 F 2 "" H 8750 2250 50  0001 C CNN
@@
 $EndComp
 $Comp
-L power:GND #PWR051
+L power:GND #PWR052
 U 1 1 5AF5F2E4
 P 7950 5800
-F 0 "#PWR051" H 7950 5550 50  0001 C CNN
+F 0 "#PWR052" H 7950 5550 50  0001 C CNN
 F 1 "GND" H 7955 5627 50  0000 C CNN
 F 2 "" H 7950 5800 50  0001 C CNN
@@
 $EndComp
 $Comp
-L power:GND #PWR042
+L power:GND #PWR043
 U 1 1 5AF5AB44
 P 3700 2950
-F 0 "#PWR042" H 3700 2700 50  0001 C CNN
+F 0 "#PWR043" H 3700 2700 50  0001 C CNN
 F 1 "GND" V 3705 2822 50  0000 R CNN
 F 2 "" H 3700 2950 50  0001 C CNN
@@
 $EndComp
 $Comp
-L power:GND #PWR041
+L power:GND #PWR042
 U 1 1 5AF5ABF2
 P 2700 2950
-F 0 "#PWR041" H 2700 2700 50  0001 C CNN
+F 0 "#PWR042" H 2700 2700 50  0001 C CNN
 F 1 "GND" V 2705 2822 50  0000 R CNN
 F 2 "" H 2700 2950 50  0001 C CNN
@@
 $EndComp
 $Comp
-L power:GND #PWR044
+L power:GND #PWR045
 U 1 1 5AF616AA
 P 1150 3750
-F 0 "#PWR044" H 1150 3500 50  0001 C CNN
+F 0 "#PWR045" H 1150 3500 50  0001 C CNN
 F 1 "GND" H 1155 3577 50  0000 C CNN
 F 2 "" H 1150 3750 50  0001 C CNN
@@
 	1150 4100 1450 4100
 $Comp
-L power:GND #PWR031
+L power:GND #PWR032
 U 1 1 5AF66D47
 P 5400 750
-F 0 "#PWR031" H 5400 500 50  0001 C CNN
+F 0 "#PWR032" H 5400 500 50  0001 C CNN
 F 1 "GND" H 5405 577 50  0000 C CNN
 F 2 "" H 5400 750 50  0001 C CNN
@@
 USB Isolation
 $Comp
-L power:GND #PWR034
+L power:GND #PWR035
 U 1 1 5AFE6191
 P 3000 1200
-F 0 "#PWR034" H 3000 950 50  0001 C CNN
+F 0 "#PWR035" H 3000 950 50  0001 C CNN
 F 1 "GND" V 3005 1072 50  0000 R CNN
 F 2 "" H 3000 1200 50  0001 C CNN
@@
 	1500 750  1500 950
 $Comp
-L power:GND #PWR033
+L power:GND #PWR034
 U 1 1 5AFC2033
 P 2450 1050
-F 0 "#PWR033" H 2450 800 50  0001 C CNN
+F 0 "#PWR034" H 2450 800 50  0001 C CNN
 F 1 "GND" V 2455 922 50  0000 R CNN
 F 2 "" H 2450 1050 50  0001 C CNN
@@
 $EndComp
 $Comp
-L power:GNDS #PWR032
+L power:GNDS #PWR033
 U 1 1 5AF88D47
 P 1100 1050
-F 0 "#PWR032" H 1100 800 50  0001 C CNN
+F 0 "#PWR033" H 1100 800 50  0001 C CNN
 F 1 "GNDS" V 1105 922 50  0000 R CNN
 F 2 "" H 1100 1050 50  0001 C CNN
@@
 $EndComp
 $Comp
-L Device:R R19
+L Device:R R20
 U 1 1 5AF72C01
 P 2500 1550
-F 0 "R19" V 2400 1650 50  0000 C CNN
+F 0 "R20" V 2400 1650 50  0000 C CNN
 F 1 "100" V 2400 1450 50  0000 C CNN
 F 2 "Resistor_SMD:R_0603_1608Metric" V 2430 1550 50  0001 C CNN
@@
 $EndComp
 $Comp
-L Device:R R17
+L Device:R R18
 U 1 1 5AF72BFA
 P 2500 1450
-F 0 "R17" V 2400 1350 50  0000 C CNN
+F 0 "R18" V 2400 1350 50  0000 C CNN
 F 1 "100" V 2400 1550 50  0000 C CNN
 F 2 "Resistor_SMD:R_0603_1608Metric" V 2430 1450 50  0001 C CNN
@@
 $EndComp
 $Comp
-L Device:R R18
+L Device:R R19
 U 1 1 5AF724F0
 P 1200 1550
-F 0 "R18" V 1050 1650 50  0000 C CNN
+F 0 "R19" V 1050 1650 50  0000 C CNN
 F 1 "100" V 1050 1450 50  0000 C CNN
 F 2 "Resistor_SMD:R_0603_1608Metric" V 1130 1550 50  0001 C CNN
@@
 $EndComp
 $Comp
-L Device:R R16
+L Device:R R17
 U 1 1 5AF72236
 P 1200 1450
-F 0 "R16" V 1100 1350 50  0000 C CNN
+F 0 "R17" V 1100 1350 50  0000 C CNN
 F 1 "100" V 1100 1550 50  0000 C CNN
 F 2 "Resistor_SMD:R_0603_1608Metric" V 1130 1450 50  0001 C CNN
@@
 Connection ~ 2050 2250
 $Comp
-L power:GND #PWR039
+L power:GND #PWR040
 U 1 1 5AF61872
 P 2050 2250
-F 0 "#PWR039" H 2050 2000 50  0001 C CNN
+F 0 "#PWR040" H 2050 2000 50  0001 C CNN
 F 1 "GND" H 2055 2077 50  0000 C CNN
 F 2 "" H 2050 2250 50  0001 C CNN
@@
 $EndComp
 $Comp
-L power:GNDS #PWR038
+L power:GNDS #PWR039
 U 1 1 5AF61805
 P 1650 2250
-F 0 "#PWR038" H 1650 2000 50  0001 C CNN
+F 0 "#PWR039" H 1650 2000 50  0001 C CNN
 F 1 "GNDS" H 1655 2077 50  0000 C CNN
 F 2 "" H 1650 2250 50  0001 C CNN
@@
 	2350 1250 2650 1250
 $Comp
-L Device:R R15
+L Device:R R16
 U 1 1 5AFBD0C4
 P 7350 1150
-F 0 "R15" H 7420 1196 50  0000 L CNN
+F 0 "R16" H 7420 1196 50  0000 L CNN
 F 1 "10k" H 7420 1105 50  0000 L CNN
 F 2 "Resistor_SMD:R_0603_1608Metric" V 7280 1150 50  0001 C CNN
@@
 	6000 750  6000 900
 $Comp
-L power:GND #PWR053
+L power:GND #PWR054
 U 1 1 5AFDE2A1
 P 950 7450
-F 0 "#PWR053" H 950 7200 50  0001 C CNN
+F 0 "#PWR054" H 950 7200 50  0001 C CNN
 F 1 "GND" H 955 7277 50  0000 C CNN
 F 2 "" H 950 7450 50  0001 C CNN
@@
 Connection ~ 7350 750
 $Comp
-L Device:R R14
+L Device:R R15
 U 1 1 5AFBD0BD
 P 7000 1150
-F 0 "R14" H 7070 1196 50  0000 L CNN
+F 0 "R15" H 7070 1196 50  0000 L CNN
 F 1 "10k" H 7070 1105 50  0000 L CNN
 F 2 "Resistor_SMD:R_0603_1608Metric" V 6930 1150 50  0001 C CNN
@@
 STATUS_LED
 $Comp
-L Device:LED D9
+L Device:LED D10
 U 1 1 5B007E50
 P 1700 6450
-F 0 "D9" H 1738 6332 50  0000 R CNN
+F 0 "D10" H 1738 6332 50  0000 R CNN
 F 1 "LTST-C194KSKT" H 2000 6600 50  0000 R CNN
 F 2 "LED_SMD:LED_0603_1608Metric" H 1700 6450 50  0001 C CNN
@@
 $EndComp
 $Comp
-L Device:R R20
+L Device:R R21
 U 1 1 5B007E5D
 P 1400 6450
-F 0 "R20" V 1550 6450 50  0000 L CNN
+F 0 "R21" V 1550 6450 50  0000 L CNN
 F 1 "1k" V 1470 6405 50  0000 L CNN
 F 2 "Resistor_SMD:R_0603_1608Metric" V 1330 6450 50  0001 C CNN
@@
 $EndComp
 $Comp
-L power:GND #PWR052
+L power:GND #PWR053
 U 1 1 5B010B0E
 P 2300 6450
-F 0 "#PWR052" H 2300 6200 50  0001 C CNN
+F 0 "#PWR053" H 2300 6200 50  0001 C CNN
 F 1 "GND" H 2305 6277 50  0000 C CNN
 F 2 "" H 2300 6450 50  0001 C CNN
@@
 NoConn ~ 8100 3250
 $Comp
-L power:GND #PWR035
+L power:GND #PWR036
 U 1 1 5B0EA618
 P 4150 1700
-F 0 "#PWR035" H 4150 1450 50  0001 C CNN
+F 0 "#PWR036" H 4150 1450 50  0001 C CNN
 F 1 "GND" H 4155 1527 50  0000 C CNN
 F 2 "" H 4150 1700 50  0001 C CNN
@@
 	4150 2950 4900 2950
 $Comp
-L Device:Q_PMOS_GSD Q5
+L Device:Q_PMOS_GSD Q6
 U 1 1 5B3AC772
 P 4050 2200
-F 0 "Q5" H 4255 2246 50  0000 L CNN
-F 1 "IRLML6401" H 4255 2155 50  0000 L CNN
+F 0 "Q6" H 4255 2246 50  0000 L CNN
+F 1 "PMV50EPEA" H 4255 2155 50  0000 L CNN
 F 2 "Package_TO_SOT_SMD:SOT-23" H 4250 2300 50  0001 C CNN
-F 3 "https://www.infineon.com/dgdl/irlml6401pbf.pdf?fileId=5546d462533600a401535668b96d2634" H 4050 2200 50  0001 C CNN
+F 3 "https://www.mouser.de/datasheet/2/916/PMV50EPEA-1320530.pdf" H 4050 2200 50  0001 C CNN
 	1    4050 2200
 	1    0    0    -1
 $EndComp
 $Comp
-L power:GND #PWR037
+L power:GND #PWR038
 U 1 1 5B3AC87D
 P 3850 2200
-F 0 "#PWR037" H 3850 1950 50  0001 C CNN
+F 0 "#PWR038" H 3850 1950 50  0001 C CNN
 F 1 "GND" H 3855 2027 50  0000 C CNN
 F 2 "" H 3850 2200 50  0001 C CNN

Commit message: Chang battery holder
This battery holder is more widely available.
Parts:
- BT1: footprint custom-footprints:VBH2032-1 -> custom-footprints:S8401-46
Changed lines of the file:
@@
 F 0 "BT1" H 4268 1896 50  0000 L CNN
 F 1 "VBH2032-1" H 4268 1805 50  0000 L CNN
-F 2 "custom-footprints:VBH2032-1" V 4150 1860 50  0001 C CNN
+F 2 "custom-footprints:S8401-46" V 4150 1860 50  0001 C CNN
 F 3 "https://www.mouser.de/datasheet/2/346/VBH2032-1_new-258024.pdf" V 4150 1860 50  0001 C CNN
 	1    4150 1800
