File: PCB/mosfets.sch (KiCad schematic (older format))
At the start: 16 parts, among them Q1 PSMN1R8-40YLC,115, Q2 BUK9840-55, Q3 PSMN1R8-40YLC,115, Q4 BUK9840-55

Commit message: Finished TMC2130 placement.
Motor sheets is now instanced. That way I simply could use
a KiCad plugin to duplicate the layout in Pcbnew.
Parts:
- Q1, Q3: footprint Package_TO_SOT_SMD:SOT-669_LFPAK_ThermalVias-2 -> custom-footprints:SOT-669_LFPAK_ThermalVias-1
Changed lines of the file:
@@
 F 0 "Q1" H 2387 1396 50  0000 L CNN
 F 1 "PSMN1R8-40YLC,115" H 2387 1305 50  0000 L CNN
-F 2 "Package_TO_SOT_SMD:SOT-669_LFPAK_ThermalVias-2" H 2200 1325 50  0001 L CIN
+F 2 "custom-footprints:SOT-669_LFPAK_ThermalVias-1" H 2200 1325 50  0001 L CIN
 F 3 "https://assets.nexperia.com/documents/data-sheet/PSMN1R8-40YLC.pdf" V 2000 1400 50  0001 L CNN
 	1    2000 1400
@@
 F 0 "Q3" H 2387 3046 50  0000 L CNN
 F 1 "PSMN1R8-40YLC,115" H 2387 2955 50  0000 L CNN
-F 2 "Package_TO_SOT_SMD:SOT-669_LFPAK_ThermalVias-2" H 2200 2975 50  0001 L CIN
+F 2 "custom-footprints:SOT-669_LFPAK_ThermalVias-1" H 2200 2975 50  0001 L CIN
 F 3 "https://assets.nexperia.com/documents/data-sheet/PSMN1R8-40YLC.pdf" V 2000 3050 50  0001 L CNN
 	1    2000 3050

Commit message: Reworked some traces for better layout.
This will also come in handy, when we add more external
connections (10 to 20pin external).
Parts:
- D5, D6, D7, D8: symbol Device:D_Schottky -> remram-rescue:D_Schottky-Device
- R10, R11, R4, R5, R6, R7, R8, R9: symbol Device:R -> remram-rescue:R-Device
Changed lines of the file:
@@
 VDD_BED
 $Comp
-L Device:D_Schottky D5
+L remram-rescue:D_Schottky-Device D5
 U 1 1 5B1A3271
 P 1750 950
@@
 PWM_HEAT
 $Comp
-L Device:R R4
+L remram-rescue:R-Device R4
 U 1 1 5B1AEA5D
 P 1300 1400
@@
 VDD_HEAT
 $Comp
-L Device:D_Schottky D7
+L remram-rescue:D_Schottky-Device D7
 U 1 1 5B1B03B6
 P 1750 2600
@@
 	2100 3500 2100 3350
 $Comp
-L Device:R R8
+L remram-rescue:R-Device R8
 U 1 1 5B1B03DE
 P 1300 3050
@@
 $EndComp
 $Comp
-L Device:R R5
+L remram-rescue:R-Device R5
 U 1 1 5B1FB287
 P 4150 1400
@@
 $EndComp
 $Comp
-L Device:R R9
+L remram-rescue:R-Device R9
 U 1 1 5B2008D0
 P 4150 3050
@@
 	1450 3050 1600 3050
 $Comp
-L Device:R R6
+L remram-rescue:R-Device R6
 U 1 1 5AF82135
 P 1750 1850
@@
 	1600 1400 1800 1400
 $Comp
-L Device:R R10
+L remram-rescue:R-Device R10
 U 1 1 5AF8339E
 P 1750 3500
@@
 	2100 3500 1900 3500
 $Comp
-L Device:R R7
+L remram-rescue:R-Device R7
 U 1 1 5AF83BB4
 P 4600 1850
@@
 Connection ~ 4350 1400
 $Comp
-L Device:R R11
+L remram-rescue:R-Device R11
 U 1 1 5AF880C0
 P 4650 3500
@@
 Connection ~ 4850 3500
 $Comp
-L Device:D_Schottky D6
+L remram-rescue:D_Schottky-Device D6
 U 1 1 5AFB8598
 P 4500 950
@@
 $EndComp
 $Comp
-L Device:D_Schottky D8
+L remram-rescue:D_Schottky-Device D8
 U 1 1 5AFBAFD7
 P 4500 2600

Commit message: Reworked some traces and labels.
Parts:
- renumbered D7 to D6, D6 to D7, Q3 to Q2, Q2 to Q3, R7 to R10, R8 to R5, R10 to R7, R5 to R8
Changed lines of the file:
@@
 	2100 1200 2100 950
 $Comp
-L power:GNDPWR #PWR028
+L power:GNDPWR #PWR027
 U 1 1 5B1B03AE
 P 2200 3500
-F 0 "#PWR028" H 2200 3300 50  0001 C CNN
+F 0 "#PWR027" H 2200 3300 50  0001 C CNN
 F 1 "GNDPWR" H 2200 3350 50  0000 C CNN
 F 2 "" H 2200 3450 50  0001 C CNN
@@
 VDD_HEAT
 $Comp
-L remram-rescue:D_Schottky-Device D7
+L remram-rescue:D_Schottky-Device D6
 U 1 1 5B1B03B6
 P 1750 2600
-F 0 "D7" H 1750 2816 50  0000 C CNN
+F 0 "D6" H 1750 2816 50  0000 C CNN
 F 1 "SK310A-TP" H 1750 2725 50  0000 C CNN
 F 2 "Diode_SMD:D_SMA" H 1750 2600 50  0001 C CNN
@@
 	1500 2600 1600 2600
 $Comp
-L remram-custom:PSMN1R8-40YLC,115 Q3
+L remram-custom:PSMN1R8-40YLC,115 Q2
 U 1 1 5B1B03C5
 P 2000 3050
-F 0 "Q3" H 2387 3046 50  0000 L CNN
+F 0 "Q2" H 2387 3046 50  0000 L CNN
 F 1 "PSMN1R8-40YLC,115" H 2387 2955 50  0000 L CNN
 F 2 "custom-footprints:SOT-669_LFPAK_ThermalVias-1" H 2200 2975 50  0001 L CIN
@@
 	2100 3500 2100 3350
 $Comp
-L remram-rescue:R-Device R8
+L remram-rescue:R-Device R5
 U 1 1 5B1B03DE
 P 1300 3050
-F 0 "R8" V 1093 3050 50  0000 C CNN
+F 0 "R5" V 1093 3050 50  0000 C CNN
 F 1 "100" V 1184 3050 50  0000 C CNN
 F 2 "Resistor_SMD:R_0603_1608Metric" V 1230 3050 50  0001 C CNN
@@
 Connection ~ 2100 2600
 $Comp
-L remram-custom:BUK9840-55 Q2
+L remram-custom:BUK9840-55 Q3
 U 1 1 5B1FB146
 P 4750 1400
-F 0 "Q2" H 4955 1446 50  0000 L CNN
+F 0 "Q3" H 4955 1446 50  0000 L CNN
 F 1 "BUK9840-55" H 4955 1355 50  0000 L CNN
 F 2 "Package_TO_SOT_SMD:SOT-223-3_TabPin2" H 4950 1325 50  0001 L CIN
@@
 $EndComp
 $Comp
-L remram-rescue:R-Device R5
+L remram-rescue:R-Device R8
 U 1 1 5B1FB287
 P 4150 1400
-F 0 "R5" V 3943 1400 50  0000 C CNN
+F 0 "R8" V 3943 1400 50  0000 C CNN
 F 1 "100" V 4034 1400 50  0000 C CNN
 F 2 "Resistor_SMD:R_0603_1608Metric" V 4080 1400 50  0001 C CNN
@@
 	3900 1400 4000 1400
 $Comp
-L power:GNDPWR #PWR027
+L power:GNDPWR #PWR028
 U 1 1 5B1FD93D
 P 4850 1850
-F 0 "#PWR027" H 4850 1650 50  0001 C CNN
+F 0 "#PWR028" H 4850 1650 50  0001 C CNN
 F 1 "GNDPWR" H 4850 1700 50  0000 C CNN
 F 2 "" H 4850 1800 50  0001 C CNN
@@
 	1600 1400 1800 1400
 $Comp
-L remram-rescue:R-Device R10
+L remram-rescue:R-Device R7
 U 1 1 5AF8339E
 P 1750 3500
-F 0 "R10" V 1543 3500 50  0000 C CNN
+F 0 "R7" V 1543 3500 50  0000 C CNN
 F 1 "100k" V 1634 3500 50  0000 C CNN
 F 2 "Resistor_SMD:R_0603_1608Metric" V 1680 3500 50  0001 C CNN
@@
 	2100 3500 1900 3500
 $Comp
-L remram-rescue:R-Device R7
+L remram-rescue:R-Device R10
 U 1 1 5AF83BB4
 P 4600 1850
-F 0 "R7" V 4393 1850 50  0000 C CNN
+F 0 "R10" V 4393 1850 50  0000 C CNN
 F 1 "100k" V 4484 1850 50  0000 C CNN
 F 2 "Resistor_SMD:R_0603_1608Metric" V 4530 1850 50  0001 C CNN
@@
 Connection ~ 4850 3500
 $Comp
-L remram-rescue:D_Schottky-Device D6
+L remram-rescue:D_Schottky-Device D7
 U 1 1 5AFB8598
 P 4500 950
-F 0 "D6" H 4450 1150 50  0000 L CNN
+F 0 "D7" H 4450 1150 50  0000 L CNN
 F 1 "BAT54GWJ" H 4350 1050 50  0000 L CNN
 F 2 "Diode_SMD:D_SOD-123" H 4500 950 50  0001 C CNN

Commit message: First draft of RemRam.
I added a 20 pin expansion connector with the following pins:
 - SPI
 - I2C
 - USART
 - 4x PWM
 - 4x GPIO
Parts:
- renumbered D7 to D6, D6 to D7, Q3 to Q2, Q2 to Q3, R7 to R10, R8 to R5, R10 to R7, R5 to R8
Changed lines of the file:
@@
 	2100 1200 2100 950
 $Comp
-L power:GNDPWR #PWR027
+L power:GNDPWR #PWR028
 U 1 1 5B1B03AE
 P 2200 3500
-F 0 "#PWR027" H 2200 3300 50  0001 C CNN
+F 0 "#PWR028" H 2200 3300 50  0001 C CNN
 F 1 "GNDPWR" H 2200 3350 50  0000 C CNN
 F 2 "" H 2200 3450 50  0001 C CNN
@@
 VDD_HEAT
 $Comp
-L remram-rescue:D_Schottky-Device D6
+L remram-rescue:D_Schottky-Device D7
 U 1 1 5B1B03B6
 P 1750 2600
-F 0 "D6" H 1750 2816 50  0000 C CNN
+F 0 "D7" H 1750 2816 50  0000 C CNN
 F 1 "SK310A-TP" H 1750 2725 50  0000 C CNN
 F 2 "Diode_SMD:D_SMA" H 1750 2600 50  0001 C CNN
@@
 	1500 2600 1600 2600
 $Comp
-L remram-custom:PSMN1R8-40YLC,115 Q2
+L remram-custom:PSMN1R8-40YLC,115 Q3
 U 1 1 5B1B03C5
 P 2000 3050
-F 0 "Q2" H 2387 3046 50  0000 L CNN
+F 0 "Q3" H 2387 3046 50  0000 L CNN
 F 1 "PSMN1R8-40YLC,115" H 2387 2955 50  0000 L CNN
 F 2 "custom-footprints:SOT-669_LFPAK_ThermalVias-1" H 2200 2975 50  0001 L CIN
@@
 	2100 3500 2100 3350
 $Comp
-L remram-rescue:R-Device R5
+L remram-rescue:R-Device R8
 U 1 1 5B1B03DE
 P 1300 3050
-F 0 "R5" V 1093 3050 50  0000 C CNN
+F 0 "R8" V 1093 3050 50  0000 C CNN
 F 1 "100" V 1184 3050 50  0000 C CNN
 F 2 "Resistor_SMD:R_0603_1608Metric" V 1230 3050 50  0001 C CNN
@@
 Connection ~ 2100 2600
 $Comp
-L remram-custom:BUK9840-55 Q3
+L remram-custom:BUK9840-55 Q2
 U 1 1 5B1FB146
 P 4750 1400
-F 0 "Q3" H 4955 1446 50  0000 L CNN
+F 0 "Q2" H 4955 1446 50  0000 L CNN
 F 1 "BUK9840-55" H 4955 1355 50  0000 L CNN
 F 2 "Package_TO_SOT_SMD:SOT-223-3_TabPin2" H 4950 1325 50  0001 L CIN
@@
 $EndComp
 $Comp
-L remram-rescue:R-Device R8
+L remram-rescue:R-Device R5
 U 1 1 5B1FB287
 P 4150 1400
-F 0 "R8" V 3943 1400 50  0000 C CNN
+F 0 "R5" V 3943 1400 50  0000 C CNN
 F 1 "100" V 4034 1400 50  0000 C CNN
 F 2 "Resistor_SMD:R_0603_1608Metric" V 4080 1400 50  0001 C CNN
@@
 	3900 1400 4000 1400
 $Comp
-L power:GNDPWR #PWR028
+L power:GNDPWR #PWR027
 U 1 1 5B1FD93D
 P 4850 1850
-F 0 "#PWR028" H 4850 1650 50  0001 C CNN
+F 0 "#PWR027" H 4850 1650 50  0001 C CNN
 F 1 "GNDPWR" H 4850 1700 50  0000 C CNN
 F 2 "" H 4850 1800 50  0001 C CNN
@@
 	1600 1400 1800 1400
 $Comp
-L remram-rescue:R-Device R7
+L remram-rescue:R-Device R10
 U 1 1 5AF8339E
 P 1750 3500
-F 0 "R7" V 1543 3500 50  0000 C CNN
+F 0 "R10" V 1543 3500 50  0000 C CNN
 F 1 "100k" V 1634 3500 50  0000 C CNN
 F 2 "Resistor_SMD:R_0603_1608Metric" V 1680 3500 50  0001 C CNN
@@
 	2100 3500 1900 3500
 $Comp
-L remram-rescue:R-Device R10
+L remram-rescue:R-Device R7
 U 1 1 5AF83BB4
 P 4600 1850
-F 0 "R10" V 4393 1850 50  0000 C CNN
+F 0 "R7" V 4393 1850 50  0000 C CNN
 F 1 "100k" V 4484 1850 50  0000 C CNN
 F 2 "Resistor_SMD:R_0603_1608Metric" V 4530 1850 50  0001 C CNN
@@
 Connection ~ 4850 3500
 $Comp
-L remram-rescue:D_Schottky-Device D7
+L remram-rescue:D_Schottky-Device D6
 U 1 1 5AFB8598
 P 4500 950
-F 0 "D7" H 4450 1150 50  0000 L CNN
+F 0 "D6" H 4450 1150 50  0000 L CNN
 F 1 "BAT54GWJ" H 4350 1050 50  0000 L CNN
 F 2 "Diode_SMD:D_SOD-123" H 4500 950 50  0001 C CNN

Commit message: v0.2 of PCB.
After some feedback, we changed following:
 - Switched FAN VDD from 24 to 5V.
 - FAN now have a ADC pin for speed sensing.
 - Expanded EXP-3 connector to 26 pin
   - Included 24V VDD.
   - Could be used to connect up to two
     extra stepper.
 - Removed GND connections on TMC2130 to
   middel GND plane.
Connections:
- net labels added: VDD5V
- net labels removed: VDD_PWR
Changed lines of the file:
@@
 	1600 3050 1800 3050
 Text GLabel 4250 950  0    50   Input ~ 0
-VDD_PWR
+VDD5V
 Text GLabel 4250 2600 0    50   Input ~ 0
-VDD_PWR
+VDD5V
 $EndSCHEMATC

Commit message: Changed LED to sane values. Updated diodes. v0.5.
Parts:
- D5, D7: value SK310A-TP -> SK310A-LTP
Changed lines of the file:
@@
 P 1750 950
 F 0 "D5" H 1750 1166 50  0000 C CNN
-F 1 "SK310A-TP" H 1750 1075 50  0000 C CNN
+F 1 "SK310A-LTP" H 1750 1075 50  0000 C CNN
 F 2 "Diode_SMD:D_SMA" H 1750 950 50  0001 C CNN
 F 3 "https://www.mouser.de/ProductDetail/Micro-Commercial-Components-MCC/SK310A-TP?qs=O2qRfqcg9D9SKx4%252bV6P4XQ%3D%3D" H 1750 950 50  0001 C CNN
@@
 P 1750 2600
 F 0 "D7" H 1750 2816 50  0000 C CNN
-F 1 "SK310A-TP" H 1750 2725 50  0000 C CNN
+F 1 "SK310A-LTP" H 1750 2725 50  0000 C CNN
 F 2 "Diode_SMD:D_SMA" H 1750 2600 50  0001 C CNN
 F 3 "https://www.mouser.de/ProductDetail/Micro-Commercial-Components-MCC/SK310A-TP?qs=O2qRfqcg9D9SKx4%252bV6P4XQ%3D%3D" H 1750 2600 50  0001 C CNN

Commit message: Version 0.7
Parts:
- Q1, Q3: value PSMN1R8-40YLC,115 -> PSMN1R2-30YLC,115
Changed lines of the file:
@@
 P 2000 1400
 F 0 "Q1" H 2387 1396 50  0000 L CNN
-F 1 "PSMN1R8-40YLC,115" H 2387 1305 50  0000 L CNN
+F 1 "PSMN1R2-30YLC,115" H 2387 1305 50  0000 L CNN
 F 2 "custom-footprints:SOT-669_LFPAK_ThermalVias-1" H 2200 1325 50  0001 L CIN
-F 3 "https://assets.nexperia.com/documents/data-sheet/PSMN1R8-40YLC.pdf" V 2000 1400 50  0001 L CNN
+F 3 "https://assets.nexperia.com/documents/data-sheet/PSMN1R2-30YLC.pdf" V 2000 1400 50  0001 L CNN
 	1    2000 1400
 	1    0    0    -1
@@
 P 2000 3050
 F 0 "Q3" H 2387 3046 50  0000 L CNN
-F 1 "PSMN1R8-40YLC,115" H 2387 2955 50  0000 L CNN
+F 1 "PSMN1R2-30YLC,115" H 2387 2955 50  0000 L CNN
 F 2 "custom-footprints:SOT-669_LFPAK_ThermalVias-1" H 2200 2975 50  0001 L CIN
-F 3 "https://assets.nexperia.com/documents/data-sheet/PSMN1R8-40YLC.pdf" V 2000 3050 50  0001 L CNN
+F 3 "https://assets.nexperia.com/documents/data-sheet/PSMN1R2-30YLC.pdf" V 2000 3050 50  0001 L CNN
 	1    2000 3050
 	1    0    0    -1
