File: PCB/mosfets.sch (KiCad schematic (older format))
At the start: 16 parts, among them Q1 PSMN1R2-30YLC,115, Q2 BUK9840-55, Q3 PSMN1R2-30YLC,115, Q4 BUK9840-55

Commit message: Change 1k resistors to 4.7k. Update Symbols
Had to update the symbols to the right library again, since
Kicad Nightly changed their library order.

Also changed the 1k resistors to 4.7k to unify resistors and
also upped the PU to a weaker value.
Parts:
- D5, D6, D7, D8: symbol remram-rescue:D_Schottky-Device -> Device:D_Schottky
- R10, R11, R4, R5, R6, R7, R8, R9: symbol remram-rescue:R-Device -> Device:R
Changed lines of the file:
@@
 VDD_BED
 $Comp
-L remram-rescue:D_Schottky-Device D5
+L Device:D_Schottky D5
 U 1 1 5B1A3271
 P 1750 950
@@
 PWM_HEAT
 $Comp
-L remram-rescue:R-Device R4
+L Device:R R4
 U 1 1 5B1AEA5D
 P 1300 1400
@@
 VDD_HEAT
 $Comp
-L remram-rescue:D_Schottky-Device D7
+L Device:D_Schottky D7
 U 1 1 5B1B03B6
 P 1750 2600
@@
 	2100 3500 2100 3350
 $Comp
-L remram-rescue:R-Device R8
+L Device:R R8
 U 1 1 5B1B03DE
 P 1300 3050
@@
 $EndComp
 $Comp
-L remram-rescue:R-Device R5
+L Device:R R5
 U 1 1 5B1FB287
 P 4150 1400
@@
 $EndComp
 $Comp
-L remram-rescue:R-Device R9
+L Device:R R9
 U 1 1 5B2008D0
 P 4150 3050
@@
 	1450 3050 1600 3050
 $Comp
-L remram-rescue:R-Device R6
+L Device:R R6
 U 1 1 5AF82135
 P 1750 1850
@@
 	1600 1400 1800 1400
 $Comp
-L remram-rescue:R-Device R10
+L Device:R R10
 U 1 1 5AF8339E
 P 1750 3500
@@
 	2100 3500 1900 3500
 $Comp
-L remram-rescue:R-Device R7
+L Device:R R7
 U 1 1 5AF83BB4
 P 4600 1850
@@
 Connection ~ 4350 1400
 $Comp
-L remram-rescue:R-Device R11
+L Device:R R11
 U 1 1 5AF880C0
 P 4650 3500
@@
 Connection ~ 4850 3500
 $Comp
-L remram-rescue:D_Schottky-Device D6
+L Device:D_Schottky D6
 U 1 1 5AFB8598
 P 4500 950
@@
 $EndComp
 $Comp
-L remram-rescue:D_Schottky-Device D8
+L Device:D_Schottky D8
 U 1 1 5AFBAFD7
 P 4500 2600

Commit message: Add a P MOSFET to protect the TPS54308
Since I fried two TPS54308 already, I think it would
be best to implement a reverse voltage protection
before the TPS that provides the 5V rail.

To reuse parts, I also switches the battery protection
P MOSFET to the same part.
Parts:
- renumbered D5 to D6, D6 to D7, D7 to D8, D8 to D9, Q1 to Q2, Q2 to Q3, Q3 to Q4, Q4 to Q5, R9 to R10, R10 to R11, R11 to R12, R4 to R5, R5 to R6, R6 to R7, R7 to R8, R8 to R9
Changed lines of the file:
@@
 Fans
 $Comp
-L power:GNDPWR #PWR027
+L power:GNDPWR #PWR028
 U 1 1 5B1A30B2
 P 2200 1850
-F 0 "#PWR027" H 2200 1650 50  0001 C CNN
+F 0 "#PWR028" H 2200 1650 50  0001 C CNN
 F 1 "GNDPWR" H 2200 1700 50  0000 C CNN
 F 2 "" H 2200 1800 50  0001 C CNN
@@
 VDD_BED
 $Comp
-L Device:D_Schottky D5
+L Device:D_Schottky D6
 U 1 1 5B1A3271
 P 1750 950
-F 0 "D5" H 1750 1166 50  0000 C CNN
+F 0 "D6" H 1750 1166 50  0000 C CNN
 F 1 "SK310A-LTP" H 1750 1075 50  0000 C CNN
 F 2 "Diode_SMD:D_SMA" H 1750 950 50  0001 C CNN
@@
 	1500 950  1600 950
 $Comp
-L remram-custom:PSMN1R8-40YLC,115 Q1
+L remram-custom:PSMN1R8-40YLC,115 Q2
 U 1 1 5B1A764D
 P 2000 1400
-F 0 "Q1" H 2387 1396 50  0000 L CNN
+F 0 "Q2" H 2387 1396 50  0000 L CNN
 F 1 "PSMN1R2-30YLC,115" H 2387 1305 50  0000 L CNN
 F 2 "custom-footprints:SOT-669_LFPAK_ThermalVias-1" H 2200 1325 50  0001 L CIN
@@
 PWM_HEAT
 $Comp
-L Device:R R4
+L Device:R R5
 U 1 1 5B1AEA5D
 P 1300 1400
-F 0 "R4" V 1093 1400 50  0000 C CNN
+F 0 "R5" V 1093 1400 50  0000 C CNN
 F 1 "100" V 1184 1400 50  0000 C CNN
 F 2 "Resistor_SMD:R_0603_1608Metric" V 1230 1400 50  0001 C CNN
@@
 	2100 1200 2100 950
 $Comp
-L power:GNDPWR #PWR029
+L power:GNDPWR #PWR030
 U 1 1 5B1B03AE
 P 2200 3500
-F 0 "#PWR029" H 2200 3300 50  0001 C CNN
+F 0 "#PWR030" H 2200 3300 50  0001 C CNN
 F 1 "GNDPWR" H 2200 3350 50  0000 C CNN
 F 2 "" H 2200 3450 50  0001 C CNN
@@
 VDD_HEAT
 $Comp
-L Device:D_Schottky D7
+L Device:D_Schottky D8
 U 1 1 5B1B03B6
 P 1750 2600
-F 0 "D7" H 1750 2816 50  0000 C CNN
+F 0 "D8" H 1750 2816 50  0000 C CNN
 F 1 "SK310A-LTP" H 1750 2725 50  0000 C CNN
 F 2 "Diode_SMD:D_SMA" H 1750 2600 50  0001 C CNN
@@
 	1500 2600 1600 2600
 $Comp
-L remram-custom:PSMN1R8-40YLC,115 Q3
+L remram-custom:PSMN1R8-40YLC,115 Q4
 U 1 1 5B1B03C5
 P 2000 3050
-F 0 "Q3" H 2387 3046 50  0000 L CNN
+F 0 "Q4" H 2387 3046 50  0000 L CNN
 F 1 "PSMN1R2-30YLC,115" H 2387 2955 50  0000 L CNN
 F 2 "custom-footprints:SOT-669_LFPAK_ThermalVias-1" H 2200 2975 50  0001 L CIN
@@
 	2100 3500 2100 3350
 $Comp
-L Device:R R8
+L Device:R R9
 U 1 1 5B1B03DE
 P 1300 3050
-F 0 "R8" V 1093 3050 50  0000 C CNN
+F 0 "R9" V 1093 3050 50  0000 C CNN
 F 1 "100" V 1184 3050 50  0000 C CNN
 F 2 "Resistor_SMD:R_0603_1608Metric" V 1230 3050 50  0001 C CNN
@@
 Connection ~ 2100 2600
 $Comp
-L remram-custom:BUK9840-55 Q2
+L remram-custom:BUK9840-55 Q3
 U 1 1 5B1FB146
 P 4750 1400
-F 0 "Q2" H 4955 1446 50  0000 L CNN
+F 0 "Q3" H 4955 1446 50  0000 L CNN
 F 1 "BUK9840-55" H 4955 1355 50  0000 L CNN
 F 2 "Package_TO_SOT_SMD:SOT-223-3_TabPin2" H 4950 1325 50  0001 L CIN
@@
 $EndComp
 $Comp
-L Device:R R5
+L Device:R R6
 U 1 1 5B1FB287
 P 4150 1400
-F 0 "R5" V 3943 1400 50  0000 C CNN
+F 0 "R6" V 3943 1400 50  0000 C CNN
 F 1 "100" V 4034 1400 50  0000 C CNN
 F 2 "Resistor_SMD:R_0603_1608Metric" V 4080 1400 50  0001 C CNN
@@
 	3900 1400 4000 1400
 $Comp
-L power:GNDPWR #PWR028
+L power:GNDPWR #PWR029
 U 1 1 5B1FD93D
 P 4850 1850
-F 0 "#PWR028" H 4850 1650 50  0001 C CNN
+F 0 "#PWR029" H 4850 1650 50  0001 C CNN
 F 1 "GNDPWR" H 4850 1700 50  0000 C CNN
 F 2 "" H 4850 1800 50  0001 C CNN
@@
 	4850 1600 4850 1850
 $Comp
-L remram-custom:BUK9840-55 Q4
+L remram-custom:BUK9840-55 Q5
 U 1 1 5B2008C9
 P 4750 3050
-F 0 "Q4" H 4955 3096 50  0000 L CNN
+F 0 "Q5" H 4955 3096 50  0000 L CNN
 F 1 "BUK9840-55" H 4955 3005 50  0000 L CNN
 F 2 "Package_TO_SOT_SMD:SOT-223-3_TabPin2" H 4950 2975 50  0001 L CIN
@@
 $EndComp
 $Comp
-L Device:R R9
+L Device:R R10
 U 1 1 5B2008D0
 P 4150 3050
-F 0 "R9" V 3943 3050 50  0000 C CNN
+F 0 "R10" V 3943 3050 50  0000 C CNN
 F 1 "100" V 4034 3050 50  0000 C CNN
 F 2 "Resistor_SMD:R_0603_1608Metric" V 4080 3050 50  0001 C CNN
@@
 	3900 3050 4000 3050
 $Comp
-L power:GNDPWR #PWR030
+L power:GNDPWR #PWR031
 U 1 1 5B2008E5
 P 4850 3500
-F 0 "#PWR030" H 4850 3300 50  0001 C CNN
+F 0 "#PWR031" H 4850 3300 50  0001 C CNN
 F 1 "GNDPWR" H 4850 3350 50  0000 C CNN
 F 2 "" H 4850 3450 50  0001 C CNN
@@
 	1450 3050 1600 3050
 $Comp
-L Device:R R6
+L Device:R R7
 U 1 1 5AF82135
 P 1750 1850
-F 0 "R6" V 1543 1850 50  0000 C CNN
+F 0 "R7" V 1543 1850 50  0000 C CNN
 F 1 "100k" V 1634 1850 50  0000 C CNN
 F 2 "Resistor_SMD:R_0603_1608Metric" V 1680 1850 50  0001 C CNN
@@
 	1600 1400 1800 1400
 $Comp
-L Device:R R10
+L Device:R R11
 U 1 1 5AF8339E
 P 1750 3500
-F 0 "R10" V 1543 3500 50  0000 C CNN
+F 0 "R11" V 1543 3500 50  0000 C CNN
 F 1 "100k" V 1634 3500 50  0000 C CNN
 F 2 "Resistor_SMD:R_0603_1608Metric" V 1680 3500 50  0001 C CNN
@@
 	2100 3500 1900 3500
 $Comp
-L Device:R R7
+L Device:R R8
 U 1 1 5AF83BB4
 P 4600 1850
-F 0 "R7" V 4393 1850 50  0000 C CNN
+F 0 "R8" V 4393 1850 50  0000 C CNN
 F 1 "100k" V 4484 1850 50  0000 C CNN
 F 2 "Resistor_SMD:R_0603_1608Metric" V 4530 1850 50  0001 C CNN
@@
 Connection ~ 4350 1400
 $Comp
-L Device:R R11
+L Device:R R12
 U 1 1 5AF880C0
 P 4650 3500
-F 0 "R11" V 4443 3500 50  0000 C CNN
+F 0 "R12" V 4443 3500 50  0000 C CNN
 F 1 "100k" V 4534 3500 50  0000 C CNN
 F 2 "Resistor_SMD:R_0603_1608Metric" V 4580 3500 50  0001 C CNN
@@
 Connection ~ 4850 3500
 $Comp
-L Device:D_Schottky D6
+L Device:D_Schottky D7
 U 1 1 5AFB8598
 P 4500 950
-F 0 "D6" H 4450 1150 50  0000 L CNN
+F 0 "D7" H 4450 1150 50  0000 L CNN
 F 1 "BAT54GWJ" H 4350 1050 50  0000 L CNN
 F 2 "Diode_SMD:D_SOD-123" H 4500 950 50  0001 C CNN
@@
 $EndComp
 $Comp
-L Device:D_Schottky D8
+L Device:D_Schottky D9
 U 1 1 5AFBAFD7
 P 4500 2600
-F 0 "D8" H 4450 2800 50  0000 L CNN
+F 0 "D9" H 4450 2800 50  0000 L CNN
 F 1 "BAT54GWJ" H 4350 2700 50  0000 L CNN
 F 2 "Diode_SMD:D_SOD-123" H 4500 2600 50  0001 C CNN

Commit message: Add compability for TPS54302
Since the TPS54308 is often not available, we added the
option to also use the TPS54038. This commit added a lot
of components and changed the CSV.
Parts:
- renumbered D6 to D5, D7 to D6, D8 to D7, D9 to D8, Q2 to Q1, Q3 to Q2, Q4 to Q3, Q5 to Q4, R7 to R10, R8 to R11, R9 to R12, R10 to R13, R11 to R14, R12 to R15, R5 to R8, R6 to R9
Changed lines of the file:
@@
 VDD_BED
 $Comp
-L Device:D_Schottky D6
+L Device:D_Schottky D5
 U 1 1 5B1A3271
 P 1750 950
-F 0 "D6" H 1750 1166 50  0000 C CNN
+F 0 "D5" H 1750 1166 50  0000 C CNN
 F 1 "SK310A-LTP" H 1750 1075 50  0000 C CNN
 F 2 "Diode_SMD:D_SMA" H 1750 950 50  0001 C CNN
@@
 	1500 950  1600 950
 $Comp
-L remram-custom:PSMN1R8-40YLC,115 Q2
+L remram-custom:PSMN1R8-40YLC,115 Q1
 U 1 1 5B1A764D
 P 2000 1400
-F 0 "Q2" H 2387 1396 50  0000 L CNN
+F 0 "Q1" H 2387 1396 50  0000 L CNN
 F 1 "PSMN1R2-30YLC,115" H 2387 1305 50  0000 L CNN
 F 2 "custom-footprints:SOT-669_LFPAK_ThermalVias-1" H 2200 1325 50  0001 L CIN
@@
 PWM_HEAT
 $Comp
-L Device:R R5
+L Device:R R8
 U 1 1 5B1AEA5D
 P 1300 1400
-F 0 "R5" V 1093 1400 50  0000 C CNN
+F 0 "R8" V 1093 1400 50  0000 C CNN
 F 1 "100" V 1184 1400 50  0000 C CNN
 F 2 "Resistor_SMD:R_0603_1608Metric" V 1230 1400 50  0001 C CNN
@@
 VDD_HEAT
 $Comp
-L Device:D_Schottky D8
+L Device:D_Schottky D7
 U 1 1 5B1B03B6
 P 1750 2600
-F 0 "D8" H 1750 2816 50  0000 C CNN
+F 0 "D7" H 1750 2816 50  0000 C CNN
 F 1 "SK310A-LTP" H 1750 2725 50  0000 C CNN
 F 2 "Diode_SMD:D_SMA" H 1750 2600 50  0001 C CNN
@@
 	1500 2600 1600 2600
 $Comp
-L remram-custom:PSMN1R8-40YLC,115 Q4
+L remram-custom:PSMN1R8-40YLC,115 Q3
 U 1 1 5B1B03C5
 P 2000 3050
-F 0 "Q4" H 2387 3046 50  0000 L CNN
+F 0 "Q3" H 2387 3046 50  0000 L CNN
 F 1 "PSMN1R2-30YLC,115" H 2387 2955 50  0000 L CNN
 F 2 "custom-footprints:SOT-669_LFPAK_ThermalVias-1" H 2200 2975 50  0001 L CIN
@@
 	2100 3500 2100 3350
 $Comp
-L Device:R R9
+L Device:R R12
 U 1 1 5B1B03DE
 P 1300 3050
-F 0 "R9" V 1093 3050 50  0000 C CNN
+F 0 "R12" V 1093 3050 50  0000 C CNN
 F 1 "100" V 1184 3050 50  0000 C CNN
 F 2 "Resistor_SMD:R_0603_1608Metric" V 1230 3050 50  0001 C CNN
@@
 Connection ~ 2100 2600
 $Comp
-L remram-custom:BUK9840-55 Q3
+L remram-custom:BUK9840-55 Q2
 U 1 1 5B1FB146
 P 4750 1400
-F 0 "Q3" H 4955 1446 50  0000 L CNN
+F 0 "Q2" H 4955 1446 50  0000 L CNN
 F 1 "BUK9840-55" H 4955 1355 50  0000 L CNN
 F 2 "Package_TO_SOT_SMD:SOT-223-3_TabPin2" H 4950 1325 50  0001 L CIN
@@
 $EndComp
 $Comp
-L Device:R R6
+L Device:R R9
 U 1 1 5B1FB287
 P 4150 1400
-F 0 "R6" V 3943 1400 50  0000 C CNN
+F 0 "R9" V 3943 1400 50  0000 C CNN
 F 1 "100" V 4034 1400 50  0000 C CNN
 F 2 "Resistor_SMD:R_0603_1608Metric" V 4080 1400 50  0001 C CNN
@@
 	4850 1600 4850 1850
 $Comp
-L remram-custom:BUK9840-55 Q5
+L remram-custom:BUK9840-55 Q4
 U 1 1 5B2008C9
 P 4750 3050
-F 0 "Q5" H 4955 3096 50  0000 L CNN
+F 0 "Q4" H 4955 3096 50  0000 L CNN
 F 1 "BUK9840-55" H 4955 3005 50  0000 L CNN
 F 2 "Package_TO_SOT_SMD:SOT-223-3_TabPin2" H 4950 2975 50  0001 L CIN
@@
 $EndComp
 $Comp
-L Device:R R10
+L Device:R R13
 U 1 1 5B2008D0
 P 4150 3050
-F 0 "R10" V 3943 3050 50  0000 C CNN
+F 0 "R13" V 3943 3050 50  0000 C CNN
 F 1 "100" V 4034 3050 50  0000 C CNN
 F 2 "Resistor_SMD:R_0603_1608Metric" V 4080 3050 50  0001 C CNN
@@
 	1450 3050 1600 3050
 $Comp
-L Device:R R7
+L Device:R R10
 U 1 1 5AF82135
 P 1750 1850
-F 0 "R7" V 1543 1850 50  0000 C CNN
+F 0 "R10" V 1543 1850 50  0000 C CNN
 F 1 "100k" V 1634 1850 50  0000 C CNN
 F 2 "Resistor_SMD:R_0603_1608Metric" V 1680 1850 50  0001 C CNN
@@
 	1600 1400 1800 1400
 $Comp
-L Device:R R11
+L Device:R R14
 U 1 1 5AF8339E
 P 1750 3500
-F 0 "R11" V 1543 3500 50  0000 C CNN
+F 0 "R14" V 1543 3500 50  0000 C CNN
 F 1 "100k" V 1634 3500 50  0000 C CNN
 F 2 "Resistor_SMD:R_0603_1608Metric" V 1680 3500 50  0001 C CNN
@@
 	2100 3500 1900 3500
 $Comp
-L Device:R R8
+L Device:R R11
 U 1 1 5AF83BB4
 P 4600 1850
-F 0 "R8" V 4393 1850 50  0000 C CNN
+F 0 "R11" V 4393 1850 50  0000 C CNN
 F 1 "100k" V 4484 1850 50  0000 C CNN
 F 2 "Resistor_SMD:R_0603_1608Metric" V 4530 1850 50  0001 C CNN
@@
 Connection ~ 4350 1400
 $Comp
-L Device:R R12
+L Device:R R15
 U 1 1 5AF880C0
 P 4650 3500
-F 0 "R12" V 4443 3500 50  0000 C CNN
+F 0 "R15" V 4443 3500 50  0000 C CNN
 F 1 "100k" V 4534 3500 50  0000 C CNN
 F 2 "Resistor_SMD:R_0603_1608Metric" V 4580 3500 50  0001 C CNN
@@
 Connection ~ 4850 3500
 $Comp
-L Device:D_Schottky D7
+L Device:D_Schottky D6
 U 1 1 5AFB8598
 P 4500 950
-F 0 "D7" H 4450 1150 50  0000 L CNN
+F 0 "D6" H 4450 1150 50  0000 L CNN
 F 1 "BAT54GWJ" H 4350 1050 50  0000 L CNN
 F 2 "Diode_SMD:D_SOD-123" H 4500 950 50  0001 C CNN
@@
 $EndComp
 $Comp
-L Device:D_Schottky D9
+L Device:D_Schottky D8
 U 1 1 5AFBAFD7
 P 4500 2600
-F 0 "D9" H 4450 2800 50  0000 L CNN
+F 0 "D8" H 4450 2800 50  0000 L CNN
 F 1 "BAT54GWJ" H 4350 2700 50  0000 L CNN
 F 2 "Diode_SMD:D_SOD-123" H 4500 2600 50  0001 C CNN

Commit message: New item designations and fixes some small manufacturing issues
Parts:
- renumbered D7 to D6, D6 to D7, Q3 to Q2, Q2 to Q3, R14 to R11, R9 to R12, R11 to R14, R12 to R9
Changed lines of the file:
@@
 Fans
 $Comp
-L power:GNDPWR #PWR028
+L power:GNDPWR #PWR031
 U 1 1 5B1A30B2
 P 2200 1850
-F 0 "#PWR028" H 2200 1650 50  0001 C CNN
+F 0 "#PWR031" H 2200 1650 50  0001 C CNN
 F 1 "GNDPWR" H 2200 1700 50  0000 C CNN
 F 2 "" H 2200 1800 50  0001 C CNN
@@
 	2100 1200 2100 950
 $Comp
-L power:GNDPWR #PWR030
+L power:GNDPWR #PWR032
 U 1 1 5B1B03AE
 P 2200 3500
-F 0 "#PWR030" H 2200 3300 50  0001 C CNN
+F 0 "#PWR032" H 2200 3300 50  0001 C CNN
 F 1 "GNDPWR" H 2200 3350 50  0000 C CNN
 F 2 "" H 2200 3450 50  0001 C CNN
@@
 VDD_HEAT
 $Comp
-L Device:D_Schottky D7
+L Device:D_Schottky D6
 U 1 1 5B1B03B6
 P 1750 2600
-F 0 "D7" H 1750 2816 50  0000 C CNN
+F 0 "D6" H 1750 2816 50  0000 C CNN
 F 1 "SK310A-LTP" H 1750 2725 50  0000 C CNN
 F 2 "Diode_SMD:D_SMA" H 1750 2600 50  0001 C CNN
@@
 	1500 2600 1600 2600
 $Comp
-L remram-custom:PSMN1R8-40YLC,115 Q3
+L remram-custom:PSMN1R8-40YLC,115 Q2
 U 1 1 5B1B03C5
 P 2000 3050
-F 0 "Q3" H 2387 3046 50  0000 L CNN
+F 0 "Q2" H 2387 3046 50  0000 L CNN
 F 1 "PSMN1R2-30YLC,115" H 2387 2955 50  0000 L CNN
 F 2 "custom-footprints:SOT-669_LFPAK_ThermalVias-1" H 2200 2975 50  0001 L CIN
@@
 	2100 3500 2100 3350
 $Comp
-L Device:R R12
+L Device:R R9
 U 1 1 5B1B03DE
 P 1300 3050
-F 0 "R12" V 1093 3050 50  0000 C CNN
+F 0 "R9" V 1093 3050 50  0000 C CNN
 F 1 "100" V 1184 3050 50  0000 C CNN
 F 2 "Resistor_SMD:R_0603_1608Metric" V 1230 3050 50  0001 C CNN
@@
 Connection ~ 2100 2600
 $Comp
-L remram-custom:BUK9840-55 Q2
+L remram-custom:BUK9840-55 Q3
 U 1 1 5B1FB146
 P 4750 1400
-F 0 "Q2" H 4955 1446 50  0000 L CNN
+F 0 "Q3" H 4955 1446 50  0000 L CNN
 F 1 "BUK9840-55" H 4955 1355 50  0000 L CNN
 F 2 "Package_TO_SOT_SMD:SOT-223-3_TabPin2" H 4950 1325 50  0001 L CIN
@@
 $EndComp
 $Comp
-L Device:R R9
+L Device:R R12
 U 1 1 5B1FB287
 P 4150 1400
-F 0 "R9" V 3943 1400 50  0000 C CNN
+F 0 "R12" V 3943 1400 50  0000 C CNN
 F 1 "100" V 4034 1400 50  0000 C CNN
 F 2 "Resistor_SMD:R_0603_1608Metric" V 4080 1400 50  0001 C CNN
@@
 	3900 1400 4000 1400
 $Comp
-L power:GNDPWR #PWR029
+L power:GNDPWR #PWR033
 U 1 1 5B1FD93D
 P 4850 1850
-F 0 "#PWR029" H 4850 1650 50  0001 C CNN
+F 0 "#PWR033" H 4850 1650 50  0001 C CNN
 F 1 "GNDPWR" H 4850 1700 50  0000 C CNN
 F 2 "" H 4850 1800 50  0001 C CNN
@@
 	3900 3050 4000 3050
 $Comp
-L power:GNDPWR #PWR031
+L power:GNDPWR #PWR034
 U 1 1 5B2008E5
 P 4850 3500
-F 0 "#PWR031" H 4850 3300 50  0001 C CNN
+F 0 "#PWR034" H 4850 3300 50  0001 C CNN
 F 1 "GNDPWR" H 4850 3350 50  0000 C CNN
 F 2 "" H 4850 3450 50  0001 C CNN
@@
 	1600 1400 1800 1400
 $Comp
-L Device:R R14
+L Device:R R11
 U 1 1 5AF8339E
 P 1750 3500
-F 0 "R14" V 1543 3500 50  0000 C CNN
+F 0 "R11" V 1543 3500 50  0000 C CNN
 F 1 "100k" V 1634 3500 50  0000 C CNN
 F 2 "Resistor_SMD:R_0603_1608Metric" V 1680 3500 50  0001 C CNN
@@
 	2100 3500 1900 3500
 $Comp
-L Device:R R11
+L Device:R R14
 U 1 1 5AF83BB4
 P 4600 1850
-F 0 "R11" V 4393 1850 50  0000 C CNN
+F 0 "R14" V 4393 1850 50  0000 C CNN
 F 1 "100k" V 4484 1850 50  0000 C CNN
 F 2 "Resistor_SMD:R_0603_1608Metric" V 4530 1850 50  0001 C CNN
@@
 Connection ~ 4850 3500
 $Comp
-L Device:D_Schottky D6
+L Device:D_Schottky D7
 U 1 1 5AFB8598
 P 4500 950
-F 0 "D6" H 4450 1150 50  0000 L CNN
+F 0 "D7" H 4450 1150 50  0000 L CNN
 F 1 "BAT54GWJ" H 4350 1050 50  0000 L CNN
 F 2 "Diode_SMD:D_SOD-123" H 4500 950 50  0001 C CNN
