File: PCB/motor.sch (KiCad schematic (older format))
At the start: 18 parts, among them J3 70543-0003, U3 TMC2130-TA

Commit message: Version 0.3.
Parts:
- renumbered C13 to C14, C14 to C15, C15 to C16, C16 to C17, C17 to C18, C18 to C19, C19 to C20, C20 to C21, C21 to C22

Commit message: Changed ordering of parts. Version 0.4.
Parts:
- renumbered C14 to C37, C15 to C38, C16 to C39, C17 to C40, C18 to C41, C19 to C42, C20 to C43, C21 to C44, C22 to C45, J3 to J20, R12 to R27, R13 to R28, R14 to R29, TP11 to TP20, TP12 to TP21, TP13 to TP22, TP14 to TP23, U3 to U5

Commit message: Added a battery for SRAM backup.
Parts:
- renumbered C37 to C36, C38 to C37, C39 to C38, C40 to C39, C41 to C40, C42 to C41, C43 to C42, C44 to C43, C45 to C44

Commit message: Change DC-DC layout
The ripple on the 5V and 3V3 rail was too high (360mV).

In an attempt to reduce the RF and HF noise, I changed the layout
to a more compact one. I also added a third 22uF output capacitor
behind the inductor to lower ESR. I also added a 100nf input
capacitor to combat HF noise, as recommended in the datasheet.

The BOM needs to be updated in such a way, that we specificly
choose low ESR resistors.
Parts:
- renumbered C36 to C37, C37 to C38, C38 to C39, C39 to C40, C40 to C41, C41 to C42, C42 to C43, C43 to C44, C44 to C45

Commit message: Add diodes and PU to endstops and fans (SCH only)
For extra protection and PU, we added some diodes and a
pull up resistor to the endstops and the fan tachometer.
Parts:
- renumbered C37 to C45, C38 to C46, C39 to C47, C40 to C48, C41 to C49, C42 to C50, C43 to C51, C44 to C52, C45 to C53, R27 to R37, R28 to R38, R29 to R39
