File: PCB/power.sch (KiCad schematic (older format))
At the start: 41 parts, among them J1 4DB-P108-06, J2 039531-1002, U1 TPS54308, U2 AP2112K-3.3TRG1

Commit message: Added the secnd Z connection.
Connections:
- no-connect marks 1 -> 2
Changed lines of the file:
@@
 	1    0    0    -1
 $EndComp
+NoConn ~ 2500 3050
 $EndSCHEMATC

Commit message: Reworked some traces for better layout.
This will also come in handy, when we add more external
connections (10 to 20pin external).
Parts:
- C1, C10, C12, C3, C4, C5, C6, C7, C8: symbol Device:C -> remram-rescue:C-Device
- C11, C2, C9: symbol Device:CP -> remram-rescue:CP-Device
- D1: symbol Device:LED -> remram-rescue:LED-Device
- D2, D3, D4: symbol Device:D -> remram-rescue:D-Device
- F1, F2, F3: symbol Device:Fuse -> remram-rescue:Fuse-Device
- J1: symbol Connector_Generic:Conn_01x06 -> remram-rescue:Conn_01x06-Connector_Generic
- J2: symbol Connector_Specialized:Conn_01x02_Male -> remram-rescue:Conn_01x02_Male-Connector_Specialized
- L1: symbol Device:L_Core_Iron -> remram-rescue:L_Core_Iron-Device
- R1, R2, R3: symbol Device:R -> remram-rescue:R-Device
- TP1, TP10, TP2, TP3, TP4, TP5, TP6, TP7, TP8, TP9: symbol Connector_Specialized:Test_Point -> remram-rescue:Test_Point-Connector_Specialized
Changed lines of the file:
@@
 	1700 2750 1800 2750
 $Comp
-L Device:C C6
+L remram-rescue:C-Device C6
 U 1 1 5AD0C5B0
 P 1350 2900
@@
 $EndComp
 $Comp
-L Device:C C7
+L remram-rescue:C-Device C7
 U 1 1 5AD0C639
 P 2700 2900
@@
 $EndComp
 $Comp
-L Device:C C3
+L remram-rescue:C-Device C3
 U 1 1 5AF61095
 P 2050 1150
@@
 Connection ~ 2050 1000
 $Comp
-L Device:C C1
+L remram-rescue:C-Device C1
 U 1 1 5AF6112E
 P 3950 1000
@@
 $EndComp
 $Comp
-L Device:C C4
+L remram-rescue:C-Device C4
 U 1 1 5AF611D6
 P 5200 1300
@@
 $EndComp
 $Comp
-L Device:C C5
+L remram-rescue:C-Device C5
 U 1 1 5AF6122A
 P 5600 1300
@@
 $EndComp
 $Comp
-L Device:L_Core_Iron L1
+L remram-rescue:L_Core_Iron-Device L1
 U 1 1 5AF61471
 P 4600 1150
@@
 Connection ~ 5200 1150
 $Comp
-L Device:R R1
+L remram-rescue:R-Device R1
 U 1 1 5AF622B8
 P 6350 1550
@@
 $EndComp
 $Comp
-L Device:R R2
+L remram-rescue:R-Device R2
 U 1 1 5AF62345
 P 6350 1850
@@
 	2050 1000 2700 1000
 $Comp
-L Device:LED D1
+L remram-rescue:LED-Device D1
 U 1 1 5AF67AB2
 P 3550 3200
@@
 max. 3 A
 $Comp
-L Connector_Generic:Conn_01x06 J1
+L remram-rescue:Conn_01x06-Connector_Generic J1
 U 1 1 5AF719E7
 P 1000 4550
@@
 $EndComp
 $Comp
-L Connector_Specialized:Test_Point TP4
+L remram-rescue:Test_Point-Connector_Specialized TP4
 U 1 1 5AF719F4
 P 1900 4400
@@
 	1900 4450 1900 4400
 $Comp
-L Connector_Specialized:Test_Point TP3
+L remram-rescue:Test_Point-Connector_Specialized TP3
 U 1 1 5AF719FF
 P 1900 4100
@@
 	1900 4100 1900 4150
 $Comp
-L Connector_Specialized:Test_Point TP6
+L remram-rescue:Test_Point-Connector_Specialized TP6
 U 1 1 5AF71A0F
 P 1900 5000
@@
 	1900 5050 1900 5000
 $Comp
-L Connector_Specialized:Test_Point TP5
+L remram-rescue:Test_Point-Connector_Specialized TP5
 U 1 1 5AF71A1A
 P 1900 4700
@@
 Connection ~ 1900 4750
 $Comp
-L Connector_Specialized:Test_Point TP10
+L remram-rescue:Test_Point-Connector_Specialized TP10
 U 1 1 5AF71A25
 P 1650 6400
@@
 	1900 5650 1900 5600
 $Comp
-L Connector_Specialized:Test_Point TP7
+L remram-rescue:Test_Point-Connector_Specialized TP7
 U 1 1 5AF71A2E
 P 1900 5300
@@
 	1450 5650 1900 5650
 $Comp
-L Connector_Specialized:Test_Point TP1
+L remram-rescue:Test_Point-Connector_Specialized TP1
 U 1 1 5B12B288
 P 6650 1150
@@
 	3850 2750 3550 2750
 $Comp
-L Connector_Specialized:Test_Point TP2
+L remram-rescue:Test_Point-Connector_Specialized TP2
 U 1 1 5B12E486
 P 3850 2750
@@
 Connection ~ 3850 2750
 $Comp
-L Device:Fuse F1
+L remram-rescue:Fuse-Device F1
 U 1 1 5AF82AAA
 P 4000 4150
@@
 $EndComp
 $Comp
-L Device:Fuse F2
+L remram-rescue:Fuse-Device F2
 U 1 1 5AF6A259
 P 4000 4700
@@
 $EndComp
 $Comp
-L Device:Fuse F3
+L remram-rescue:Fuse-Device F3
 U 1 1 5AF6B243
 P 4000 5300
@@
 	2550 1150 2700 1150
 $Comp
-L Device:D D2
+L remram-rescue:D-Device D2
 U 1 1 5AFA3F16
 P 4350 4300
@@
 $EndComp
 $Comp
-L Device:CP C9
+L remram-rescue:CP-Device C9
 U 1 1 5AFA5D98
 P 5000 4850
@@
 $EndComp
 $Comp
-L Device:D D3
+L remram-rescue:D-Device D3
 U 1 1 5AFAB14E
 P 4350 4850
@@
 $EndComp
 $Comp
-L Device:C C12
+L remram-rescue:C-Device C12
 U 1 1 5AFBE17F
 P 5450 5450
@@
 $EndComp
 $Comp
-L Device:D D4
+L remram-rescue:D-Device D4
 U 1 1 5AFBE18D
 P 4350 5450
@@
 $EndComp
 $Comp
-L Device:C C10
+L remram-rescue:C-Device C10
 U 1 1 5AFCAA09
 P 5450 4850
@@
 $EndComp
 $Comp
-L Device:C C8
+L remram-rescue:C-Device C8
 U 1 1 5AFCC3AE
 P 5450 4300
@@
 	4150 5300 4350 5300
 $Comp
-L Device:CP C11
+L remram-rescue:CP-Device C11
 U 1 1 5AFD173F
 P 5000 5450
@@
 BED_OUT
 $Comp
-L Connector_Specialized:Conn_01x02_Male J2
+L remram-rescue:Conn_01x02_Male-Connector_Specialized J2
 U 1 1 5B1B2A8C
 P 1000 6100
@@
 HEAT_OUT
 $Comp
-L Connector_Specialized:Test_Point TP9
+L remram-rescue:Test_Point-Connector_Specialized TP9
 U 1 1 5B1B93AE
 P 1650 6100
@@
 $EndComp
 $Comp
-L Connector_Specialized:Test_Point TP8
+L remram-rescue:Test_Point-Connector_Specialized TP8
 U 1 1 5B1BD224
 P 1900 5600
@@
 	1250 1000 1550 1000
 $Comp
-L Device:CP C2
+L remram-rescue:CP-Device C2
 U 1 1 5AFA3BBA
 P 1550 1150
@@
 	2700 2750 3550 2750
 $Comp
-L Device:R R3
+L remram-rescue:R-Device R3
 U 1 1 5AF56C08
 P 3550 2900

Commit message: Reworked some traces and labels.
Parts:
- renumbered C6 to C1, C12 to C11, C5 to C12, C7 to C4, C1 to C5, C9 to C6, C11 to C7, C4 to C8, C8 to C9, R3 to R1, R1 to R2, R2 to R3, TP9 to TP1, TP1 to TP10, TP10 to TP2, TP2 to TP9, U2 to U1, U1 to U2

Commit message: First draft of RemRam.
I added a 20 pin expansion connector with the following pins:
 - SPI
 - I2C
 - USART
 - 4x PWM
 - 4x GPIO
Parts:
- renumbered C5 to C1, C7 to C11, C11 to C12, C8 to C4, C12 to C5, C1 to C6, C4 to C7, C9 to C8, C6 to C9, R2 to R1, R3 to R2, R1 to R3, TP10 to TP1, TP2 to TP10, TP9 to TP2, TP1 to TP9, U2 to U1, U1 to U2

Commit message: Version 0.3.
Parts:
- added C8: 100uF, Capacitor_THT:CP_Radial_D6.3mm_P2.50mm, symbol remram-rescue:CP-Device
- C3: footprint Capacitor_SMD:C_0603_1608Metric -> Capacitor_SMD:C_1206_3216Metric
- renumbered C9 to C10, C10 to C11, C11 to C12, C12 to C13, C8 to C9
Connections:
- wire segments 90 -> 91
Changed lines of the file:
@@
 F 0 "C3" H 2165 1196 50  0000 L CNN
 F 1 "10uF" H 2165 1105 50  0000 L CNN
-F 2 "Capacitor_SMD:C_0603_1608Metric" H 2088 1000 50  0001 C CNN
+F 2 "Capacitor_SMD:C_1206_3216Metric" H 2088 1000 50  0001 C CNN
 F 3 "~" H 2050 1150 50  0001 C CNN
 	1    2050 1150
 	1    0    0    -1
 $EndComp
-Connection ~ 2050 1000
 $Comp
 L remram-rescue:C-Device C1
@@
 Connection ~ 5600 1150
 Connection ~ 6350 1150
-Wire Wire Line
-	2050 1000 2700 1000
 $Comp
 L remram-rescue:LED-Device D1
@@
 	1900 4450 2650 4450
 $Comp
-L power:GNDPWR #PWR018
+L power:GNDPWR #PWR019
 U 1 1 5AF87BAE
 P 2650 5050
-F 0 "#PWR018" H 2650 4850 50  0001 C CNN
+F 0 "#PWR019" H 2650 4850 50  0001 C CNN
 F 1 "GNDPWR" H 2650 4900 50  0000 C CNN
 F 2 "" H 2650 5000 50  0001 C CNN
@@
 	1    0    0    -1
 $EndComp
-Wire Wire Line
-	1550 1600 1550 1300
-Wire Wire Line
-	1550 1300 2050 1300
 $Comp
 L power:GNDPWR #PWR06
@@
 $EndComp
 $Comp
-L remram-rescue:CP-Device C9
+L remram-rescue:CP-Device C10
 U 1 1 5AFA5D98
 P 5000 4850
-F 0 "C9" H 5118 4896 50  0000 L CNN
+F 0 "C10" H 5118 4896 50  0000 L CNN
 F 1 "100uF" H 5118 4805 50  0000 L CNN
 F 2 "Capacitor_THT:CP_Radial_D6.3mm_P2.50mm" H 5038 4700 50  0001 C CNN
@@
 $EndComp
 $Comp
-L power:GNDPWR #PWR014
+L power:GNDPWR #PWR015
 U 1 1 5AFB71B9
 P 5450 4450
-F 0 "#PWR014" H 5450 4250 50  0001 C CNN
+F 0 "#PWR015" H 5450 4250 50  0001 C CNN
 F 1 "GNDPWR" H 5450 4300 50  0000 C CNN
 F 2 "" H 5450 4400 50  0001 C CNN
@@
 $EndComp
 $Comp
-L power:GNDPWR #PWR015
+L power:GNDPWR #PWR016
 U 1 1 5AFB8B47
 P 4350 5000
-F 0 "#PWR015" H 4350 4800 50  0001 C CNN
+F 0 "#PWR016" H 4350 4800 50  0001 C CNN
 F 1 "GNDPWR" H 4350 4850 50  0000 C CNN
 F 2 "" H 4350 4950 50  0001 C CNN
@@
 $EndComp
 $Comp
-L power:GNDPWR #PWR016
+L power:GNDPWR #PWR017
 U 1 1 5AFBA4D5
 P 5000 5000
-F 0 "#PWR016" H 5000 4800 50  0001 C CNN
+F 0 "#PWR017" H 5000 4800 50  0001 C CNN
 F 1 "GNDPWR" H 5000 4850 50  0000 C CNN
 F 2 "" H 5000 4950 50  0001 C CNN
@@
 $EndComp
 $Comp
-L power:GNDPWR #PWR017
+L power:GNDPWR #PWR018
 U 1 1 5AFBBE63
 P 5450 5000
-F 0 "#PWR017" H 5450 4800 50  0001 C CNN
+F 0 "#PWR018" H 5450 4800 50  0001 C CNN
 F 1 "GNDPWR" H 5450 4850 50  0000 C CNN
 F 2 "" H 5450 4950 50  0001 C CNN
@@
 $EndComp
 $Comp
-L remram-rescue:C-Device C12
+L remram-rescue:C-Device C13
 U 1 1 5AFBE17F
 P 5450 5450
-F 0 "C12" H 5565 5496 50  0000 L CNN
+F 0 "C13" H 5565 5496 50  0000 L CNN
 F 1 "100nF" H 5565 5405 50  0000 L CNN
 F 2 "Capacitor_SMD:C_1812_4532Metric" H 5488 5300 50  0001 C CNN
@@
 Connection ~ 5450 5300
 $Comp
-L power:GNDPWR #PWR019
+L power:GNDPWR #PWR020
 U 1 1 5AFC4CE3
 P 4350 5600
-F 0 "#PWR019" H 4350 5400 50  0001 C CNN
+F 0 "#PWR020" H 4350 5400 50  0001 C CNN
 F 1 "GNDPWR" H 4350 5450 50  0000 C CNN
 F 2 "" H 4350 5550 50  0001 C CNN
@@
 $EndComp
 $Comp
-L power:GNDPWR #PWR020
+L power:GNDPWR #PWR021
 U 1 1 5AFC4CE9
 P 5000 5600
-F 0 "#PWR020" H 5000 5400 50  0001 C CNN
+F 0 "#PWR021" H 5000 5400 50  0001 C CNN
 F 1 "GNDPWR" H 5000 5450 50  0000 C CNN
 F 2 "" H 5000 5550 50  0001 C CNN
@@
 $EndComp
 $Comp
-L power:GNDPWR #PWR021
+L power:GNDPWR #PWR022
 U 1 1 5AFC4CEF
 P 5450 5600
-F 0 "#PWR021" H 5450 5400 50  0001 C CNN
+F 0 "#PWR022" H 5450 5400 50  0001 C CNN
 F 1 "GNDPWR" H 5450 5450 50  0000 C CNN
 F 2 "" H 5450 5550 50  0001 C CNN
@@
 $EndComp
 $Comp
-L remram-rescue:C-Device C10
+L remram-rescue:C-Device C11
 U 1 1 5AFCAA09
 P 5450 4850
-F 0 "C10" H 5565 4896 50  0000 L CNN
+F 0 "C11" H 5565 4896 50  0000 L CNN
 F 1 "100nF" H 5565 4805 50  0000 L CNN
 F 2 "Capacitor_SMD:C_1812_4532Metric" H 5488 4700 50  0001 C CNN
@@
 $EndComp
 $Comp
-L remram-rescue:C-Device C8
+L remram-rescue:C-Device C9
 U 1 1 5AFCC3AE
 P 5450 4300
-F 0 "C8" H 5565 4346 50  0000 L CNN
+F 0 "C9" H 5565 4346 50  0000 L CNN
 F 1 "100nF" H 5565 4255 50  0000 L CNN
 F 2 "Capacitor_SMD:C_1812_4532Metric" H 5488 4150 50  0001 C CNN
@@
 Connection ~ 5450 4150
 Wire Wire Line
-	5450 4150 4350 4150
-Wire Wire Line
 	5000 4700 5450 4700
 Connection ~ 5000 4700
@@
 	4150 5300 4350 5300
 $Comp
-L remram-rescue:CP-Device C11
+L remram-rescue:CP-Device C12
 U 1 1 5AFD173F
 P 5000 5450
-F 0 "C11" H 5118 5496 50  0000 L CNN
+F 0 "C12" H 5118 5496 50  0000 L CNN
 F 1 "100uF" H 5118 5405 50  0000 L CNN
 F 2 "Capacitor_THT:CP_Radial_D6.3mm_P2.50mm" H 5038 5300 50  0001 C CNN
@@
 Connection ~ 1900 4150
 $Comp
-L power:GNDPWR #PWR023
+L power:GNDPWR #PWR024
 U 1 1 5AFD7C84
 P 1300 7250
-F 0 "#PWR023" H 1300 7050 50  0001 C CNN
+F 0 "#PWR024" H 1300 7050 50  0001 C CNN
 F 1 "GNDPWR" H 1300 7100 50  0000 C CNN
 F 2 "" H 1300 7200 50  0001 C CNN
@@
 $EndComp
 $Comp
-L power:GND #PWR024
+L power:GND #PWR025
 U 1 1 5AFD7DB1
 P 1200 7350
-F 0 "#PWR024" H 1200 7100 50  0001 C CNN
+F 0 "#PWR025" H 1200 7100 50  0001 C CNN
 F 1 "GND" H 1200 7200 50  0000 C CNN
 F 2 "" H 1200 7350 50  0001 C CNN
@@
 Ground Plane Connections
 $Comp
-L power:GNDA #PWR022
+L power:GNDA #PWR023
 U 1 1 5B058B1E
 P 1100 7250
-F 0 "#PWR022" H 1100 7000 50  0001 C CNN
+F 0 "#PWR023" H 1100 7000 50  0001 C CNN
 F 1 "GNDA" H 1105 7077 50  0000 C CNN
 F 2 "" H 1100 7250 50  0001 C CNN
@@
 	1    0    0    -1
 $EndComp
-Wire Wire Line
-	1250 1000 1550 1000
 $Comp
 L remram-rescue:CP-Device C2
@@
 	1    0    0    -1
 $EndComp
-Connection ~ 1550 1000
-Wire Wire Line
-	1550 1000 2050 1000
 Wire Wire Line
 	1100 7250 1200 7250
@@
 	1200 7250 1300 7250
 $Comp
-L power:GNDPWR #PWR025
+L power:GNDPWR #PWR026
 U 1 1 5AFCD887
 P 4050 7350
-F 0 "#PWR025" H 4050 7150 50  0001 C CNN
+F 0 "#PWR026" H 4050 7150 50  0001 C CNN
 F 1 "GNDPWR" H 4054 7196 50  0000 C CNN
 F 2 "" H 4050 7300 50  0001 C CNN
@@
 $EndComp
 NoConn ~ 2500 3050
+Wire Wire Line
+	2050 1000 2700 1000
+Connection ~ 2050 1000
+Wire Wire Line
+	1550 1300 2050 1300
+Wire Wire Line
+	5450 4150 4950 4150
+Wire Wire Line
+	1550 1600 1550 1300
+Connection ~ 1550 1000
+Wire Wire Line
+	1550 1000 2050 1000
+Wire Wire Line
+	1250 1000 1550 1000
+$Comp
+L remram-rescue:CP-Device C8
+U 1 1 5B0321B5
+P 4950 4300
+F 0 "C8" H 5068 4346 50  0000 L CNN
+F 1 "100uF" H 5068 4255 50  0000 L CNN
+F 2 "Capacitor_THT:CP_Radial_D6.3mm_P2.50mm" H 4988 4150 50  0001 C CNN
+F 3 "https://eu.mouser.com/datasheet/2/293/e-uvz-1219460.pdf" H 4950 4300 50  0001 C CNN
+	1    4950 4300
+	1    0    0    -1
+$EndComp
+$Comp
+L power:GNDPWR #PWR014
+U 1 1 5B034E9B
+P 4950 4450
+F 0 "#PWR014" H 4950 4250 50  0001 C CNN
+F 1 "GNDPWR" H 4950 4300 50  0000 C CNN
+F 2 "" H 4950 4400 50  0001 C CNN
+F 3 "" H 4950 4400 50  0001 C CNN
+	1    4950 4450
+	1    0    0    -1
+$EndComp
+Connection ~ 4950 4150
+Wire Wire Line
+	4950 4150 4350 4150
 $EndSCHEMATC

Commit message: Change DC-DC layout
The ripple on the 5V and 3V3 rail was too high (360mV).

In an attempt to reduce the RF and HF noise, I changed the layout
to a more compact one. I also added a third 22uF output capacitor
behind the inductor to lower ESR. I also added a 100nf input
capacitor to combat HF noise, as recommended in the datasheet.

The BOM needs to be updated in such a way, that we specificly
choose low ESR resistors.
Parts:
- added C6: 22uF, Capacitor_SMD:C_1206_3216Metric, symbol remram-rescue:C-Device
- C3: renamed from C2; value 100uF -> 100nF; footprint Capacitor_THT:CP_Radial_D6.3mm_P2.50mm -> Capacitor_SMD:C_1206_3216Metric; symbol remram-rescue:CP-Device -> Device:C
- C4, C5: footprint Capacitor_SMD:C_0603_1608Metric -> Capacitor_SMD:C_1206_3216Metric
- renumbered C9 to C10, C10 to C11, C11 to C12, C12 to C13, C13 to C14, C3 to C2, C6 to C7, C7 to C8, C8 to C9
Connections:
- wire segments 91 -> 92
Other:
- note added: "TODO: Insert a 100nF?"

Commit message: Change 1k resistors to 4.7k. Update Symbols
Had to update the symbols to the right library again, since
Kicad Nightly changed their library order.

Also changed the 1k resistors to 4.7k to unify resistors and
also upped the PU to a weaker value.
Parts:
- C1, C10, C12, C14, C2, C4, C5, C6, C7, C8: symbol remram-rescue:C-Device -> Device:C
- C11, C13, C9: symbol remram-rescue:CP-Device -> Device:CP
- D1: symbol remram-rescue:LED-Device -> Device:LED
- D2, D3, D4: symbol remram-rescue:D-Device -> Device:D
- F1, F2, F3: symbol remram-rescue:Fuse-Device -> Device:Fuse
- J1: symbol remram-rescue:Conn_01x06-Connector_Generic -> Connector_Generic:Conn_01x06
- J2: symbol remram-rescue:Conn_01x02_Male-Connector_Specialized -> Connector:Conn_01x02_Male
- L1: symbol remram-rescue:L_Core_Iron-Device -> Device:L_Core_Iron
- R1, R2: symbol remram-rescue:R-Device -> Device:R
- R3: value 1k -> 4.7k; symbol remram-rescue:R-Device -> Device:R
- TP1, TP10, TP2, TP3, TP4, TP5, TP6, TP7, TP8, TP9: symbol remram-rescue:Test_Point-Connector_Specialized -> Connector:Test_Point
Changed lines of the file:
@@
 	1700 2750 1800 2750
 $Comp
-L remram-rescue:C-Device C7
+L Device:C C7
 U 1 1 5AD0C5B0
 P 1350 2900
@@
 $EndComp
 $Comp
-L remram-rescue:C-Device C8
+L Device:C C8
 U 1 1 5AD0C639
 P 2700 2900
@@
 $EndComp
 $Comp
-L remram-rescue:C-Device C2
+L Device:C C2
 U 1 1 5AF61095
 P 1550 1150
@@
 $EndComp
 $Comp
-L remram-rescue:C-Device C1
+L Device:C C1
 U 1 1 5AF6112E
 P 3950 1000
@@
 $EndComp
 $Comp
-L remram-rescue:C-Device C4
+L Device:C C4
 U 1 1 5AF611D6
 P 5200 1300
@@
 $EndComp
 $Comp
-L remram-rescue:C-Device C5
+L Device:C C5
 U 1 1 5AF6122A
 P 5600 1300
@@
 $EndComp
 $Comp
-L remram-rescue:L_Core_Iron-Device L1
+L Device:L_Core_Iron L1
 U 1 1 5AF61471
 P 4600 1150
@@
 Connection ~ 5200 1150
 $Comp
-L remram-rescue:R-Device R1
+L Device:R R1
 U 1 1 5AF622B8
 P 6350 1550
@@
 $EndComp
 $Comp
-L remram-rescue:R-Device R2
+L Device:R R2
 U 1 1 5AF62345
 P 6350 1850
@@
 Connection ~ 6350 1150
 $Comp
-L remram-rescue:LED-Device D1
+L Device:LED D1
 U 1 1 5AF67AB2
 P 3550 3200
@@
 max. 3 A
 $Comp
-L remram-rescue:Conn_01x06-Connector_Generic J1
+L Connector_Generic:Conn_01x06 J1
 U 1 1 5AF719E7
 P 1000 4550
@@
 $EndComp
 $Comp
-L remram-rescue:Test_Point-Connector_Specialized TP4
+L Connector:Test_Point TP4
 U 1 1 5AF719F4
 P 1900 4400
@@
 	1900 4450 1900 4400
 $Comp
-L remram-rescue:Test_Point-Connector_Specialized TP3
+L Connector:Test_Point TP3
 U 1 1 5AF719FF
 P 1900 4100
@@
 	1900 4100 1900 4150
 $Comp
-L remram-rescue:Test_Point-Connector_Specialized TP6
+L Connector:Test_Point TP6
 U 1 1 5AF71A0F
 P 1900 5000
@@
 	1900 5050 1900 5000
 $Comp
-L remram-rescue:Test_Point-Connector_Specialized TP5
+L Connector:Test_Point TP5
 U 1 1 5AF71A1A
 P 1900 4700
@@
 Connection ~ 1900 4750
 $Comp
-L remram-rescue:Test_Point-Connector_Specialized TP10
+L Connector:Test_Point TP10
 U 1 1 5AF71A25
 P 1650 6400
@@
 	1900 5650 1900 5600
 $Comp
-L remram-rescue:Test_Point-Connector_Specialized TP7
+L Connector:Test_Point TP7
 U 1 1 5AF71A2E
 P 1900 5300
@@
 	1450 5650 1900 5650
 $Comp
-L remram-rescue:Test_Point-Connector_Specialized TP1
+L Connector:Test_Point TP1
 U 1 1 5B12B288
 P 6650 1150
@@
 	3850 2750 3550 2750
 $Comp
-L remram-rescue:Test_Point-Connector_Specialized TP2
+L Connector:Test_Point TP2
 U 1 1 5B12E486
 P 3850 2750
@@
 Connection ~ 3850 2750
 $Comp
-L remram-rescue:Fuse-Device F1
+L Device:Fuse F1
 U 1 1 5AF82AAA
 P 4000 4150
@@
 $EndComp
 $Comp
-L remram-rescue:Fuse-Device F2
+L Device:Fuse F2
 U 1 1 5AF6A259
 P 4000 4700
@@
 $EndComp
 $Comp
-L remram-rescue:Fuse-Device F3
+L Device:Fuse F3
 U 1 1 5AF6B243
 P 4000 5300
@@
 	2550 1150 2700 1150
 $Comp
-L remram-rescue:D-Device D2
+L Device:D D2
 U 1 1 5AFA3F16
 P 4350 4300
@@
 $EndComp
 $Comp
-L remram-rescue:CP-Device C11
+L Device:CP C11
 U 1 1 5AFA5D98
 P 5000 4850
@@
 $EndComp
 $Comp
-L remram-rescue:D-Device D3
+L Device:D D3
 U 1 1 5AFAB14E
 P 4350 4850
@@
 $EndComp
 $Comp
-L remram-rescue:C-Device C14
+L Device:C C14
 U 1 1 5AFBE17F
 P 5450 5450
@@
 $EndComp
 $Comp
-L remram-rescue:D-Device D4
+L Device:D D4
 U 1 1 5AFBE18D
 P 4350 5450
@@
 $EndComp
 $Comp
-L remram-rescue:C-Device C12
+L Device:C C12
 U 1 1 5AFCAA09
 P 5450 4850
@@
 $EndComp
 $Comp
-L remram-rescue:C-Device C10
+L Device:C C10
 U 1 1 5AFCC3AE
 P 5450 4300
@@
 	4150 5300 4350 5300
 $Comp
-L remram-rescue:CP-Device C13
+L Device:CP C13
 U 1 1 5AFD173F
 P 5000 5450
@@
 BED_OUT
 $Comp
-L remram-rescue:Conn_01x02_Male-Connector_Specialized J2
+L Connector:Conn_01x02_Male J2
 U 1 1 5B1B2A8C
 P 1000 6100
@@
 HEAT_OUT
 $Comp
-L remram-rescue:Test_Point-Connector_Specialized TP9
+L Connector:Test_Point TP9
 U 1 1 5B1B93AE
 P 1650 6100
@@
 $EndComp
 $Comp
-L remram-rescue:Test_Point-Connector_Specialized TP8
+L Connector:Test_Point TP8
 U 1 1 5B1BD224
 P 1900 5600
@@
 	2700 2750 3550 2750
 $Comp
-L remram-rescue:R-Device R3
+L Device:R R3
 U 1 1 5AF56C08
 P 3550 2900
 F 0 "R3" H 3620 2946 50  0000 L CNN
-F 1 "1k" H 3620 2855 50  0000 L CNN
+F 1 "4.7k" H 3620 2855 50  0000 L CNN
 F 2 "Resistor_SMD:R_0603_1608Metric" V 3480 2900 50  0001 C CNN
 F 3 "~" H 3550 2900 50  0001 C CNN
@@
 	1250 1000 1550 1000
 $Comp
-L remram-rescue:CP-Device C9
+L Device:CP C9
 U 1 1 5B0321B5
 P 4950 4300
@@
 	2050 1000 2700 1000
 $Comp
-L remram-rescue:C-Device C6
+L Device:C C6
 U 1 1 5B31591E
 P 6000 1300
